File: Kicad test/Kicad test.kicad_sch (KiCad schematic)
At the start: 49 parts, among them J1 Conn_01x02_Pin, J2 Conn_01x02_Pin, J3 XT60-M, J4 22035035, J5 XT60-M, U1 INA181A1QDBVRQ1, U2 PADS131M04QPWRQ1, U4 UA78M05QDCYRG4Q1 LDO, X1 ASCO

Commit message: added some values
Parts:
- removed C11: 1uF,50V, C0805, symbol SMV_Custom:C0805C102K5GACTU
- removed C15: 0.1uF,50V, C0805, symbol SMV_Custom:C0805C104K5RACTU
- removed C6: C_Small, symbol Device:C_Small
- removed J1, J2: Conn_01x02_Pin, symbol Connector:Conn_01x02_Pin
- removed R3, R7: R, symbol Device:R
- added C11: 0.1uF,50V, C0805, symbol SMV_Custom:C0805C104K5RACTU
- added D1, D2: LED, symbol Device:LED
- added R20: 1k, symbol Device:R
- added R21: 2.49k, symbol Device:R
- added R22: 1.00k, symbol Device:R
- added R23, R7: CRCW080510R0FKEAHP, RES_CRCW_0805_VIS, symbol SMV_Custom:CRCW080510R0FKEAHP
- added R3: 10k, 0.125W, CRCW080510K0FKEAC:RESC2012X60N, symbol SMV_Custom:CRCW080510K0FKEAC
- added TP1, TP2, TP3, TP4, TP5, TP6, TP7, TP8, TP9: TestPoint, symbol Connector:TestPoint
- C1: value 220-nF -> 0.1u
- C13: value C_Small -> 10u
- C2, C4, C7, C8, C9: value C_Small -> 0.1u
- C3: value 1u -> 10u
- R15, R17: value R -> 10k
- R16: value R -> 10
- R2: value R -> 1k
- R4: value R -> 50
- R6: value R -> 14.0k
- R9: value R -> 1.00k
Connections:
- net +12V: now also TP1.1; no longer C10.1, J3.P (POS), R18.1
- net +12VOUT: now also C10.1, J3.P (POS), R18.1, TP2.1
- net +3V3: now also C16.1, U2.20 (DVDD), D1.2 (A), D2.2 (A), R21.1, R23.2, R3.1, R7.2; no longer R2.1
- net +5V: now also C3.1, TP5.1
- net A2: now also R2.2
- net A3: now also R20.2
- net GND: now also C1.2, C3.2, C5.2, C11.2, R22.2; no longer U2.7 (AIN2P)
- net ~{RESET}: now also C5.1, R15.2
- net at C1.1: now also U2.7 (AIN2P), R21.2, R22.1
- net at C18.1, U2.1 (AVDD): now also R23.1
- net at R4.1, U1.1: now also TP3.1
- net at U1.6: now also C11.1, R7.1; no longer R2.2
- net at C7.1, R6.2, R9.1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: now also TP4.1
- net DIN_R: now reaches R8.1, U2.16 (DIN)
- net DIN_R: now also TP9.1
- net SYNC/RESET_R: now reaches R14.1, U2.11 (SYNC/RESET)
- net CS_R: now reaches R13.1, U2.12 (CS)
- net CS_R: now also R3.2, TP7.1; no longer R15.2
- net DRDY_R: now reaches R12.1, U2.13 (DRDY)
- net SCLK_R: now reaches R11.1, U2.14 (SCLK)
- net SCLK_R: now also TP6.1
- net DOUT_R: now reaches R10.1, U2.15 (DOUT)
- net DOUT_R: now also TP8.1
- net D4 renamed CS
- net MISO renamed DOUT
- net MOSI renamed DIN
- net VBAT: no longer names the net of JP2.1
- new net: D2.1 (K), R20.1
- new net: D1.1 (K), R2.1
Other:
- note added: "Battery"
- note added: "Load"
- note added: "Q: do we need to generate a reset signal?"
- note added: "Resistors are helpful for tuning after manufacturing 22ohm"
- note added: "r10, r12 close to ADC"
- note added: "resistors placed on source side"
- note removed: "220n or 0.22u"
- note removed: "Resistors are helpful for tuning after manufacturing"
- note removed: "power connector"
- moved on the sheet: C10, C12, C13, C14, C18, C2, C4, C9, J3, J5, R1, R10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
