File: Headlight and Sensors/H&S Board/H&S Board.kicad_sch (KiCad schematic)
At the start: 33 parts, among them J1 XT60-M, J2 XT60-M, J3 22035035, J4 Molex Micro-Fit 4 Pin, J5 XT60-M, J6 XT60-M, J7 DAQ Board, J8 Driver UI, J9 XT60-M, Q1 PSMN1R8-40YLC,115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

Commit message: looked at it
Other:
- note added: "Am I allowed to put two sensors onto a single ADC? How to read individual sensor data? Yes, you're allowed up to 4. To read individual sensor data you would need to access some registers (so software mainly)"
- note added: "DRDY can be left floating if unused? Yes"
- note removed: "Am I allowed to put two sensors onto a single ADC? How to read individual sensor data?"
- note removed: "DRDY can be left floating if unused?"
Changed lines of the file:
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@@
 		)
 	)
-	(text "Am I allowed to put two sensors onto a single ADC? How to read individual sensor data?"
+	(text "Am I allowed to put two sensors onto a single ADC? How to read individual sensor data?\nYes, you're allowed up to 4. To read individual sensor data you would\nneed to access some registers (so software mainly)\n"
 		(exclude_from_sim no)
 		(at 57.404 142.494 0)
@@
 		)
 	)
-	(text "DRDY can be left floating if unused?"
+	(text "DRDY can be left floating if unused? Yes\n"
 		(exclude_from_sim no)
 		(at 120.904 121.412 0)
