File: Headlight and Sensors/H&S Board/H&S Board.kicad_sch (KiCad schematic)
At the start: 49 parts, among them J1 XT60-M, J2 XT60-M, J3 22035035, J4 Molex Micro-Fit 4 Pin, J5 XT60-M, J6 XT60-M, J7 DAQ Board, J8 Driver UI, J9 XT60-M, Q1 PSMN1R8-40YLC,115, Q2 PSMN1R8-40YLC,115, Q3 PSMN1R8-40YLC,115, U1 ASM330LHHTR, U2 UA78M05QDCYRG4Q1, U3 MCP6286T-E/OT, U4 ADS131M04IPWR, U5 MCP6286T-E/OT, U6 MCP6286T-E/OT

Commit message: replaced dummy resistors and caps
Parts:
- removed C1, C3: 100 uF, symbol Device:C
- removed C10: 0.33 uF, symbol Device:C
- removed C11, C7, C8: 4.7 nF, symbol Device:C
- removed C2: 10 uF, symbol Device:C
- removed C4: 1 uF, symbol Device:C
- removed C5: 1 uF, symbol Device:C_Small
- removed C9: 0.1 uF, symbol Device:C
- removed R10: 10kohms, 0.125W, SMV_Passives:0805RESC2012X60N, symbol SMV_Custom:CRCW080510K0FKEAC
- removed R11, R13: 50ohms, SMV_Passives:0805RESC2012X60N, symbol SMV_Custom:CRCW080544R2FKEA
- removed R12, R16: 20kohms, SMV_Passives:0805RESC2012X60N, symbol SMV_Custom:CRCW080544R2FKEA
- removed R18: 50 ohms, SMV_Passives:0805RESC2012X60N, symbol SMV_Custom:CRCW080544R2FKEA
- removed R2, R3, R7: 1kohm, SMV_Passives:0805RESC2012X60N, symbol SMV_Custom:CRCW080544R2FKEA
- removed R5, R6: R_US, symbol Device:R_US
- removed R9: 2.5kohms, SMV_Passives:0805RESC2012X60N, symbol SMV_Custom:CRCW080544R2FKEA
- removed RP1: ~, symbol SMV_Custom:RP2040
- added C1: C0805C106K8RACTU, SMV_Passives:Cap0805, symbol SMV_Custom:C0805C106K8RACTU
- added C10, C4: 1uF,16V, SMV_Passives:Cap0805, symbol SMV_Custom:C0805C105K4RACTU
- added C11, C12, C3: 0.1uF,50V, SMV_Passives:Cap0805, symbol SMV_Custom:C0805C104K5RACTU
- added C5, C7, C8: 4.7uF,16V, SMV_Passives:Cap0805, symbol SMV_Custom:C0805C475K4RACTU
- added C9: 0.33uF,50V, SMV_Passives:Cap0805, symbol SMV_Custom:C0805C334K5RACTU
- added D1: WL-SMCW_0603, SMV_Passives:WL-SMCW_0603(diode), symbol SMV_Custom:WL-SMCW_0603
- added R10: CRCW080540K0FKEA, SMV_Passives:0805RESC2012X60N, symbol SMV_Custom:CRCW080540K0FKEA
- added R11, R13, R5: CRCW020149R9FNED, 50Ω, SMV_Passives:0805RESC2012X60N, symbol SMV_Custom:CRCW020149R9FNED
- added R12, R7: CRCW080520K0FKEAC, SMV_Passives:0805RESC2012X60N, symbol SMV_Custom:CRCW080520K0FKEAC
- added R16, R2, R3: CRCW06031K00FKEA, 1KΩ, SMV_Passives:0805RESC2012X60N, symbol SMV_Custom:CRCW06031K00FKEA
- added R6, R8, R9: 10kohms, 0.125W, SMV_Passives:0805RESC2012X60N, symbol SMV_Custom:CRCW080510K0FKEAC
- added RP2: ~, SMV_Connectors:RP2040, symbol SMV_Custom:RP2040
- added TP3, TP4: TestPoint, TestPoint:TestPoint_Pad_D1.0mm, symbol Connector:TestPoint
Connections:
- net 3.3V is gone; now on net +3.3V: U4.20 (DVDD)
- net 3V3 is gone; now on net +3.3V: U1.5 (VDD_IO), U1.8 (VDD)
- net 5V is gone; now on net +5V: J3.1, J4.1
- net CAN2 is gone; now on net GND: J7.2, J8.2
- net VDDIO is gone; now on net D12: U1.2 (RES), U1.3 (RES)
- net +12V: now also C9.2
- net +3.3V: now also C1.2, C10.1, C11.1, C3.1, C4.1, D1.1
- net +5V: now also C12.2
- net A0: now also RP2.24 (A0)
- net A1: now also RP2.23 (A1)
- net A2: now also RP2.22 (A2)
- net A3: now also RP2.21 (A3)
- net CS 0: now also R6.1, TP4.1
- net CS 1: now also R8.1
- net D24: now also RP2.20 (D24)
- net D25: now also RP2.19 (D25)
- net D4: now also R16.1, R2.1, R3.1, RP2.13 (D4)
- net DVDD: now also R6.2
- net GND: now also C1.1, C10.2, C11.2, C12.1, C3.2, C4.2, C5.1, C7.1, C8.1, C9.1, R10.1, RP2.25 (GND), RP2.30 (GND)
- net MISO: now also RP2.16 (MISO)
- net MOSI: now also RP2.17 (MOSI)
- net Press_ADC_P: now also C5.2, R13.2
- net Press_P: now also R9.1
- net RX: now also RP2.15 (RX)
- net SCK: now also RP2.18 (SCK)
- net TX: now also RP2.14 (TX)
- net Torque_ADC_N: now also C8.2, R5.2
- net Torque_ADC_P: now also C7.2, R11.2
- net Torque_N: now also R12.2
- net Torque_P: now also R7.2
- net VDD_IO: now also R8.2
- net ~{RESET}: now also RP2.28 (RESET)
- net at Q1.4 (G), R15.2: now also R16.2
- net at Q2.4 (G), R1.2: now also R2.2
- net at U3.3 (VIN+): now also R10.2, R9.2
- net at R14.1, U5.3 (VIN+): now also R7.1
- net at Q3.4 (G), R4.2: now also R3.2
- net at U3.1 (VOUT), U3.4 (VIN-): now also R13.1
- net at R17.1, U6.3 (VIN+): now also R12.1
- net at U6.1 (VOUT), U6.4 (VIN-): now also R5.1
- net at U5.1 (VOUT), U5.4 (VIN-): now also R11.1
- net CAN1: no longer names the net of J7.3, J8.3
- net CAN1: now also RP2.31 (CAN_H)
- net CAN3: no longer names the net of J7.1, J8.1
- net CAN3: now also RP2.29 (CAN_L)
- new net: D1.2, RP2.26 (3.3V), RP2.27 (3.3V)
Other:
- note removed: "Change the VDDIO"
- moved on the sheet: C6, J6, J7, J8, Q1, Q2, Q3, R1, R15, R17, R4, TP1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

Commit message: added buffer sheet
Parts:
- removed C5, C7, C8: 4.7uF,16V, SMV_Passives:Cap0805, symbol SMV_Custom:C0805C475K4RACTU
- removed C6: 220 nF, symbol Device:C_Small
- removed C9: 0.33uF,50V, SMV_Passives:Cap0805, symbol SMV_Custom:C0805C334K5RACTU
- removed R10: CRCW080540K0FKEA, SMV_Passives:0805RESC2012X60N, symbol SMV_Custom:CRCW080540K0FKEA
- removed R11, R13, R5: CRCW020149R9FNED, 50Ω, SMV_Passives:0805RESC2012X60N, symbol SMV_Custom:CRCW020149R9FNED
- removed R12, R7: CRCW080520K0FKEAC, SMV_Passives:0805RESC2012X60N, symbol SMV_Custom:CRCW080520K0FKEAC
- removed R14, R17, R9: 10kohms, 0.125W, SMV_Passives:0805RESC2012X60N, symbol SMV_Custom:CRCW080510K0FKEAC
- removed U3, U5, U6: MCP6286T-E/OT, SMV_ICs:SOT-23-5_MC_MCH, symbol SMV_Custom:MCP6286T-E_OT
- added C2: C0805C224K3RACTU, SMV_Passives:Cap0805, symbol SMV_Custom:C0805C224K3RACTU
- added C6: 0.47uF, SMV_Passives:Cap0805, symbol SMV_Custom:C0805C475K4RACTU
- C1: value C0805C106K8RACTU -> 10u
- C11: value 0.1uF,50V -> 0.1u
- C3: value 0.1uF,50V -> 0.1uF
- R6, R8: value 10kohms, 0.125W -> 10k
Connections:
- net DVDD is gone; now on net +3.3V: R6.2
- net VDD_IO is gone; now on net +3.3V: R8.2
- net +12V: now also C6.2
- net +5V: now also RP2.3 (VBUS)
- net CS 0: now also RP2.10 (D5)
- net CS 1: now also RP2.8 (D9)
- net D10: now also RP2.7 (D10), U4.17 (CLKIN)
- net D11: now also RP2.6 (D11)
- net D12: now also RP2.5 (D12); no longer U4.17 (CLKIN)
- net D13: now also RP2.4 (D13)
- net D24: now also R2.1
- net D25: now also R3.1
- net D4: no longer R2.1, R3.1
- net D6: now also RP2.9 (D6)
- net EN: now also RP2.2 (EN)
- net GND: now also TP3.1, U4.5 (AIN1N), C2.2, C6.1; no longer U4.6 (AIN1P)
- net Press_ADC_P: now also U4.6 (AIN1P); no longer U4.5 (AIN1N)
- net SCK: now also TP1.1, U4.14 (SCLK)
- net SCL: now also RP2.11 (SCL); no longer TP1.1, U4.14 (SCLK)
- net SDA: now also RP2.12 (SDA)
- net VBAT: now also RP2.1 (VBAT)
- net at U4.18 (CAP): now also C2.1
- no-connect marks 3 -> 15
Other:
- added sheet Buffers (untitled.kicad_sch)
- note removed: "Am I allowed to put two sensors onto a single ADC? How to read individual sensor data?"
- note removed: "Assume ADC max input voltage is 3.6 V"
- note removed: "Assume max voltage is 12 V"
- note removed: "Assume max voltage is 4.5 V"
- note removed: "Buffers for ADC"
- note removed: "Serial Clock"
- moved on the sheet: C1, C10, C11, C12, C3, C4, D1, J1, J7, J8, R6, R8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
