File: Headlight and Sensors/H&S Board/H&S Board.kicad_sch (KiCad schematic)
At the start: 61 parts, among them J1 430450200, J2 430450200, J3 22035035, J4 Molex Micro-Fit 4 Pin, J5 430450200, J6 430450200, J7 DAQ Board, J8 Driver UI, J9 430450200, Q1 PSMN1R8-40YLC,115, Q2 PSMN1R8-40YLC,115, Q3 PSMN1R8-40YLC,115, U1 ASM330LHHTR, U2 UA78M05QDCYRG4Q1, U4 ADS131M04IPWR

Commit message: darn
Parts:
- R10, R9: value 40k -> 10k; footprint SMV_Passives:0805RESC2012X60N -> SMV_Passives:RES_TNPW0402_VIS
Changed lines of the file:
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@@
 			)
 		)
-		(property "Description" ""
+		(property "Description" "C2286"
 			(at 204.47 67.31 0)
 			(effects
@@
 			)
 		)
-		(property "Datasheet" ""
+		(property "Datasheet" "CRCW080510K0FKEAHP"
 			(at 135.89 24.13 0)
 			(effects
@@
 			)
 		)
-		(property "Description" ""
+		(property "Description" "C313823"
 			(at 135.89 24.13 0)
 			(effects
@@
 			)
 		)
-		(property "Datasheet" "CRCW06031K00FKEA"
+		(property "Datasheet" "CRCW08051K00JNEA"
 			(at 236.22 34.29 0)
 			(effects
@@
 			)
 		)
-		(property "Description" ""
+		(property "Description" "C844604"
 			(at 236.22 34.29 0)
 			(effects
@@
 			)
 		)
-		(property "Description" ""
+		(property "Description" "C459826"
 			(at 208.28 133.35 0)
 			(effects
@@
 			)
 		)
-		(property "Datasheet" ""
+		(property "Datasheet" "CRCW080510K0FKEAHP"
 			(at 46.99 25.4 0)
 			(effects
@@
 			)
 		)
-		(property "Description" ""
+		(property "Description" "C313823"
 			(at 46.99 25.4 0)
 			(effects
@@
 			)
 		)
-		(property "Datasheet" "https://content.kemet.com/datasheets/KEM_C1002_X7R_SMD.pdf"
+		(property "Datasheet" "C0805C106K8RACAUTO"
 			(at 466.7 152.4 0)
 			(effects
@@
 			)
 		)
-		(property "Description" "SMD Comm X7R, Ceramic, 10 uF, 10%, 10 VDC, 25 VDC, 125C, -55C, X7R, SMD, MLCC, Temperature Stable, Class II, 10 % , 10 MOhms, 21 mg, 0805, 2mm, 1.25mm, 1.25mm, 0.75mm, 0.5mm, 2500, 78  Weeks, 80"
+		(property "Description" "C696369"
 			(at 270.51 161.29 0)
 			(effects
@@
 			)
 		)
-		(property "Datasheet" "https://content.kemet.com/datasheets/KEM_C1002_X7R_SMD.pdf"
+		(property "Datasheet" "C0805X474K5RACAUTO"
 			(at 318.11 69.85 0)
 			(effects
@@
 			)
 		)
-		(property "Description" "SMD Comm X7R, Ceramic, 4.7 uF, 10%, 16 VDC, 40 VDC, 125C, -55C, X7R, SMD, MLCC, Temperature Stable, Class II, 10 % , 21.3 MOhms, 21 mg, 0805, 2mm, 1.25mm, 1.25mm, 0.75mm, 0.5mm, 2500, 78  Weeks, 80"
+		(property "Description" "C2173145"
 			(at 121.92 78.74 0)
 			(effects
@@
 			)
 		)
-		(property "Datasheet" "https://content.kemet.com/datasheets/KEM_C1002_X7R_SMD.pdf"
+		(property "Datasheet" "C0805F104K5RACAUTO"
 			(at 61.62 157.48 0)
 			(effects
@@
 			)
 		)
-		(property "Description" "SMD Comm X7R, Ceramic, 0.1 uF, 10%, 50 VDC, 125 VDC, 125C, -55C, X7R, SMD, MLCC, Temperature Stable, Class II, 2.5 % , 5 GOhms, 11 mg, 0805, 2mm, 1.25mm, 0.78mm, 0.75mm, 0.5mm, 4000, 78  Weeks, 80"
+		(property "Description" "C141162"
 			(at 257.81 148.59 0)
 			(effects
@@
 			)
 		)
-		(property "Description" "NEXPERIA - PSMN1R8-40YLC,115 - Power MOSFET, N Channel, 40 V, 100 A, 0.0015 ohm, SOT-669, Surface Mount"
+		(property "Description" "C88071"
 			(at 17.78 35.56 0)
 			(effects
@@
 			)
 		)
-		(property "Datasheet" "https://content.kemet.com/datasheets/KEM_C1002_X7R_SMD.pdf"
+		(property "Datasheet" "C0805C224K5RACAUTO"
 			(at 337.16 107.95 0)
 			(effects
@@
 			)
 		)
-		(property "Description" "SMD Comm X7R, Ceramic, 0.22 uF, 10%, 25 VDC, 62.5 VDC, 125C, -55C, X7R, SMD, MLCC, Temperature Stable, Class II, 3.5 % , 2.2727 GOhms, 11 mg, 0805, 2mm, 1.25mm, 0.78mm, 0.75mm, 0.5mm, 4000, 78  Weeks, 80"
+		(property "Description" "C129652"
 			(at 140.97 116.84 0)
 			(effects
@@
 			)
 		)
-		(property "Description" ""
+		(property "Description" "C2286"
 			(at 175.26 54.61 0)
 			(effects
@@
 			)
 		)
-		(property "Description" "NEXPERIA - PSMN1R8-40YLC,115 - Power MOSFET, N Channel, 40 V, 100 A, 0.0015 ohm, SOT-669, Surface Mount"
+		(property "Description" "C88071"
 			(at 196.85 34.29 0)
 			(effects
@@
 			)
 		)
-		(property "Datasheet" "CRCW06031K00FKEA"
+		(property "Datasheet" "CRCW0805150RFKEA"
 			(at 160.02 54.61 0)
 			(effects
@@
 			)
 		)
-		(property "Description" ""
+		(property "Description" "C844818"
 			(at 160.02 54.61 0)
 			(effects
@@
 			)
 		)
-		(property "Datasheet" "CRCW06031K00FKEA"
+		(property "Datasheet" "CRCW08051K00JNEA"
 			(at 143.51 34.29 0)
 			(effects
@@
 			)
 		)
-		(property "Description" ""
+		(property "Description" "C844604"
 			(at 143.51 34.29 0)
 			(effects
@@
 			)
 		)
-		(property "Datasheet" ""
+		(property "Datasheet" "CRCW080510K0FKEAHP"
 			(at 157.48 142.24 0)
 			(effects
@@
 			)
 		)
-		(property "Description" ""
+		(property "Description" "C313823"
 			(at 157.48 142.24 0)
 			(effects
@@
 			)
 		)
-		(property "Datasheet" "C0805C105K4RACTU"
+		(property "Datasheet" "C0805X105K5RACAUTO"
 			(at 66.04 106.68 0)
 			(effects
@@
 			)
 		)
-		(property "Description" ""
+		(property "Description" "C3858054"
 			(at 66.04 106.68 0)
 			(effects
@@
 			)
 		)
-		(property "Datasheet" "C0805C105K4RACTU"
+		(property "Datasheet" "C0805X105K5RACAUTO"
 			(at 146.05 96.52 0)
 			(effects
@@
 			)
 		)
-		(property "Description" ""
+		(property "Description" "C3858054"
 			(at 146.05 96.52 0)
 			(effects
@@
 			)
 		)
-		(property "Value" "40k"
+		(property "Value" "10k"
 			(at 54.61 152.4 0)
 			(effects
@@
 			)
 		)
-		(property "Footprint" "SMV_Passives:0805RESC2012X60N"
+		(property "Footprint" "SMV_Passives:RES_TNPW0402_VIS"
 			(at 48.26 156.21 0)
 			(effects
@@
 			)
 		)
-		(property "Datasheet" "CRCW080540K0FKEA"
+		(property "Datasheet" "TNPW040210K0BEED"
 			(at 48.26 156.21 0)
 			(effects
@@
 			)
 		)
-		(property "Description" ""
+		(property "Description" "C844452"
 			(at 48.26 156.21 0)
 			(effects
@@
 			)
 		)
-		(property "Datasheet" "CRCW06031K00FKEA"
+		(property "Datasheet" "CRCW08051K00JNEA"
 			(at 55.88 35.56 0)
 			(effects
@@
 			)
 		)
-		(property "Description" ""
+		(property "Description" "C844604"
 			(at 55.88 35.56 0)
 			(effects
@@
 			)
 		)
-		(property "Datasheet" "https://content.kemet.com/datasheets/KEM_C1002_X7R_SMD.pdf"
+		(property "Datasheet" "C0805F104K5RACAUTO"
 			(at -9.5 152.4 0)
 			(effects
@@
 			)
 		)
-		(property "Description" "SMD Comm X7R, Ceramic, 0.1 uF, 10%, 50 VDC, 125 VDC, 125C, -55C, X7R, SMD, MLCC, Temperature Stable, Class II, 2.5 % , 5 GOhms, 11 mg, 0805, 2mm, 1.25mm, 0.78mm, 0.75mm, 0.5mm, 4000, 78  Weeks, 80"
+		(property "Description" "C141162"
 			(at 186.69 143.51 0)
 			(effects
@@
 			)
 		)
-		(property "Datasheet" ""
+		(property "Datasheet" "CRCW080510K0FKEAHP"
 			(at 226.06 24.13 0)
 			(effects
@@
 			)
 		)
-		(property "Description" ""
+		(property "Description" "C313823"
 			(at 226.06 24.13 0)
 			(effects
@@
 			)
 		)
-		(property "Datasheet" "https://content.kemet.com/datasheets/KEM_C1002_X7R_SMD.pdf"
+		(property "Datasheet" "C0805F104K5RACAUTO"
 			(at 255.88 67.31 0)
 			(effects
@@
 			)
 		)
-		(property "Description" "SMD Comm X7R, Ceramic, 0.1 uF, 10%, 50 VDC, 125 VDC, 125C, -55C, X7R, SMD, MLCC, Temperature Stable, Class II, 2.5 % , 5 GOhms, 11 mg, 0805, 2mm, 1.25mm, 0.78mm, 0.75mm, 0.5mm, 4000, 78  Weeks, 80"
+		(property "Description" "C141162"
 			(at 59.69 76.2 0)
 			(effects
@@
 			)
 		)
-		(property "Description" ""
+		(property "Description" "C485570"
 			(at 66.04 63.5 0)
 			(effects
@@
 			)
 		)
-		(property "Value" "40k"
+		(property "Value" "10k"
 			(at 38.1 152.4 0)
 			(effects
@@
 			)
 		)
-		(property "Footprint" "SMV_Passives:0805RESC2012X60N"
+		(property "Footprint" "SMV_Passives:RES_TNPW0402_VIS"
 			(at 31.75 156.21 0)
 			(effects
@@
 			)
 		)
-		(property "Datasheet" "CRCW080540K0FKEA"
+		(property "Datasheet" "TNPW040210K0BEED"
 			(at 31.75 156.21 0)
 			(effects
@@
 			)
 		)
-		(property "Description" ""
+		(property "Description" "C844452"
 			(at 31.75 156.21 0)
 			(effects
@@
 			)
 		)
-		(property "Datasheet" "CRCW06031K00FKEA"
+		(property "Datasheet" "CRCW0805150RFKEA"
 			(at 204.47 54.61 0)
 			(effects
@@
 			)
 		)
-		(property "Description" ""
+		(property "Description" "C844818"
 			(at 204.47 54.61 0)
 			(effects
@@
 			)
 		)
-		(property "Description" "NEXPERIA - PSMN1R8-40YLC,115 - Power MOSFET, N Channel, 40 V, 100 A, 0.0015 ohm, SOT-669, Surface Mount"
+		(property "Description" "C88071"
 			(at 106.68 34.29 0)
 			(effects
@@
 			)
 		)
-		(property "Datasheet" ""
+		(property "Datasheet" "CRCW080510K0FKEAHP"
 			(at 273.05 128.27 0)
 			(effects
@@
 			)
 		)
-		(property "Description" ""
+		(property "Description" "C313823"
 			(at 273.05 128.27 0)
 			(effects

Commit message: f me
Parts:
- added TP1: TestPoint, SMV_Logo:SEM_logo, symbol Connector:TestPoint
- renumbered TP1 to 12V1, TP19 to 12V2, TP20 to 5V1, U1 to Accel1, J8 to CAN1, TP5 to CLKIN1, TP22 to CS0, TP4 to CS1, TP15 to FET1, TP17 to FET2, TP16 to FET3, TP3 to GND1, TP7 to MISO1, TP6 to MOSI1, TP12 to Press_Sig1, TP8 to RST1, TP9 to SCK1, TP14 to Torque_N1, TP13 to Torque_P1
Changed lines of the file:
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@@
 		(on_board yes)
 		(dnp no)
-		(property "Reference" "TP8"
+		(property "Reference" "RST1"
 			(at 166.116 72.39 90)
 			(effects
@@
 			(project "H&S Board"
 				(path "/cdf86217-7949-4457-8f19-2e0a76b22e93"
-					(reference "TP8")
+					(reference "RST1")
 					(unit 1)
 				)
@@
 		(on_board yes)
 		(dnp no)
-		(property "Reference" "TP13"
+		(property "Reference" "Torque_P1"
 			(at 32.512 188.976 0)
 			(effects
@@
 			(project "H&S Board"
 				(path "/cdf86217-7949-4457-8f19-2e0a76b22e93"
-					(reference "TP13")
+					(reference "Torque_P1")
 					(unit 1)
 				)
@@
 		(on_board yes)
 		(dnp no)
-		(property "Reference" "TP16"
+		(property "Reference" "FET3"
 			(at 70.358 28.194 0)
 			(effects
@@
 			(project "H&S Board"
 				(path "/cdf86217-7949-4457-8f19-2e0a76b22e93"
-					(reference "TP16")
+					(reference "FET3")
 					(unit 1)
 				)
@@
 		(on_board yes)
 		(dnp no)
-		(property "Reference" "J8"
+		(property "Reference" "CAN1"
 			(at 247.396 109.474 0)
 			(effects
@@
 			(project "H&S Board"
 				(path "/cdf86217-7949-4457-8f19-2e0a76b22e93"
-					(reference "J8")
+					(reference "CAN1")
 					(unit 1)
 				)
@@
 		(dnp no)
 		(fields_autoplaced yes)
-		(property "Reference" "U1"
+		(property "Reference" "Accel1"
 			(at 231.14 123.19 0)
 			(effects
@@
 			(project ""
 				(path "/cdf86217-7949-4457-8f19-2e0a76b22e93"
-					(reference "U1")
+					(reference "Accel1")
 					(unit 1)
 				)
@@
 		(on_board yes)
 		(dnp no)
-		(property "Reference" "TP19"
+		(property "Reference" "12V2"
 			(at 113.284 58.674 0)
 			(effects
@@
 			(project "H&S Board"
 				(path "/cdf86217-7949-4457-8f19-2e0a76b22e93"
-					(reference "TP19")
+					(reference "12V2")
 					(unit 1)
 				)
@@
 		(on_board yes)
 		(dnp no)
-		(property "Reference" "TP9"
+		(property "Reference" "SCK1"
 			(at 166.116 77.47 90)
 			(effects
@@
 			(project "H&S Board"
 				(path "/cdf86217-7949-4457-8f19-2e0a76b22e93"
-					(reference "TP9")
+					(reference "SCK1")
 					(unit 1)
 				)
@@
 		(on_board yes)
 		(dnp no)
-		(property "Reference" "TP15"
+		(property "Reference" "FET1"
 			(at 157.988 26.924 0)
 			(effects
@@
 			(project "H&S Board"
 				(path "/cdf86217-7949-4457-8f19-2e0a76b22e93"
-					(reference "TP15")
+					(reference "FET1")
 					(unit 1)
 				)
@@
 	(symbol
 		(lib_id "Connector:TestPoint")
+		(at 77.47 149.86 0)
+		(unit 1)
+		(exclude_from_sim no)
+		(in_bom yes)
+		(on_board yes)
+		(dnp no)
+		(fields_autoplaced yes)
+		(property "Reference" "TP1"
+			(at 80.01 145.2879 0)
+			(effects
+				(font
+					(size 1.27 1.27)
+				)
+				(justify left)
+			)
+		)
+		(property "Value" "TestPoint"
+			(at 80.01 147.8279 0)
+			(effects
+				(font
+					(size 1.27 1.27)
+				)
+				(justify left)
+			)
+		)
+		(property "Footprint" "SMV_Logo:SEM_logo"
+			(at 82.55 149.86 0)
+			(effects
+				(font
+					(size 1.27 1.27)
+				)
+				(hide yes)
+			)
+		)
+		(property "Datasheet" "~"
+			(at 82.55 149.86 0)
+			(effects
+				(font
+					(size 1.27 1.27)
+				)
+				(hide yes)
+			)
+		)
+		(property "Description" "test point"
+			(at 77.47 149.86 0)
+			(effects
+				(font
+					(size 1.27 1.27)
+				)
+				(hide yes)
+			)
+		)
+		(pin "1"
+		)
+		(instances
+			(project ""
+				(path "/cdf86217-7949-4457-8f19-2e0a76b22e93"
+					(reference "TP1")
+					(unit 1)
+				)
+			)
+		)
+	)
+	(symbol
+		(lib_id "Connector:TestPoint")
 		(at 180.34 64.77 90)
 		(unit 1)
@@
 		(on_board yes)
 		(dnp no)
-		(property "Reference" "TP6"
+		(property "Reference" "MOSI1"
 			(at 166.116 64.77 90)
 			(effects
@@
 			(project "H&S Board"
 				(path "/cdf86217-7949-4457-8f19-2e0a76b22e93"
-					(reference "TP6")
+					(reference "MOSI1")
 					(unit 1)
 				)
@@
 		(on_board yes)
 		(dnp no)
-		(property "Reference" "TP20"
+		(property "Reference" "5V1"
 			(at 115.824 169.164 0)
 			(effects
@@
 			(project "H&S Board"
 				(path "/cdf86217-7949-4457-8f19-2e0a76b22e93"
-					(reference "TP20")
+					(reference "5V1")
 					(unit 1)
 				)
@@
 		(on_board yes)
 		(dnp no)
-		(property "Reference" "TP3"
+		(property "Reference" "GND1"
 			(at 65.786 120.65 0)
 			(effects
@@
 			(project "H&S Board"
 				(path "/cdf86217-7949-4457-8f19-2e0a76b22e93"
-					(reference "TP3")
+					(reference "GND1")
 					(unit 1)
 				)
@@
 		(on_board yes)
 		(dnp no)
-		(property "Reference" "TP14"
+		(property "Reference" "Torque_N1"
 			(at 28.194 171.196 0)
 			(effects
@@
 			(project "H&S Board"
 				(path "/cdf86217-7949-4457-8f19-2e0a76b22e93"
-					(reference "TP14")
+					(reference "Torque_N1")
 					(unit 1)
 				)
@@
 		(on_board yes)
 		(dnp no)
-		(property "Reference" "TP17"
+		(property "Reference" "FET2"
 			(at 249.428 26.924 0)
 			(effects
@@
 			(project "H&S Board"
 				(path "/cdf86217-7949-4457-8f19-2e0a76b22e93"
-					(reference "TP17")
+					(reference "FET2")
 					(unit 1)
 				)
@@
 		(on_board yes)
 		(dnp no)
-		(property "Reference" "TP7"
+		(property "Reference" "MISO1"
 			(at 166.116 67.31 90)
 			(effects
@@
 			(project "H&S Board"
 				(path "/cdf86217-7949-4457-8f19-2e0a76b22e93"
-					(reference "TP7")
+					(reference "MISO1")
 					(unit 1)
 				)
@@
 		(on_board yes)
 		(dnp no)
-		(property "Reference" "TP12"
+		(property "Reference" "Press_Sig1"
 			(at 108.712 188.976 0)
 			(effects
@@
 			(project "H&S Board"
 				(path "/cdf86217-7949-4457-8f19-2e0a76b22e93"
-					(reference "TP12")
+					(reference "Press_Sig1")
 					(unit 1)
 				)
@@
 			)
 		)
-		(property "Description" "Micro-Fit 3.0 Vertical Header, 3.00mm Pitch, Dual Row,  Circuits, with PCB Polarizing Peg, Tin, Glow-Wire Capable, Black"
+		(property "Description" ""
 			(at 41.91 179.07 0)
 			(effects
@@
 		(on_board yes)
 		(dnp no)
-		(property "Reference" "TP1"
+		(property "Reference" "12V1"
 			(at 90.678 32.258 0)
 			(effects
@@
 			(project "H&S Board"
 				(path "/cdf86217-7949-4457-8f19-2e0a76b22e93"
-					(reference "TP1")
+					(reference "12V1")
 					(unit 1)
 				)
@@
 		(on_board yes)
 		(dnp no)
-		(property "Reference" "TP5"
+		(property "Reference" "CLKIN1"
 			(at 166.116 62.23 90)
 			(effects
@@
 			(project "H&S Board"
 				(path "/cdf86217-7949-4457-8f19-2e0a76b22e93"
-					(reference "TP5")
+					(reference "CLKIN1")
 					(unit 1)
 				)
@@
 		(on_board yes)
 		(dnp no)
-		(property "Reference" "TP22"
+		(property "Reference" "CS0"
 			(at 261.874 131.064 0)
 			(effects
@@
 			(project "H&S Board"
 				(path "/cdf86217-7949-4457-8f19-2e0a76b22e93"
-					(reference "TP22")
+					(reference "CS0")
 					(unit 1)
 				)
@@
 		(on_board yes)
 		(dnp no)
-		(property "Reference" "TP4"
+		(property "Reference" "CS1"
 			(at 145.288 139.446 0)
 			(effects
@@
 			(project "H&S Board"
 				(path "/cdf86217-7949-4457-8f19-2e0a76b22e93"
-					(reference "TP4")
+					(reference "CS1")
 					(unit 1)
 				)
