File: Headlight and Sensors/H&S Board/H&S Board.kicad_pcb (KiCad board)
At the start: 2 copper layers, 78 parts, among them J1 430450200, J2 430450200, J3 22035035, J4 Molex Micro-Fit 4 Pin, J5 430450200, J6 430450200, J7 DAQ Board, J8 Driver UI, J9 430450200, Q1 PSMN1R8-40YLC,115, Q2 PSMN1R8-40YLC,115, Q3 PSMN1R8-40YLC,115, U1 ASM330LHHTR, U2 UA78M05QDCYRG4Q1, U4 ADS131M04IPWR, U7 MCP6286T-E/OT, U8 MCP6286T-E/OT, U9 MCP6286T-E/OT

Commit message: basically done
Parts:
- moved TP10 51.9 mm to (179.3, 151.9)
- moved TP11 44.4 mm to (179.3, 146.9)
- moved TP22 17.6 mm to (117.4, 135.8)
- moved TP4 17.2 mm to (115.2, 118.8)
- moved C13 1.10 mm to (101.7, 115.1)
- moved R19 1.10 mm to (99.0, 115.2)
- moved R15 0.48 mm to (154.2, 138.6)
- moved R16 0.48 mm to (152.0, 138.6)
Connections:
- R8 pad 1: /CS 1 -> /CS 0
- RP2 pad 16: /MISO -> unconnected-(RP2-MISO-Pad16)
- RP2 pad 17: /MOSI -> unconnected-(RP2-MOSI-Pad17)
- RP2 pad 4: /CS 1 -> /CS 0
- TP22 pad 1: /CS 1 -> /CS 0
- U1 pad 12: /CS 1 -> /CS 0
Routing:
- net /CS 0: track 0.00 -> 38.1 mm
- net /CS 1: track 55.5 -> 17.4 mm
- net GND: track 5.42 -> 21.8 mm, vias 3 -> 100
- net /MISO: track 16.8 -> 31.9 mm, vias 0 -> 1
- net /MOSI: track 23.2 -> 35.9 mm, vias 0 -> 1
- net /CAN_N: track 112.4 -> 118.3 mm
- net /CAN_P: track 112.3 -> 118.2 mm
- net +3.3V: track 94.2 -> 97.7 mm
- net Net-(U8-VIN-): track 5.68 -> 6.78 mm
- net /Torque_ADC_P: track 7.17 -> 6.07 mm

Commit message: Finished!
Parts:
- removed TP18, TP2, TP21: TestPoint, TestPoint:TestPoint_Pad_D1.0mm
- added H1: MountingHole, MountingHole:MountingHole_3.2mm_M3, F.Cu at (76.4, 87.6)
- added H2: MountingHole, MountingHole:MountingHole_3.2mm_M3, F.Cu at (177.8, 87.6)
- added H3: MountingHole, MountingHole:MountingHole_3.2mm_M3, F.Cu at (76.4, 151.9)
- added H4: MountingHole, MountingHole:MountingHole_3.2mm_M3, F.Cu at (176.9, 151.9)
- added REF**: SEM_logo, SMV_Logo:SEM_logo, F.Cu at (96.0, 142.8)
- moved GND 37.1 mm to (77.0, 142.2)
- moved J7 31.1 mm to (109.3, 146.8)
- moved TP10 16.0 mm to (163.3, 151.9)
- moved TP11 16.0 mm to (163.3, 146.9)
- moved CAN 16.0 mm to (157.5, 146.8)
- moved J1 5.94 mm to (172.2, 95.4)
- moved J9 5.26 mm to (82.0, 95.4)
- moved 5V 2.69 mm to (88.1, 99.6)
- renumbered TP1 to 12V, TP20 to 5V, U1 to Accel, J8 to CAN, TP5 to CLKIN, TP22 to CS0, TP4 to CS1, TP15 to FET1, TP17 to FET2, TP16 to FET3, TP3 to GND, TP7 to MISO, TP6 to MOSI, TP12 to P_sense, TP8 to Reset, TP9 to SCK
Routing:
- net /CAN_P: track 118.2 -> 71.9 mm
- net /CAN_N: track 118.3 -> 71.9 mm
- net GND: track 21.8 -> 20.8 mm, vias 100 -> 85
- net +5V: track 87.1 -> 86.3 mm
Other:
- board outline added: 109.8 x 74 mm
- board text added: "CAN"
- board text added: "Light #1"
- board text added: "Light #2"
- board text added: "Light #3"
- board text added: "Power"
- board text removed: "Accelerometer"
- board text removed: "LDO"
- board text removed: "Left Connector"
- board text removed: "MOSFET #1"
- board text removed: "MOSFET #2"
- board text removed: "MOSFET #3"
- board text removed: "Right Connector"

Commit message: Finished!
Other:
- board text added: "Benjamin Li 1/27/25 Lights and Sensors Board"
Changed lines of the file:
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@@
 		(fp_arc
 			(start -8.304556 8.25436)
-			(mid -8.304689 8.247611)
+			(mid -8.304689 8.247612)
 			(end -8.300511 8.24231)
 			(stroke
@@
 		(fp_arc
 			(start -7.774364 12.655021)
-			(mid -7.771131 12.665267)
+			(mid -7.771131 12.665266)
 			(end -7.776942 12.674303)
 			(stroke
@@
 		(fp_arc
 			(start -4.883602 11.697921)
-			(mid -4.883173 11.693202)
+			(mid -4.883173 11.693201)
 			(end -4.878724 11.69157)
 			(stroke
@@
 		(fp_arc
 			(start -3.156379 11.616037)
-			(mid -3.16113 11.513181)
+			(mid -3.161129 11.513181)
 			(end -3.16328 11.410238)
 			(stroke
@@
 		(fp_arc
 			(start -0.45284 6.767971)
-			(mid -0.453954 6.770747)
+			(mid -0.453954 6.770748)
 			(end -0.456677 6.771986)
 			(stroke
@@
 		(layer "F.SilkS")
 		(effects
+			(font
+				(size 1.5 1.5)
+				(thickness 0.3)
+				(bold yes)
+			)
+			(justify left bottom)
+		)
+	)
+	(gr_text "Benjamin Li\n1/27/25\nLights and Sensors Board\n"
+		(at 87.5 91.5 0)
+		(layer "F.SilkS")
+		(effects
