File: Headlight and Sensors/H&S Board/H&S Board.kicad_pcb (KiCad board)
At the start: 2 copper layers, 109.8 x 74 mm, 80 parts, among them J1 430450200, J2 430450200, J3 22035035, J4 Molex Micro-Fit 4 Pin, J5 430450200, J6 430450200, J7 DAQ Board, J9 430450200, Q1 PSMN1R8-40YLC,115, Q2 PSMN1R8-40YLC,115, Q3 PSMN1R8-40YLC,115, U2 UA78M05QDCYRG4Q1, U4 ADS131M04IPWR, U7 MCP6286T-E/OT, U8 MCP6286T-E/OT, U9 MCP6286T-E/OT

Commit message: Finalized!
Routing:
- net Net-(Q2-D_1): track 5.34 -> 2.35 mm
- net GND: vias 85 -> 86
Changed lines of the file:
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@@
 		(fp_arc
 			(start -8.304556 8.25436)
-			(mid -8.304689 8.247611)
+			(mid -8.304689 8.247612)
 			(end -8.300511 8.24231)
 			(stroke
@@
 		(fp_arc
 			(start -7.774364 12.655021)
-			(mid -7.771131 12.665267)
+			(mid -7.771131 12.665266)
 			(end -7.776942 12.674303)
 			(stroke
@@
 		(fp_arc
 			(start -4.883602 11.697921)
-			(mid -4.883173 11.693202)
+			(mid -4.883173 11.693201)
 			(end -4.878724 11.69157)
 			(stroke
@@
 		(fp_arc
 			(start -3.156379 11.616037)
-			(mid -3.16113 11.513181)
+			(mid -3.161129 11.513181)
 			(end -3.16328 11.410238)
 			(stroke
@@
 		(fp_arc
 			(start -0.45284 6.767971)
-			(mid -0.453954 6.770747)
+			(mid -0.453954 6.770748)
 			(end -0.456677 6.771986)
 			(stroke
@@
 	(gr_poly
 		(pts
+			(xy 163.25 135.36) (xy 166.49 135.36) (xy 166.49 140.03) (xy 163.25 140.03)
+		)
+		(stroke
+			(width 0)
+			(type solid)
+		)
+		(fill solid)
+		(layer "F.Cu")
+		(net 15)
+	)
+	(gr_poly
+		(pts
+			(xy 163.16 113.63) (xy 166.4 113.63) (xy 166.4 118.3) (xy 163.16 118.3)
+		)
+		(stroke
+			(width 0)
+			(type solid)
+		)
+		(fill solid)
+		(layer "F.Cu")
+		(net 11)
+	)
+	(gr_poly
+		(pts
+			(xy 163.25 124.56) (xy 166.49 124.56) (xy 166.49 129.23) (xy 163.25 129.23)
+		)
+		(stroke
+			(width 0)
+			(type solid)
+		)
+		(fill solid)
+		(layer "F.Cu")
+		(net 16)
+	)
+	(gr_line
+		(start 157.59 118.05)
+		(end 157.59 118.15)
+		(stroke
+			(width 0.2)
+			(type default)
+		)
+		(layer "F.Cu")
+		(net 18)
+	)
+	(gr_poly
+		(pts
+			(xy 153.85 123.88) (xy 157.69 123.88) (xy 157.69 127.28) (xy 153.85 127.28)
+		)
+		(stroke
+			(width 0)
+			(type solid)
+		)
+		(fill solid)
+		(layer "F.Cu")
+		(net 1)
+	)
+	(gr_poly
+		(pts
 			(xy 106.9 113) (xy 103.8 113) (xy 103.8 114.6) (xy 106.9 114.6)
 		)
@@
 		(net 1)
 	)
+	(gr_poly
+		(pts
+			(xy 153.86 113.72) (xy 157.7 113.72) (xy 157.7 116.42) (xy 153.86 116.42)
+		)
+		(stroke
+			(width 0)
+			(type solid)
+		)
+		(fill solid)
+		(layer "F.Cu")
+		(net 1)
+	)
+	(gr_poly
+		(pts
+			(xy 153.54 134.8) (xy 157.69 134.8) (xy 157.69 138.09) (xy 153.54 138.09)
+		)
+		(stroke
+			(width 0)
+			(type solid)
+		)
+		(fill solid)
+		(layer "F.Cu")
+		(net 1)
+	)
 	(gr_line
 		(start 182 83.4)
@@
 	)
 	(via
-		(at 84.475 142.1)
+		(at 85.77 142.51)
 		(size 0.6)
 		(drill 0.3)
@@
 	)
 	(via
+		(at 132.03 146.19)
+		(size 0.6)
+		(drill 0.3)
+		(layers "F.Cu" "B.Cu")
+		(free yes)
+		(net 1)
+	)
+	(via
 		(at 149.6 144.4)
 		(size 0.6)
@@
 		(width 0.2)
 		(layer "F.Cu")
-		(net 11)
-	)
-	(segment
-		(start 162.599 115.9666)
-		(end 165.592899 115.9666)
-		(width 0.2)
-		(layer "F.Cu")

Commit message: darn
Parts:
- C13, C14, C9: footprint SMV_Passives:Cap0805 -> SMV_Passives:CAPC17595_87N_KEM
- R10, R9: value 40k -> 10k; footprint SMV_Passives:0805RESC2012X60N -> SMV_Passives:RES_TNPW0402_VIS
- R18, R19, R20: value CRCW020149R9FNED, 50Ω -> 50 Ohms
- R21: footprint SMV_Passives:0805RESC2012X60N -> SMV_Passives:RES_TNPW0402_VIS
- R22: footprint SMV_Passives:0805RESC2012X60N -> SMV_Passives:RES_CRCW_0402
- R23: value 40Kohms -> 47Kohms; footprint SMV_Passives:0805RESC2012X60N -> SMV_Passives:0603_resistors
- R24, R7: value 10kohms, 0.125W -> 12.1kohms, 0.125W; footprint SMV_Passives:0805RESC2012X60N -> SMV_Passives:0603_resistors
- R25: value 40kohms -> 47kohms; footprint SMV_Passives:0805RESC2012X60N -> SMV_Passives:0603_resistors
- renumbered CAN to J8, 12V to TP1, P_sense to TP12, FET1 to TP15, FET3 to TP16, FET2 to TP17, 5V to TP20, CS0 to TP22, GND to TP3, CS1 to TP4, CLKIN to TP5, MOSI to TP6, MISO to TP7, Reset to TP8, SCK to TP9, Accel to U1
Routing:
- net Net-(U7-VIN+): track 4.67 -> 5.38 mm

Commit message: f me
Parts:
- removed REF**: SEM_logo, SMV_Logo:SEM_logo
- added TP1: TestPoint, SMV_Logo:SEM_logo, F.Cu at (96.2, 142.8)
- renumbered TP1 to 12V1, TP19 to 12V2, TP20 to 5V1, U1 to Accel1, J8 to CAN1, TP5 to CLKIN1, TP22 to CS0, TP4 to CS1, TP15 to FET1, TP17 to FET2, TP16 to FET3, TP3 to GND1, TP7 to MISO1, TP6 to MOSI1, TP12 to Press_Sig1, TP8 to RST1, TP9 to SCK1, TP14 to Torque_N1, TP13 to Torque_P1

Commit message: ldo fixed
Parts:
- moved U2 5.12 mm to (154.0, 108.1), turned to 180 degrees
- moved C6 2.02 mm to (159.4, 106.0)
- moved 12V2 2.02 mm to (159.5, 102.6)
- moved C12 1.30 mm to (148.7, 106.1)
Connections:
- U2 pad 1: +5V -> +12V
- U2 pad 3: +12V -> +5V
Routing:
- net +12V: track 22.7 -> 21.4 mm
- net +5V: track 86.3 -> 87.1 mm
- net GND: vias 86 -> 83
