File: Headlight and Sensors/H&S Board/untitled.kicad_sch (KiCad schematic)
At the start: 18 parts, among them U7 MCP6286T-E/OT, U8 MCP6286T-E/OT, U9 MCP6286T-E/OT

Commit message: darn
Parts:
- C13, C14, C9: footprint SMV_Passives:Cap0805 -> SMV_Passives:CAPC17595_87N_KEM
- R18, R19, R20: value CRCW020149R9FNED, 50Ω -> 50 Ohms
- R21: footprint SMV_Passives:0805RESC2012X60N -> SMV_Passives:RES_TNPW0402_VIS
- R22: footprint SMV_Passives:0805RESC2012X60N -> SMV_Passives:RES_CRCW_0402
- R23: value 40Kohms -> 47Kohms; footprint SMV_Passives:0805RESC2012X60N -> SMV_Passives:0603_resistors
- R24, R7: value 10kohms, 0.125W -> 12.1kohms, 0.125W; footprint SMV_Passives:0805RESC2012X60N -> SMV_Passives:0603_resistors
- R25: value 40kohms -> 47kohms; footprint SMV_Passives:0805RESC2012X60N -> SMV_Passives:0603_resistors
Changed lines of the file:
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@@
 			)
 		)
-		(property "Datasheet" "https://content.kemet.com/datasheets/KEM_C1002_X7R_SMD.pdf"
+		(property "Datasheet" "C0805F104K5RACAUTO"
 			(at 338.43 36.83 0)
 			(effects
@@
 			)
 		)
-		(property "Description" "SMD Comm X7R, Ceramic, 4.7 uF, 10%, 16 VDC, 40 VDC, 125C, -55C, X7R, SMD, MLCC, Temperature Stable, Class II, 10 % , 21.3 MOhms, 21 mg, 0805, 2mm, 1.25mm, 1.25mm, 0.75mm, 0.5mm, 2500, 78  Weeks, 80"
+		(property "Description" "C141162"
 			(at 142.24 45.72 0)
 			(effects
@@
 			)
 		)
-		(property "Description" ""
+		(property "Description" "C623478"
 			(at 74.93 102.87 0)
 			(effects
@@
 			)
 		)
-		(property "Footprint" "SMV_Passives:Cap0805"
+		(property "Footprint" "SMV_Passives:CAPC17595_87N_KEM"
 			(at 145.72 106.68 0)
 			(effects
@@
 			)
 		)
-		(property "Datasheet" "https://content.kemet.com/datasheets/KEM_C1002_X7R_SMD.pdf"
+		(property "Datasheet" "C0603C472K5RACAUTO"
 			(at 245.72 106.68 0)
 			(effects
@@
 			)
 		)
-		(property "Description" "SMD Comm X7R, Ceramic, 4.7 uF, 10%, 16 VDC, 40 VDC, 125C, -55C, X7R, SMD, MLCC, Temperature Stable, Class II, 10 % , 21.3 MOhms, 21 mg, 0805, 2mm, 1.25mm, 1.25mm, 0.75mm, 0.5mm, 2500, 78  Weeks, 80"
+		(property "Description" "C141106"
 			(at 49.53 115.57 0)
 			(effects
@@
 			)
 		)
-		(property "Description" ""
+		(property "Description" "C623478"
 			(at 69.85 163.83 0)
 			(effects
@@
 			)
 		)
-		(property "Footprint" "SMV_Passives:0805RESC2012X60N"
+		(property "Footprint" "SMV_Passives:RES_CRCW_0402"
 			(at 156.21 118.11 0)
 			(effects
@@
 			)
 		)
-		(property "Datasheet" ""
+		(property "Datasheet" "TNPW040210K0BEED"
 			(at 156.21 118.11 0)
 			(effects
@@
 			)
 		)
-		(property "Description" ""
+		(property "Description" "C844452"
 			(at 156.21 118.11 0)
 			(effects
@@
 			)
 		)
-		(property "Value" "40Kohms"
+		(property "Value" "47Kohms"
 			(at 154.94 160.0199 90)
 			(effects
@@
 			)
 		)
-		(property "Footprint" "SMV_Passives:0805RESC2012X60N"
+		(property "Footprint" "SMV_Passives:0603_resistors"
 			(at 151.13 158.75 0)
 			(effects
@@
 			)
 		)
-		(property "Datasheet" ""
+		(property "Datasheet" "TNPW060347K0BEEA"
 			(at 151.13 158.75 0)
 			(effects
@@
 			)
 		)
-		(property "Description" ""
+		(property "Description" "C2089026"
 			(at 151.13 158.75 0)
 			(effects
@@
 			)
 		)
-		(property "Footprint" "SMV_Passives:Cap0805"
+		(property "Footprint" "SMV_Passives:CAPC17595_87N_KEM"
 			(at 141.91 167.64 0)
 			(effects
@@
 			)
 		)
-		(property "Datasheet" "https://content.kemet.com/datasheets/KEM_C1002_X7R_SMD.pdf"
+		(property "Datasheet" "C0603C472K5RACAUTO"
 			(at 241.91 167.64 0)
 			(effects
@@
 			)
 		)
-		(property "Description" "SMD Comm X7R, Ceramic, 4.7 uF, 10%, 16 VDC, 40 VDC, 125C, -55C, X7R, SMD, MLCC, Temperature Stable, Class II, 10 % , 21.3 MOhms, 21 mg, 0805, 2mm, 1.25mm, 1.25mm, 0.75mm, 0.5mm, 2500, 78  Weeks, 80"
+		(property "Description" "C141106"
 			(at 45.72 176.53 0)
 			(effects
@@
 			)
 		)
-		(property "Value" "CRCW020149R9FNED, 50Ω"
+		(property "Value" "50 Ohms"
 			(at 57.15 99.06 0)
 			(effects
@@
 			)
 		)
-		(property "Datasheet" "CRCW020149R9FNED"
+		(property "Datasheet" "CRCW080549R9FKEA"
 			(at 44.958 111.506 0)
 			(effects
@@
 			)
 		)
-		(property "Description" ""
+		(property "Description" "C844847"
 			(at 50.8 102.87 0)
 			(effects
@@
 			)
 		)
-		(property "Datasheet" "https://content.kemet.com/datasheets/KEM_C1002_X7R_SMD.pdf"
+		(property "Datasheet" "C0805F104K5RACAUTO"
 			(at 328.27 154.94 0)
 			(effects
@@
 			)
 		)
-		(property "Description" "SMD Comm X7R, Ceramic, 4.7 uF, 10%, 16 VDC, 40 VDC, 125C, -55C, X7R, SMD, MLCC, Temperature Stable, Class II, 10 % , 21.3 MOhms, 21 mg, 0805, 2mm, 1.25mm, 1.25mm, 0.75mm, 0.5mm, 2500, 78  Weeks, 80"
+		(property "Description" "C141162"
 			(at 132.08 163.83 0)
 			(effects
@@
 			)
 		)
-		(property "Value" "CRCW020149R9FNED, 50Ω"
+		(property "Value" "50 Ohms"
 			(at 53.34 160.02 0)
 			(effects
@@
 			)
 		)
-		(property "Datasheet" "CRCW020149R9FNED"
+		(property "Datasheet" "CRCW080549R9FKEA"
 			(at 41.148 172.466 0)
 			(effects
@@
 			)
 		)
-		(property "Description" ""
+		(property "Description" "C844847"
 			(at 46.99 163.83 0)
 			(effects
@@
 			)
 		)
-		(property "Value" "10kohms, 0.125W"
+		(property "Value" "12.1kohms, 0.125W"
 			(at 167.64 63.4999 90)
 			(effects
@@
 			)
 		)
-		(property "Footprint" "SMV_Passives:0805RESC2012X60N"
+		(property "Footprint" "SMV_Passives:0603_resistors"
 			(at 162.56 62.23 0)
 			(effects
@@
 			)
 		)
-		(property "Datasheet" ""
+		(property "Datasheet" "TNPW060312K1BEEA"
 			(at 162.56 62.23 0)
 			(effects
@@
 			)
 		)
-		(property "Description" ""
+		(property "Description" "C2075023"
 			(at 162.56 62.23 0)
 			(effects
@@
 			)
 		)
-		(property "Value" "CRCW020149R9FNED, 50Ω"
+		(property "Value" "50 Ohms"
 			(at 72.39 41.91 0)
 			(effects
@@
 			)
 		)
-		(property "Datasheet" "CRCW020149R9FNED"
+		(property "Datasheet" "CRCW080549R9FKEA"
 			(at 60.198 54.356 0)
 			(effects
@@
 			)
 		)
-		(property "Description" ""
+		(property "Description" "C844847"
 			(at 66.04 45.72 0)
 			(effects
@@
 			)
 		)
-		(property "Value" "40kohms"
+		(property "Value" "47kohms"
 			(at 166.37 41.9099 90)
 			(effects
@@
 			)
 		)
-		(property "Footprint" "SMV_Passives:0805RESC2012X60N"
+		(property "Footprint" "SMV_Passives:0603_resistors"
 			(at 162.56 40.64 0)
 			(effects
@@
 			)
 		)
-		(property "Datasheet" ""
+		(property "Datasheet" "TNPW060347K0BEEA"
 			(at 162.56 40.64 0)
 			(effects
@@
 			)
 		)
-		(property "Description" ""
+		(property "Description" "C2089026"
 			(at 162.56 40.64 0)
 			(effects
@@
 			)
 		)
-		(property "Value" "10kohms, 0.125W"
+		(property "Value" "12.1kohms, 0.125W"
 			(at 156.21 180.3399 90)
 			(effects
@@
 			)
 		)
-		(property "Footprint" "SMV_Passives:0805RESC2012X60N"
+		(property "Footprint" "SMV_Passives:0603_resistors"
 			(at 151.13 179.07 0)
 			(effects
@@
 			)
 		)
-		(property "Datasheet" ""
+		(property "Datasheet" "TNPW060312K1BEEA"
 			(at 151.13 179.07 0)
 			(effects
@@
 			)
 		)
-		(property "Description" ""
+		(property "Description" "C2075023"
 			(at 151.13 179.07 0)
 			(effects
@@
 			)
 		)
-		(property "Description" ""
+		(property "Description" "C623478"
 			(at 81.28 45.72 0)
 			(effects
@@
 			)
 		)
-		(property "Footprint" "SMV_Passives:0805RESC2012X60N"
+		(property "Footprint" "SMV_Passives:RES_TNPW0402_VIS"
 			(at 156.21 97.79 0)
 			(effects
@@
 			)
 		)
-		(property "Datasheet" ""
+		(property "Datasheet" "TNPW040210K0BEED"
 			(at 156.21 97.79 0)
 			(effects
@@
 			)
 		)
-		(property "Description" ""
+		(property "Description" "C844452"
 			(at 156.21 97.79 0)
 			(effects
@@
 			)
 		)
-		(property "Datasheet" "https://content.kemet.com/datasheets/KEM_C1002_X7R_SMD.pdf"
+		(property "Datasheet" "C0805F104K5RACAUTO"
 			(at 332.08 93.98 0)
 			(effects
@@
 			)
 		)
-		(property "Description" "SMD Comm X7R, Ceramic, 4.7 uF, 10%, 16 VDC, 40 VDC, 125C, -55C, X7R, SMD, MLCC, Temperature Stable, Class II, 10 % , 21.3 MOhms, 21 mg, 0805, 2mm, 1.25mm, 1.25mm, 0.75mm, 0.5mm, 2500, 78  Weeks, 80"
+		(property "Description" "C141162"
 			(at 135.89 102.87 0)
 			(effects
@@
 			)
 		)
-		(property "Footprint" "SMV_Passives:Cap0805"
+		(property "Footprint" "SMV_Passives:CAPC17595_87N_KEM"
 			(at 162.23 49.53 0)
 			(effects
@@
 			)
 		)
-		(property "Datasheet" "https://content.kemet.com/datasheets/KEM_C1002_X7R_SMD.pdf"
+		(property "Datasheet" "C0603C472K5RACAUTO"
 			(at 262.23 49.53 0)
 			(effects
@@
 			)
 		)
-		(property "Description" "SMD Comm X7R, Ceramic, 4.7 uF, 10%, 16 VDC, 40 VDC, 125C, -55C, X7R, SMD, MLCC, Temperature Stable, Class II, 10 % , 21.3 MOhms, 21 mg, 0805, 2mm, 1.25mm, 1.25mm, 0.75mm, 0.5mm, 2500, 78  Weeks, 80"
+		(property "Description" "C141106"
 			(at 66.04 58.42 0)
 			(effects
