File: Joulemeter/joulemeter.kicad_sch (KiCad schematic)
At the start: 10 parts, among them J1 XT60-M, J2 XT60-M, J3 22035035, U2 INA240A1PW, U5 PADS131M04QPWRQ1

Commit message: added more connections to things
Parts:
- added C1, C2: 1μF, symbol Device:C
- added C3: 220nF, symbol Device:C
Connections:
- net 3V3: now also U2.6 (REF2), C1.1, C2.1
- net GND: now also U2.7 (REF1), U5.19 (DGND), U5.2 (AGND), U5.5 (AIN1N), C1.2, C2.2, C3.2
- net CSENSE_OUT: now reaches U2.8
- net CSENSE_OUT: now also U5.6 (AIN1P)
- net DATA: now reaches RP2.10
- net DATA: now also U5.15 (DOUT)
- net SERIALCLOCK: now reaches RP2.12
- net SERIALCLOCK: now also U5.14 (SCLK)
- net RESET: now reaches RP2.7
- net RESET: now also U5.11 (SYNC/RESET)
- net CLCKIN: now reaches RP2.8
- net CLCKIN: now also U5.17 (CLKIN)
- net CHIPSELECT: now reaches RP2.9
- net CHIPSELECT: now also U5.12 (CS)
- net at U5.18 (CAP): now also C3.1
- no-connect marks 0 -> 26
Other:
- moved on the sheet: R1, R2, U5

Commit message: schematic feedback
Parts:
- removed R_shunt: R_US, symbol Device:R_US
- removed U2: INA240A1PW, Package_SO:TSSOP-8_4.4x3mm_P0.65mm, symbol Amplifier_Current:INA240A1PW
- added C1206C103JBGACAUTO7210: 10nF, symbol Device:C
- added C1210C105K1RACAUTO: 1μF, symbol Device:C
- added C1210C106K3RACAUTO: 10μF, symbol Device:C
- added CRCW060310K0FKEA (x2): 10k ohms, symbol Device:R_US
- added IC1: INA240A3PWR, SOP65P640X120-8N, symbol INA240A3PWR:INA240A3PWR
- added PSR400ITQFF0L50: 0.0005ohm, symbol Device:R_Shunt_US
- added TP_3V3, TP_48V, TP_5V, TP_CLK, TP_CS, TP_CSENSE_OUT, TP_GND, TP_MISO, TP_MOSI, TP_SHUNT_IN, TP_SHUNT_OUT: ~, symbol Connector:TestPoint
- added U1: OPA333AIDCKRG4, Package_TO_SOT_SMD:SOT-353_SC-70-5, symbol Amplifier_Operational:OPA333xxDCK
- TNPW080510K0BEEA: renamed from R2; value R_US -> 10k ohms
- TNPW1206249KBEEA: renamed from R1; value R_US -> 249k ohms
- renumbered C3 to C0603C224K5RACTU, C2 to C1210C105K1RACAUTO
Connections:
- net CLCKIN is gone; now on net CLKOUT: RP2.8, U5.17 (CLKIN)
- net DATA is gone; now on net MISO: RP2.10, U5.15 (DOUT)
- net SERIALCLOCK is gone; now on net CLK: RP2.12, U5.14 (SCLK)
- net +48V: now also LDO1.6 (VIN), C1210C105K1RACAUTO.1, PSR400ITQFF0L50.1, PSR400ITQFF0L50.4, TP_48V.1, TP_SHUNT_IN.1, TP_SHUNT_OUT.1
- net +5V: now also C1210C106K3RACAUTO.1, TP_5V.1
- net CSENSE_OUT: now also IC1.8 (OUT), TP_CSENSE_OUT.1
- net GND: now also C1.1, LDO1.4 (GND), C1206C103JBGACAUTO7210.2, C1210C105K1RACAUTO.2, C1210C106K3RACAUTO.2, IC1.4 (GND), IC1.7 (REF1), TP_GND.1, U1.2 (V-); no longer C0603C224K5RACTU.2, C1.2, U5.19 (DGND), U5.2 (AGND)
- net MISO: now reaches RP2.10
- net MISO: now also TP_MISO.1
- net MOSI: now reaches RP2.11
- net MOSI: now also U5.16 (DIN), TP_MOSI.1
- net CLK: now reaches RP2.12
- net CLK: now also TP_CLK.1
- net CLKOUT: now reaches RP2.8
- net CS: now reaches RP2.9
- net CS: now also CRCW060310K0FKEA.2, TP_CS.1
- net 3V3 renamed +3V3
- net +3V3: now also U5.3 (AIN0P), C1206C103JBGACAUTO7210.1, CRCW060310K0FKEA.1, IC1.5 (VS), IC1.6 (REF2), TP_3V3.1, U1.5 (V+); no longer C1.1, C1210C105K1RACAUTO.1
- net CHIPSELECT: no longer names the net of U5.12 (CS)
- net CHIPSELECT: now also CRCW060310K0FKEA.1; no longer RP2.9
- net Vdivider: no longer names the net of TNPW080510K0BEEA.1, TNPW1206249KBEEA.2
- net Vdivider: now also U1.1 (+); no longer U5.3 (AIN0P)
- new net: IC1.2 (IN+), PSR400ITQFF0L50.3
- new net: C1.2, U5.2 (AGND)
- new net: C0603C224K5RACTU.2, C1210C105K1RACAUTO.1, U5.19 (DGND)
- new net AMP_OUT: CRCW060310K0FKEA.2, U1.3 (-), U1.4
- new net SHUNT_LOAD: IC1.3 (IN-), PSR400ITQFF0L50.2
- no-connect marks 26 -> 24
Other:
- moved on the sheet: C1210C105K1RACAUTO, J1, J2, LDO1, RP2, TNPW080510K0BEEA, TNPW1206249KBEEA

Commit message: new schematic feedback
Parts:
- removed CRCW060310K0FKEA: 10k ohms, symbol Device:R_US
- removed U1: OPA333AIDCKRG4, Package_TO_SOT_SMD:SOT-353_SC-70-5, symbol Amplifier_Operational:OPA333xxDCK
- added C0603S223K5RACTU: 0.022uF, symbol Device:C
- added CRCW060310K0FKEA1, CRCW060310K0FKEA2, CRCW060310K0FKEA3: 10k ohms, symbol Device:R_US
- added CRCW060350R0FKTA: 50 ohm, symbol Device:R_US
- added D1: WL-SMCW_0603, SMV_Passives:WL-SMCW_0603(diode), symbol SMV_Custom:WL-SMCW_0603
- added J4: 22035035, CON_22035035_MOL, symbol SMV_Custom:3-pin Mini Molex Spox
- added TS_CAN_H, TS_CAN_H1, TS_CAN_L, TS_CAN_L1: ~, symbol Connector:TestPoint
- added U2: MCP6286T-E/OT, SMV_ICs:SOT-23-5_MC_MCH, symbol SMV_Custom:MCP6286T-E_OT
Connections:
- net +3V3: now also C0603S223K5RACTU.2, CRCW060310K0FKEA1.1, CRCW060310K0FKEA3.1, CRCW060350R0FKTA.2, U2.5 (VDD); no longer C1206C103JBGACAUTO7210.1, CRCW060310K0FKEA.1, U5.3 (AIN0P)
- net AMP_OUT: now also U2.1 (VOUT), U2.4 (VIN-)
- net CAN_H: now also J4.1, TS_CAN_H.1, TS_CAN_H1.1
- net CAN_L: now also J4.3, TS_CAN_L.1, TS_CAN_L1.1
- net CS: now also U5.12 (CS), CRCW060310K0FKEA3.2
- net GND: now also U5.8 (AIN2N), C0603S223K5RACTU.1, CRCW060310K0FKEA2.1, D1.1, J4.2, U2.2 (VSS)
- net at TNPW080510K0BEEA.1, TNPW1206249KBEEA.2: now also U2.3 (VIN+)
- net at U5.7 (AIN2P): now also CRCW060310K0FKEA1.2, CRCW060310K0FKEA2.2
- new net: CRCW060350R0FKTA.1, D1.2
- new net Vdivider: C1206C103JBGACAUTO7210.1, CRCW060310K0FKEA.1, U5.3 (AIN0P)
- no-connect marks 24 -> 22
Other:
- moved on the sheet: C0603C224K5RACTU, C1, C1206C103JBGACAUTO7210, C1210C105K1RACAUTO, CRCW060310K0FKEA, IC1, PSR400ITQFF0L50, TNPW080510K0BEEA, TNPW1206249KBEEA, TP_CSENSE_OUT, TP_SHUNT_IN, TP_SHUNT_OUT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

Commit message: extra new fixes
Parts:
- added C0805C475K4RACTU1: 4.7uF, symbol Device:C
- added CRCW060350R0FKTA1: 50 ohms, symbol Device:R_US
- C0805C475K4RACTU: renamed from C1206C103JBGACAUTO7210; value 10nF -> 4.7uF
- CRCW0603150RFKEC: renamed from CRCW060350R0FKTA; value 50 ohm -> 150 ohm
- CRCW060350R0FKTA: renamed from CRCW060310K0FKEA; value 10k ohms -> 50 ohms
- renumbered C1 to C1210C105K1RACAUTO
Connections:
- net GND is gone; now on net +3V3: C0603S223K5RACTU.1, C0805C475K4RACTU.2, C1210C105K1RACAUTO.1, C1210C105K1RACAUTO.2, C1210C105K1RACAUTO.2, C1210C106K3RACAUTO.2, CRCW060310K0FKEA2.1, D1.1, IC1.4 (GND), IC1.7 (REF1), J1.N (NEG), J2.N (NEG), J3.2, J4.2, LDO1.4 (GND), RP2.13, RP2.2, TNPW080510K0BEEA.2, TP_GND.1, U2.2 (VSS), U5.4 (AIN0N), U5.5 (AIN1N), U5.8 (AIN2N)
- net +3V3: now also C0603C224K5RACTU.2, U5.19 (DGND), U5.2 (AGND), C0805C475K4RACTU1.2; no longer U5.1 (AVDD), U5.20 (DVDD)
- net CSENSE_OUT: now also C0805C475K4RACTU1.1, CRCW060350R0FKTA1.2; no longer IC1.8 (OUT)
- net at C1210C105K1RACAUTO.2: now also U5.1 (AVDD); no longer U5.2 (AGND)
- new net: CRCW060350R0FKTA1.1, IC1.8 (OUT)
- new net: C1210C105K1RACAUTO.1, U5.20 (DVDD)
Other:
- moved on the sheet: C0603S223K5RACTU, C0805C475K4RACTU, C1210C105K1RACAUTO, CRCW060350R0FKTA, IC1, PSR400ITQFF0L50, TNPW080510K0BEEA, TNPW1206249KBEEA, TP_CSENSE_OUT, TP_SHUNT_IN, TP_SHUNT_OUT, U2
