File: Joulemeter/joulemeter.kicad_sch (KiCad schematic)
At the start: 50 parts, among them J1 XT60-M, J2 XT60-M, J3 22035035, J4 22035035, U2 MCP6286T-E/OT, U5 PADS131M04QPWRQ1

Commit message: imsad
Parts:
- removed TS_CAN_H2, TS_CAN_L1: ~, TestPoint:TestPoint_Pad_D2.5mm, symbol Connector:TestPoint
- added TP1: TestPoint, SMV_Logo:SEM_logo, symbol Connector:TestPoint
- U5: footprint TSSOP20_PW_TEX -> SMV_ICs:TSSOP20_PW_TEX
- renumbered J2 to 48V_Power1, J4 to CAN1, TP_CLK1 to CLK1, TP_CSENSE_OUT1 to CSNSE1, INA240A3PWR1 to INA240A3, TP_MOSI1 to MOSI1
Changed lines of the file:
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@@
 	)
 	(symbol
-		(lib_id "Connector:TestPoint")
-		(at 77.47 175.26 270)
-		(unit 1)
-		(exclude_from_sim no)
-		(in_bom yes)
-		(on_board yes)
-		(dnp no)
-		(property "Reference" "TS_CAN_H2"
-			(at 78.994 173.482 90)
-			(effects
-				(font
-					(size 1.27 1.27)
-				)
-				(justify left)
-			)
-		)
-		(property "Value" "~"
-			(at 79.502 177.8 0)
-			(effects
-				(font
-					(size 1.27 1.27)
-				)
-				(justify left)
-			)
-		)
-		(property "Footprint" "TestPoint:TestPoint_Pad_D2.5mm"
-			(at 77.47 180.34 0)
-			(effects
-				(font
-					(size 1.27 1.27)
-				)
-				(hide yes)
-			)
-		)
-		(property "Datasheet" "~"
-			(at 77.47 180.34 0)
-			(effects
-				(font
-					(size 1.27 1.27)
-				)
-				(hide yes)
-			)
-		)
-		(property "Description" ""
-			(at 77.47 175.26 0)
-			(effects
-				(font
-					(size 1.27 1.27)
-				)
-				(hide yes)
-			)
-		)
-		(pin "1"
-		)
-		(instances
-			(project "joulemeter"
-				(path "/62c9b90f-facd-44d7-9ffc-18aee2f06026"
-					(reference "TS_CAN_H2")
-					(unit 1)
-				)
-			)
-		)
-	)
-	(symbol
 		(lib_id "Device:R_US")
 		(at 127 130.81 0)
@@
 	)
 	(symbol
+		(lib_id "Connector:TestPoint")
+		(at 45.72 163.83 0)
+		(unit 1)
+		(exclude_from_sim no)
+		(in_bom yes)
+		(on_board yes)
+		(dnp no)
+		(fields_autoplaced yes)
+		(property "Reference" "TP1"
+			(at 48.26 159.2579 0)
+			(effects
+				(font
+					(size 1.27 1.27)
+				)
+				(justify left)
+			)
+		)
+		(property "Value" "TestPoint"
+			(at 48.26 161.7979 0)
+			(effects
+				(font
+					(size 1.27 1.27)
+				)
+				(justify left)
+			)
+		)
+		(property "Footprint" "SMV_Logo:SEM_logo"
+			(at 50.8 163.83 0)
+			(effects
+				(font
+					(size 1.27 1.27)
+				)
+			)
+		)
+		(property "Datasheet" "~"
+			(at 50.8 163.83 0)
+			(effects
+				(font
+					(size 1.27 1.27)
+				)
+				(hide yes)
+			)
+		)
+		(property "Description" "test point"
+			(at 45.72 163.83 0)
+			(effects
+				(font
+					(size 1.27 1.27)
+				)
+				(hide yes)
+			)
+		)
+		(pin "1"
+		)
+		(instances
+			(project ""
+				(path "/62c9b90f-facd-44d7-9ffc-18aee2f06026"
+					(reference "TP1")
+					(unit 1)
+				)
+			)
+		)
+	)
+	(symbol
 		(lib_id "power:GND")
 		(at 237.49 17.78 90)
@@
 		(on_board yes)
 		(dnp no)
-		(property "Reference" "TP_CSENSE_OUT1"
+		(property "Reference" "CSNSE1"
 			(at 265.176 51.054 0)
 			(effects
@@
 			(project "joulemeter"
 				(path "/62c9b90f-facd-44d7-9ffc-18aee2f06026"
-					(reference "TP_CSENSE_OUT1")
+					(reference "CSNSE1")
 					(unit 1)
 				)
@@
 		(on_board yes)
 		(dnp no)
-		(property "Reference" "J2"
+		(property "Reference" "48V_Power1"
 			(at 270.51 50.8 0)
 			(effects
@@
 			(project "joulemeter"
 				(path "/62c9b90f-facd-44d7-9ffc-18aee2f06026"
-					(reference "J2")
+					(reference "48V_Power1")
 					(unit 1)
 				)
@@
 	)
 	(symbol
-		(lib_id "Connector:TestPoint")
-		(at 106.68 175.26 90)
-		(unit 1)
-		(exclude_from_sim no)
-		(in_bom yes)
-		(on_board yes)
-		(dnp no)
-		(property "Reference" "TS_CAN_L1"
-			(at 104.648 173.736 90)
-			(effects
-				(font
-					(size 1.27 1.27)
-				)
-				(justify left)
-			)
-		)
-		(property "Value" "~"
-			(at 104.648 172.72 0)
-			(effects
-				(font
-					(size 1.27 1.27)
-				)
-				(justify left)
-			)
-		)
-		(property "Footprint" "TestPoint:TestPoint_Pad_D2.5mm"
-			(at 106.68 170.18 0)
-			(effects
-				(font
-					(size 1.27 1.27)
-				)
-				(hide yes)
-			)
-		)
-		(property "Datasheet" "~"
-			(at 106.68 170.18 0)
-			(effects
-				(font
-					(size 1.27 1.27)
-				)
-				(hide yes)
-			)
-		)
-		(property "Description" ""
-			(at 106.68 175.26 0)
-			(effects
-				(font
-					(size 1.27 1.27)
-				)
-				(hide yes)
-			)
-		)
-		(pin "1"
-		)
-		(instances
-			(project "joulemeter"
-				(path "/62c9b90f-facd-44d7-9ffc-18aee2f06026"
-					(reference "TS_CAN_L1")
-					(unit 1)
-				)
-			)
-		)
-	)
-	(symbol
 		(lib_name "3-pin Mini Molex Spox_1")
 		(lib_id "SMV_Custom:3-pin Mini Molex Spox")
@@
 		(on_board yes)
 		(dnp no)
-		(property "Reference" "TP_MOSI1"
+		(property "Reference" "MOSI1"
 			(at 22.86 102.362 90)
 			(effects
@@
 			(project "joulemeter"
 				(path "/62c9b90f-facd-44d7-9ffc-18aee2f06026"
-					(reference "TP_MOSI1")
+					(reference "MOSI1")
 					(unit 1)
 				)
@@
 		(on_board yes)
 		(dnp no)
-		(property "Reference" "INA240A3PWR1"
+		(property "Reference" "INA240A3"
 			(at 226.06 53.086 0)
 			(effects
@@
 			(project ""
 				(path "/62c9b90f-facd-44d7-9ffc-18aee2f06026"
-					(reference "INA240A3PWR1")
+					(reference "INA240A3")
 					(unit 1)
 				)
@@
 			)
 		)
-		(property "Datasheet" "AP7387-50FDCR-7"
+		(property "Datasheet" ""
 			(at 74.93 57.15 0)
 			(effects
@@
 			)
 		)
-		(property "Footprint" "TSSOP20_PW_TEX"
+		(property "Footprint" "SMV_ICs:TSSOP20_PW_TEX"
 			(at 153.67 120.65 0)
 			(effects
@@
 		(on_board yes)
 		(dnp no)
-		(property "Reference" "TP_CLK1"
+		(property "Reference" "CLK1"
 			(at 21.844 99.822 90)
 			(effects
@@
 			(project "joulemeter"
 				(path "/62c9b90f-facd-44d7-9ffc-18aee2f06026"
-					(reference "TP_CLK1")
+					(reference "CLK1")
 					(unit 1)
 				)
@@
 		(dnp no)
 		(fields_autoplaced yes)
-		(property "Reference" "J4"
+		(property "Reference" "CAN1"
 			(at 78.74 182.8799 90)
 			(effects
@@
 			(project "joulemeter"
 				(path "/62c9b90f-facd-44d7-9ffc-18aee2f06026"
-					(reference "J4")
+					(reference "CAN1")
 					(unit 1)
 				)
