File: Joulemeter/joulemeter.kicad_pcb (KiCad board)
At the start: 2 copper layers, 129.5 x 83.5 mm, 50 parts, among them J1 XT60-M, J2 XT60-M, J3 22035035, J4 22035035, U2 MCP6286T-E/OT, U5 PADS131M04QPWRQ1

Commit message: pcb changes 2
Parts:
- removed TP_SHUNT_OUT2: ~, TestPoint:TestPoint_Pad_D2.5mm
- moved TP_5V1 176.9 mm to (184.2, 108.2)
- moved TP_48V1 161.9 mm to (161.0, 83.6)
- moved TS_CAN_H2 147.8 mm to (179.6, 141.7)
- moved TP_SHUNT_IN1 147.7 mm to (153.5, 69.2)
- moved TP_CLK1 146.1 mm to (154.8, 94.2)
- moved TP_MOSI1 143.9 mm to (154.8, 97.9)
- moved TS_CAN_L1 142.5 mm to (174.0, 141.8)
- moved TP_CS1 141.7 mm to (152.7, 106.0)
- moved TP_MISO1 140.9 mm to (154.9, 101.5)
- moved TS_CAN_L2 135.7 mm to (166.9, 141.8)
- moved TS_CAN_H1 134.5 mm to (161.2, 141.8)
- moved TP_CSENSE_OUT1 129.0 mm to (134.4, 99.0)
- moved TP_3V3 127.5 mm to (136.3, 111.5)
- moved TP_GND1 117.0 mm to (131.7, 103.2)
- moved J3 18.1 mm to (161.5, 136.6), turned to 180 degrees
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Connections:
- C70 pad 3: (no net) -> Net-(C70-Pad1)
- C70 pad 4: (no net) -> +48V
- C71 pad 3: (no net) -> +48V
- C71 pad 4: (no net) -> Net-(C71-Pad1)
- C74 pad 1: Net-(J2-POS) -> +48V
- RP2 pad 1: /CAN_H -> (no net)
- RP2 pad 2: GND -> (no net)
- RP2 pad 29: (no net) -> /CAN_L
- RP2 pad 30: (no net) -> GND
- RP2 pad 31: (no net) -> /CAN_H
Routing:
- net GND: track 13.7 -> 105.8 mm, vias 3 -> 29
- net +48V: track 116.8 -> 199.1 mm
- net /CAN_H: track 0.00 -> 40.9 mm
- net +5V: track 0.06 -> 34.1 mm
- net /SHUNT_LOAD: track 4.01 -> 33.6 mm
- net /CAN_L: track 0.00 -> 28.4 mm
- net +3V3: track 62.9 -> 80.9 mm
- net Net-(U2-VIN+): track 0.00 -> 11.3 mm
- net /CSENSE_OUT: track 0.00 -> 11.2 mm
- net /GPIO_CLKIN: track 7.48 -> 15.3 mm
- net /MOSI: track 7.13 -> 13.6 mm
- net Net-(C71-Pad1): track 0.00 -> 6.20 mm
- net /Vdivider: track 0.00 -> 6.05 mm
- net Net-(U5-CAP): track 2.38 -> 8.08 mm
- net Net-(C70-Pad1): track 0.00 -> 5.65 mm
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Other:
- board size 129.5 x 83.5 mm -> 64.3 x 90 mm

Commit message: pcb 4
Parts:
- added TP_SHUNT_OUT2: ~, TestPoint:TestPoint_Pad_D2.5mm, F.Cu at (134.8, 71.1)
- C1: renamed from C72; value C2220C475M1R2C7186 -> 4.7 µF
- C10: renamed from C1210C105K1RACAUTO2; value 1μF -> 1 µF
- C4: renamed from C74; value C2220C475M1R2C7186 -> 4.7 µF
- moved C3 54.6 mm to (130.8, 82.2)
- moved C4 46.2 mm to (131.5, 66.2)
- moved R2 42.1 mm to (131.3, 74.0)
- moved R10 6.46 mm to (148.9, 112.8)
- moved CSNS 5.55 mm to (139.5, 101.2)
- moved CS 5.37 mm to (148.7, 109.5)
- moved R5 4.12 mm to (133.2, 99.8)
- moved C9 3.64 mm to (136.0, 100.5)
- moved C6 2.52 mm to (184.2, 86.2), turned to 90 degrees
- moved R4 0.35 mm to (130.7, 98.2)
- renumbered C1210C105K1RACAUTO3 to C11, C1210C105K1RACAUTO4 to C12, C0603C224K5RACTU1 to C13, C3 to C14, C71 to C2, C70 to C3, C1210C105K1RACAUTO1 to C5, C1210C106K3RACAUTO1 to C6, C0603S223K5RACTU1 to C7, C0805C475K4RACTU2 to C8, C0805C475K4RACTU1 to C9, J4 to CAN, TP_CLK1 to CLKIN, TP_CS1 to CS, TP_CSENSE_OUT1 to CSNS, TP_GND1 to GND, INA240A3PWR1 to INA240, TP_MISO1 to MISO, TP_MOSI1 to MOSI, R10 to R1, CRCW060310K0FKEA3 to R10, R70 to R2, CRCW060350R0FKTA2 to R3, TNPW1206249KBEEA1 to R4, TNPW080510K0BEEA1 to R5, CRCW060350R0FKTA1 to R6, CRCW0603150RFKEC1 to R7, CRCW060310K0FKEA1 to R8, CRCW060310K0FKEA2 to R9, RP2 to RP2040, PSR400ITQFF0L50 to R_sht1
Connections:
- C2 pad 3: +48V -> (no net)
- C2 pad 4: Net-(C71-Pad1) -> (no net)
- C3 pad 4: +48V -> /SHUNT_LOAD
- C4 pad 1: +48V -> /SHUNT_LOAD
- R1 pad 2: Net-(C71-Pad1) -> Net-(C2-Pad1)
- RP2040 pad 1: (no net) -> /CAN_H
- RP2040 pad 2: (no net) -> GND
- RP2040 pad 29: /CAN_L -> (no net)
- RP2040 pad 30: GND -> (no net)
- RP2040 pad 31: /CAN_H -> (no net)
Routing:
- net /SHUNT_LOAD: track 33.6 -> 58.4 mm
- net +3V3: track 80.9 -> 90.9 mm
- net Net-(U2-VIN+): track 11.3 -> 2.96 mm
- net /CS: track 15.9 -> 22.6 mm
- net Net-(C71-Pad1): track 6.20 -> 0.00 mm
- net Net-(C2-Pad1): track 0.00 -> 6.20 mm
- net Net-(C3-Pad1): track 5.65 -> 10.1 mm
- net +5V: track 34.1 -> 31.7 mm
- net /CSENSE_OUT: track 11.2 -> 13.0 mm
- net GND: track 105.8 -> 106.1 mm, vias 29 -> 30
Other:
- board size 64.3 x 90 mm -> 78.9 x 89.7 mm

Commit message: pcb possibly final
Parts:
- moved TS_CAN_L2 21.0 mm to (146.2, 138.4), turned to -90 degrees
- moved TS_CAN_L1 19.0 mm to (192.7, 138.3), turned to 90 degrees
- moved TS_CAN_H1 17.4 mm to (146.3, 132.7), turned to -90 degrees
- moved TS_CAN_H2 15.7 mm to (192.6, 132.7), turned to 90 degrees
- moved J3 10.7 mm to (151.4, 133.0), turned to 90 degrees
- moved CAN 7.32 mm to (186.2, 133.0), turned to 90 degrees
- moved C1 5.78 mm to (167.1, 77.0)
- moved C13 3.64 mm to (151.2, 96.5), turned to 90 degrees
- moved C5 3.42 mm to (192.4, 86.8), turned to 90 degrees
- moved C11 1.29 mm to (144.1, 94.5)
- moved C12 1.29 mm to (148.1, 94.5)
- moved C14 0.15 mm to (136.6, 94.7)
Connections:
- RP2040 pad 29: (no net) -> /CAN_L
- RP2040 pad 30: (no net) -> GND
- RP2040 pad 31: (no net) -> /CAN_H
Routing:
- net /CAN_L: track 28.4 -> 53.4 mm
- net GND: track 106.1 -> 85.7 mm
- net Net-(U5-CAP): track 8.08 -> 3.76 mm
- net /CAN_H: track 40.9 -> 44.9 mm
- net +3V3: track 90.9 -> 88.3 mm
- net +48V: track 199.1 -> 197.1 mm

Commit message: pcb v1384
Parts:
- removed TS_CAN_H2, TS_CAN_L1: ~, TestPoint:TestPoint_Pad_D2.5mm
- moved R2 15.8 mm to (130.2, 89.8), turned to 180 degrees
- moved TS_CAN_L2 10.7 mm to (142.9, 128.2)
- moved J3 10.1 mm to (149.0, 123.2)
- moved TS_CAN_H1 10.0 mm to (142.9, 123.2)
- moved CAN 10.0 mm to (188.0, 123.2)
- moved C2 9.29 mm to (165.9, 76.1), turned to -90 degrees
- moved C1 8.67 mm to (175.7, 78.5), turned to 90 degrees
- moved J2 8.43 mm to (187.3, 75.5)
- moved R1 7.74 mm to (157.9, 70.9)
- moved R10 7.50 mm to (143.1, 108.2), turned to -90 degrees
- moved C4 6.64 mm to (129.8, 72.5)
- moved TP_SHUNT_OUT2 2.46 mm to (135.2, 73.5)
- moved GND 2.34 mm to (130.4, 105.2)
- moved C6 0.98 mm to (184.3, 87.2)
- moved R9 0.97 mm to (145.6, 106.4)
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Connections:
- net /CAN_L renamed CAN_N
- C2 pad 3: (no net) -> +48V
- C2 pad 4: (no net) -> Net-(C2-Pad1)
- CAN pad 1: /CAN_H -> CAN_P
- J3 pad 1: /CAN_H -> CAN_P
- RP2040 pad 31: /CAN_H -> CAN_P
- TS_CAN_H1 pad 1: /CAN_H -> CAN_P
Routing:
- net CAN_P: track 0.00 -> 56.9 mm
- net /CAN_H: track 44.9 -> 0.00 mm
- net +48V: track 197.1 -> 156.1 mm
- net GND: track 85.7 -> 69.9 mm, vias 30 -> 53
- net /SHUNT_LOAD: track 58.4 -> 44.9 mm
- net +3V3: track 88.3 -> 96.1 mm
- net Net-(U2-VIN+): track 2.96 -> 7.23 mm
- net /SCK: track 18.5 -> 22.6 mm, vias 1 -> 0
- net CAN_N: track 53.4 -> 56.7 mm
- net /CS: track 22.6 -> 25.3 mm
- net Net-(C3-Pad1): track 10.1 -> 7.71 mm
- net /RESET: track 14.0 -> 12.2 mm
- net +5V: track 31.7 -> 30.0 mm
- net Net-(C2-Pad1): track 6.20 -> 7.20 mm
- added copper zone on B.Cu, net GND
- added copper zone on F.Cu, net GND
Other:
- board size 78.9 x 89.7 mm -> 77.1 x 69.3 mm

Commit message: Finalized layout
Parts:
- moved C1 2.24 mm to (176.0, 76.3)
- moved R6 0.30 mm to (139.8, 98.4)
Routing:
- net GND: track 69.9 -> 58.6 mm
- net +48V: track 156.1 -> 146.2 mm
- net +3V3: track 96.1 -> 93.1 mm
- net /CSENSE_OUT: track 13.0 -> 11.0 mm

Commit message: Finishedd!
Parts:
- added REF**: MountingHole_3.2mm_M3, MountingHole:MountingHole_3.2mm_M3, F.Cu at (115.5, 69.5)
- added REF**: MountingHole_3.2mm_M3, MountingHole:MountingHole_3.2mm_M3, F.Cu at (192.8, 69.5)
- added REF**: MountingHole_3.2mm_M3, MountingHole:MountingHole_3.2mm_M3, F.Cu at (192.8, 130.8)
- added REF**: SEM_logo, SMV_Logo:SEM_logo, F.Cu at (129.8, 114.7)
- added REF**: MountingHole_3.2mm_M3, MountingHole:MountingHole_3.2mm_M3, F.Cu at (115.3, 130.8)
- 48V_IN CONNECTOR: renamed from J2
- moved TS_CAN_H1 5.88 mm to (143.9, 117.4)
- moved J3 5.74 mm to (149.6, 117.5)
- moved CAN 5.74 mm to (188.8, 117.5)
- moved TS_CAN_L2 5.66 mm to (143.9, 122.7)
- moved TP_3V3 5.49 mm to (141.8, 111.8)
- moved 48V_IN CONNECTOR 3.80 mm to (188.1, 79.3)
- renumbered TP_SHUNT_OUT2 to LOAD_CONNECTOR, TP_48V1 to TP_48V
Routing:
- net CAN_P: track 56.9 -> 68.5 mm
- net GND: track 58.6 -> 49.7 mm, vias 53 -> 52
- net CAN_N: track 56.7 -> 64.4 mm
- net +3V3: track 93.1 -> 93.9 mm
Other:
- board size 77.1 x 69.3 mm -> 85.4 x 69.3 mm
- board text added: "CAN"
- board text added: "CAN_N"
- board text added: "CAN_P"
- board text added: "Leo Chen 1/27/25 HIGH POWER JOULEMETER"

Commit message: helllo
Parts:
- C1, C4: footprint SMV_Passives:CAP_C2220C_2S_KEM-L -> SMV_Passives:CAPC340180_180N_KEM
- C10, C11, C12, C5, C6: footprint SMV_Passives:CAPC340270_190N_KEM-M -> SMV_Passives:Cap0805
- C13: footprint SMV_Passives:CAPC17595_87N_KEM-L -> SMV_Passives:Cap0805
- C7: value 0.022uF -> 0.1uF; footprint SMV_Passives:CAPC17595_87N_KEM-L -> SMV_Passives:Cap0805
- C8, C9: value 4.7uF -> 4.7nF; footprint SMV_Passives:Cap0805 -> SMV_Passives:CAPC17595_87N_KEM
- J2: renamed from 48V_IN CONNECTOR
- R10, R8, R9: value 10k ohms -> 20k ohms; footprint SMV_Passives:RESC1608X50N -> SMV_Passives:0603_resistors
- R3, R6, R7: footprint SMV_Passives:RESC1608X50N -> SMV_Passives:0805RESC2012X60N
- R4: value 249k ohms -> 500k ohms; footprint SMV_Passives:RES_TNPW1206_VIS-M -> SMV_Passives:0805RESC2012X60N
- R5: value 10k ohms -> 20k ohms; footprint SMV_Passives:0805RESC2012X60N -> SMV_Passives:0603_resistors
- moved C13 1.22 mm to (151.5, 95.4)
- moved U2 1.03 mm to (135.3, 104.8)
- moved TP_CLK1 0.83 mm to (155.7, 94.2)
- moved C12 0.81 mm to (147.8, 95.3)
- moved C11 0.74 mm to (143.9, 95.2)
- moved C1 0.74 mm to (175.9, 77.0)
- moved TP_MOSI1 0.67 mm to (155.4, 98.0)
- moved C6 0.57 mm to (184.3, 87.8)
- moved C5 0.50 mm to (192.2, 87.3)
- moved C10 0.42 mm to (184.2, 103.1)
- moved R7 0.22 mm to (183.9, 95.2)
- moved R3 0.19 mm to (139.0, 104.3)
- moved D1 0.18 mm to (184.2, 97.0)
- moved C7 0.12 mm to (136.7, 108.8)
- renumbered INA240 to INA240A3PWR1, CAN to J4, RP2040 to RP2, R_sht1 to R_shunt1, TP_48V to TP_48V1, CLKIN to TP_CLK1, CS to TP_CS1, CSNS to TP_CSENSE_OUT1, GND to TP_GND1, MISO to TP_MISO1, MOSI to TP_MOSI1, LOAD_CONNECTOR to TP_SHUNT_OUT2
Connections:
- C2 pad 3: +48V -> (no net)
- C2 pad 4: Net-(C2-Pad1) -> (no net)
- C3 pad 3: Net-(C3-Pad1) -> (no net)
- INA240A3PWR1 pad 2: +48V -> Net-(INA240A3PWR1-IN+)
- J3 pad 1: CAN_P -> /CAN_H
- J3 pad 3: CAN_N -> /CAN_L
- J4 pad 1: CAN_P -> /CAN_H
- J4 pad 3: CAN_N -> /CAN_L
- RP2 pad 29: CAN_N -> (no net)
- RP2 pad 30: GND -> (no net)
- RP2 pad 31: CAN_P -> (no net)
- TS_CAN_H1 pad 1: CAN_P -> /CAN_H
- TS_CAN_L2 pad 1: CAN_N -> /CAN_L
Routing:
- net CAN_P: track 68.5 -> 0.00 mm
- net /CAN_H: track 0.00 -> 68.5 mm
- net CAN_N: track 64.4 -> 0.00 mm
- net /CAN_L: track 0.00 -> 64.4 mm
- net GND: track 49.7 -> 55.7 mm
- net +3V3: track 93.9 -> 95.4 mm
- net Net-(U5-CAP): track 3.76 -> 4.79 mm
- net /SHUNT_LOAD: track 44.9 -> 45.8 mm
- net Net-(U2-VIN+): track 7.23 -> 6.41 mm
- net +48V: track 145.9 -> 146.5 mm

Commit message: hi
Parts:
- renumbered J2 to 48V_Power, J4 to CAN, TP_CLK1 to CLK, TP_CSENSE_OUT1 to CSNSE, INA240A3PWR1 to INA240A3, TP_MOSI1 to MOSI
Changed lines of the file:
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@@
 		(grid_origin 0 210)
 		(pcbplotparams
-			(layerselection 0x00010fc_ffffffff)
+			(layerselection 0x000103c_ffffffff)
 			(plot_on_all_layers_selection 0x0000000_00000000)
 			(disableapertmacros no)
@@
 			(outputformat 1)
 			(mirror no)
-			(drillshape 1)
+			(drillshape 0)
 			(scaleselection 1)
-			(outputdirectory "")
+			(outputdirectory "../../leos_order/")
 		)
 	)
@@
 		(tags "Capacitor")
 		(property "Reference" "C6"
-			(at 0 3 90)
+			(at 1.29 2.62 90)
 			(layer "F.SilkS")
 			(effects
@@
 		(layer "F.Cu")
 		(at 188.06 79.28)
-		(property "Reference" "J2"
+		(property "Reference" "48V_Power"
 			(at -0.345 -5.21 0)
 			(layer "F.SilkS")
@@
 		(tags "Capacitor")
 		(property "Reference" "C11"
-			(at 0 3 -90)
+			(at -3.18 -0.17 0)
 			(layer "F.SilkS")
 			(effects
@@
 		(tags "PADS131M04QPWRQ1 ")
 		(property "Reference" "U5"
-			(at 0 0 0)
+			(at 2.185 4.379398 0)
 			(unlocked yes)
 			(layer "F.SilkS")
@@
 		(tags "C1206C105K1RACTU ")
 		(property "Reference" "C1"
-			(at 0 0 90)
+			(at 0.62 -2.02 90)
 			(unlocked yes)
 			(layer "F.SilkS")
@@
 		(at 188.75924 117.48 90)
 		(tags "22035035 ")
-		(property "Reference" "J4"
+		(property "Reference" "CAN"
 			(at -9.79 -39.11924 0)
 			(unlocked yes)
@@
 		(descr "SMD pad as test Point, diameter 2.5mm")
 		(tags "test point SMD pad")
-		(property "Reference" "TP_CLK1"
-			(at -0.595 -2.59 0)
+		(property "Reference" "CLK"
+			(at -0.59 -2.21 0)
 			(layer "F.SilkS")
 			(effects
@@
 		(tags "test point SMD pad")
 		(property "Reference" "TP_GND1"
-			(at -3.05 1.1 0)
+			(at -1.51 2.46 0)
 			(layer "F.SilkS")
 			(effects
@@
 		(descr "SMD pad as test Point, diameter 2.5mm")
 		(tags "test point SMD pad")
-		(property "Reference" "TP_MOSI1"
-			(at -3.145 0.955 0)
+		(property "Reference" "MOSI"
+			(at -3.28 1.02 0)
 			(layer "F.SilkS")
 			(effects
@@
 		(tags "Capacitor")
 		(property "Reference" "C12"
-			(at 0 3 90)
+			(at 3.06 0.06 180)
 			(layer "F.SilkS")
 			(effects
@@
 		(layer "F.Cu")
 		(at 140.1 93.070602 -90)
-		(property "Reference" "INA240A3PWR1"
-			(at -2.980602 2.73 90)
+		(property "Reference" "INA240A3"
+			(at -3.780602 2.59 90)
 			(layer "F.SilkS")
 			(effects
@@
 		(tags "C0603C472K4RACTU ")
 		(property "Reference" "C8"
-			(at 0 0 -90)
+			(at 0.034398 -1.38 -90)
 			(unlocked yes)
 			(layer "F.SilkS")
@@
 		(tags "Capacitor")
 		(property "Reference" "C7"
-			(at 0 3 180)
+			(at -1.21 2.45 180)
 			(layer "F.SilkS")
 			(effects
@@
 		(descr "SMD pad as test Point, diameter 2.5mm")
 		(tags "test point SMD pad")
-		(property "Reference" "TP_CSENSE_OUT1"
-			(at -2.925 1.765 0)
+		(property "Reference" "CSNSE"
+			(at -2.035 -0.675 -90)
 			(layer "F.SilkS")
 			(effects
@@
 		(tags "Capacitor")
 		(property "Reference" "C13"
-			(at 0 3 90)
+			(at 2.49 0.1 180)
 			(layer "F.SilkS")
 			(effects
@@
 		(fp_arc
 			(start -8.304556 8.25436)
-			(mid -8.304689 8.247612)
+			(mid -8.304689 8.247611)
 			(end -8.300511 8.24231)
 			(stroke
@@
 		(fp_arc
 			(start -7.774364 12.655021)
-			(mid -7.771131 12.665266)
+			(mid -7.771131 12.665267)
 			(end -7.776942 12.674303)
 			(stroke
@@
 		(fp_arc
 			(start -4.883602 11.697921)
-			(mid -4.883173 11.693201)
+			(mid -4.883173 11.693202)
 			(end -4.878724 11.69157)
 			(stroke
@@
 		(fp_arc
 			(start -3.156379 11.616037)
-			(mid -3.161129 11.513181)
+			(mid -3.16113 11.513181)
 			(end -3.16328 11.410238)
 			(stroke
@@
 		(fp_arc
 			(start -0.45284 6.767971)
-			(mid -0.453954 6.770748)
+			(mid -0.453954 6.770747)
 			(end -0.456677 6.771986)
 			(stroke
@@
 		(tags "C1206C105K1RACTU ")
 		(property "Reference" "C4"
-			(at 0 0 180)
+			(at -1.0999 2.07 0)
 			(unlocked yes)
 			(layer "F.SilkS")
