File: Joulemeter/joulemeter.kicad_pcb (KiCad board)
At the start: 2 copper layers, 85.4 x 69.3 mm, 53 parts, among them J1 XT60-M, J3 22035035, U2 MCP6286T-E/OT, U5 PADS131M04QPWRQ1

Commit message: imsad
Parts:
- removed the REF** at (129.8, 114.7)
- added TP1: TestPoint, SMV_Logo:SEM_logo, F.Cu at (130.1, 114.7)
- renumbered 48V_Power to 48V_Power1, CAN to CAN1, CLK to CLK1, CSNSE to CSNSE1, MOSI to MOSI1
Connections:
- 48V_Power1 pad P: +48V -> Net-(48V_Power1-POS)
- C3 pad 4: /SHUNT_LOAD -> (no net)
- C4 pad 1: /SHUNT_LOAD -> Net-(48V_Power1-POS)
- J1 pad P: /SHUNT_LOAD -> +48V
- TP_SHUNT_OUT2 pad 1: /SHUNT_LOAD -> Net-(48V_Power1-POS)
