File: edwin_joulemeter/Joulemeter.kicad_sch (KiCad schematic)
At the start: 55 parts, among them J1 XT60-M, J2 22035035, J3 22035035, J4 XT60-M, U1 INA240A1PWR, U3 MCP6286T-E/OT, U4 PADS131M04QPWRQ1

Commit message: third update 1/22/25
Parts:
- added C2: 0.1uF, 16V, SMV_Passives:CAPC10555_55N_KEM, symbol SMV_Custom:C0402C104K4RACTU
- renumbered TP11 to 1V6, TP12 to 3V3, TP6 to 48V1, TP5 to 5V1, TP9 to CAN_H1, TP7 to CAN_L1, TP21 to CLKIN1, TP23 to CS1, TP1 to GND1, TP10 to I_ADC1, TP22 to MISO1, TP26 to MOSI1, TP25 to RESET1, TP8 to SCK1, TP13 to SHUNT_OUT1, TP4 to V_ADC1, TP3 to V_DIVIDER1
Connections:
- net +3V3: now also C2.1
- net GND: now also C2.2
Changed lines of the file:
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@@
 	)
 	(junction
+		(at 77.47 119.38)
+		(diameter 0)
+		(color 0 0 0 0)
+	)
+	(junction
 		(at 149.86 144.78)
 		(diameter 0)
@@
 	(wire
 		(pts
-			(xy 76.2 119.38) (xy 92.71 119.38)
+			(xy 76.2 119.38) (xy 77.47 119.38)
 		)
 		(stroke
@@
 	(wire
 		(pts
+			(xy 77.47 119.38) (xy 92.71 119.38)
+		)
+		(stroke
+			(width 0)
+			(type default)
+		)
+	)
+	(wire
+		(pts
 			(xy 228.6 157.48) (xy 246.38 157.48)
 		)
@@
 	(wire
 		(pts
+			(xy 77.47 127) (xy 77.47 128.27)
+		)
+		(stroke
+			(width 0)
+			(type default)
+		)
+	)
+	(wire
+		(pts
 			(xy 257.81 22.86) (xy 257.81 20.32)
 		)
@@
 		(on_board yes)
 		(dnp no)
-		(property "Reference" "TP11"
+		(property "Reference" "1V6"
 			(at 88.265 59.055 0)
 			(effects
@@
 			(project "Joulemeter"
 				(path "/ef45e13b-2349-4ec0-be73-c9420dd02b88"
-					(reference "TP11")
+					(reference "1V6")
 					(unit 1)
 				)
@@
 	)
 	(symbol
+		(lib_id "SMV_Custom:C0402C104K4RACTU")
+		(at 77.47 119.38 270)
+		(unit 1)
+		(exclude_from_sim no)
+		(in_bom yes)
+		(on_board yes)
+		(dnp no)
+		(property "Reference" "C2"
+			(at 78.105 121.92 90)
+			(effects
+				(font
+					(size 1.524 1.524)
+				)
+				(justify left)
+			)
+		)
+		(property "Value" "0.1uF, 16V"
+			(at 78.105 124.46 90)
+			(effects
+				(font
+					(size 1.524 1.524)
+				)
+				(justify left)
+			)
+		)
+		(property "Footprint" "SMV_Passives:CAPC10555_55N_KEM"
+			(at 77.47 119.38 0)
+			(effects
+				(font
+					(size 1.27 1.27)
+					(italic yes)
+				)
+				(hide yes)
+			)
+		)
+		(property "Datasheet" "C0402C104K4RACTU"
+			(at 77.47 119.38 0)
+			(effects
+				(font
+					(size 1.27 1.27)
+					(italic yes)
+				)
+				(hide yes)
+			)
+		)
+		(property "Description" ""
+			(at 77.47 119.38 0)
+			(effects
+				(font
+					(size 1.27 1.27)
+				)
+				(hide yes)
+			)
+		)
+		(pin "1"
+		)
+		(pin "2"
+		)
+		(instances
+			(project ""
+				(path "/ef45e13b-2349-4ec0-be73-c9420dd02b88"
+					(reference "C2")
+					(unit 1)
+				)
+			)
+		)
+	)
+	(symbol
 		(lib_id "power:GND")
 		(at 275.59 144.78 0)
@@
 		(on_board yes)
 		(dnp no)
-		(property "Reference" "TP9"
+		(property "Reference" "CAN_H1"
 			(at 149.86 101.6 90)
 			(effects
@@
 			(project "Joulemeter"
 				(path "/ef45e13b-2349-4ec0-be73-c9420dd02b88"
-					(reference "TP9")
+					(reference "CAN_H1")
 					(unit 1)
 				)
@@
 		(dnp no)
 		(fields_autoplaced yes)
-		(property "Reference" "TP4"
+		(property "Reference" "V_ADC1"
 			(at 115.57 169.6719 0)
 			(effects
@@
 			(project "Joulemeter"
 				(path "/ef45e13b-2349-4ec0-be73-c9420dd02b88"
-					(reference "TP4")
+					(reference "V_ADC1")
 					(unit 1)
 				)
@@
 	)
 	(symbol
+		(lib_id "power:GND")
+		(at 77.47 128.27 0)
+		(unit 1)
+		(exclude_from_sim no)
+		(in_bom yes)
+		(on_board yes)
+		(dnp no)
+		(fields_autoplaced yes)
+		(property "Reference" "#PWR031"
+			(at 77.47 134.62 0)
+			(effects
+				(font
+					(size 1.27 1.27)
+				)
+				(hide yes)
+			)
+		)
+		(property "Value" "GND"
+			(at 77.47 133.35 0)
+			(effects
+				(font
+					(size 1.27 1.27)
+				)
+			)
+		)
+		(property "Footprint" ""
+			(at 77.47 128.27 0)
+			(effects
+				(font
+					(size 1.27 1.27)
+				)
+				(hide yes)
+			)
+		)
+		(property "Datasheet" ""
+			(at 77.47 128.27 0)
+			(effects
+				(font
+					(size 1.27 1.27)
+				)
+				(hide yes)
+			)
+		)
+		(property "Description" "Power symbol creates a global label with name \"GND\" , ground"
+			(at 77.47 128.27 0)
+			(effects
+				(font
+					(size 1.27 1.27)
+				)
+				(hide yes)
+			)
+		)
+		(pin "1"
+		)
+		(instances
+			(project ""
+				(path "/ef45e13b-2349-4ec0-be73-c9420dd02b88"
+					(reference "#PWR031")
+					(unit 1)
+				)
+			)
+		)
+	)
+	(symbol
 		(lib_id "SMV_Custom:3-pin Mini Molex Spox")
 		(at 173.355 107.95 270)
@@
 		(on_board yes)
 		(dnp no)
-		(property "Reference" "TP10"
+		(property "Reference" "I_ADC1"
 			(at 105.41 102.87 0)
 			(effects
@@
 			(project "Joulemeter"
 				(path "/ef45e13b-2349-4ec0-be73-c9420dd02b88"
-					(reference "TP10")
+					(reference "I_ADC1")
 					(unit 1)
 				)
@@
 		(dnp no)
 		(fields_autoplaced yes)
-		(property "Reference" "TP5"
+		(property "Reference" "5V1"
 			(at 124.46 53.8479 0)
 			(effects
@@
 			(project "Joulemeter"
 				(path "/ef45e13b-2349-4ec0-be73-c9420dd02b88"
-					(reference "TP5")
+					(reference "5V1")
 					(unit 1)
 				)
@@
 		(dnp no)
 		(fields_autoplaced yes)
-		(property "Reference" "TP3"
+		(property "Reference" "V_DIVIDER1"
 			(at 38.1 157.9879 0)
 			(effects
@@
 			(project "Joulemeter"
 				(path "/ef45e13b-2349-4ec0-be73-c9420dd02b88"
-					(reference "TP3")
+					(reference "V_DIVIDER1")
 					(unit 1)
 				)
@@
 		(dnp no)
 		(fields_autoplaced yes)
-		(property "Reference" "TP1"
+		(property "Reference" "GND1"
 			(at 35.56 187.9599 90)
 			(effects
@@
 			(project "Joulemeter"
 				(path "/ef45e13b-2349-4ec0-be73-c9420dd02b88"
-					(reference "TP1")
+					(reference "GND1")
 					(unit 1)
 				)
@@
 		(on_board yes)
 		(dnp no)
-		(property "Reference" "TP8"
+		(property "Reference" "SCK1"
 			(at 203.835 90.17 90)
 			(effects
@@
 			(project "Joulemeter"
 				(path "/ef45e13b-2349-4ec0-be73-c9420dd02b88"
-					(reference "TP8")
+					(reference "SCK1")
 					(unit 1)
 				)
@@
 		(on_board yes)
 		(dnp no)
-		(property "Reference" "TP21"
+		(property "Reference" "CLKIN1"
 			(at 207.01 76.2 90)
 			(effects
@@
 			(project "Joulemeter"
 				(path "/ef45e13b-2349-4ec0-be73-c9420dd02b88"
-					(reference "TP21")
+					(reference "CLKIN1")
 					(unit 1)
 				)
@@
 		(dnp no)
 		(fields_autoplaced yes)
-		(property "Reference" "TP13"
+		(property "Reference" "SHUNT_OUT1"
 			(at 210.82 20.8279 0)
 			(effects
@@
 			(project "Joulemeter"
 				(path "/ef45e13b-2349-4ec0-be73-c9420dd02b88"
-					(reference "TP13")
+					(reference "SHUNT_OUT1")
 					(unit 1)
 				)
@@
 		(on_board yes)
 		(dnp no)
-		(property "Reference" "TP23"
+		(property "Reference" "CS1"
 			(at 199.39 100.33 90)
 			(effects
@@
 			(project "Joulemeter"
 				(path "/ef45e13b-2349-4ec0-be73-c9420dd02b88"
-					(reference "TP23")
+					(reference "CS1")
 					(unit 1)
 				)
@@
 		(dnp no)
 		(fields_autoplaced yes)
-		(property "Reference" "TP6"
+		(property "Reference" "48V1"
 			(at 143.51 20.8279 0)
 			(effects
@@
 					(size 1.27 1.27)
 				)
+				(hide yes)
 			)
 		)
@@
 			(project "Joulemeter"
 				(path "/ef45e13b-2349-4ec0-be73-c9420dd02b88"
-					(reference "TP6")
+					(reference "48V1")
 					(unit 1)
 				)
@@
 		(on_board yes)
 		(dnp no)
-		(property "Reference" "TP25"
+		(property "Reference" "RESET1"
 			(at 203.2 85.09 90)
 			(effects
@@
 			(project "Joulemeter"
 				(path "/ef45e13b-2349-4ec0-be73-c9420dd02b88"
-					(reference "TP25")
+					(reference "RESET1")
 					(unit 1)
 				)
@@
 		(dnp no)
 		(fields_autoplaced yes)
-		(property "Reference" "TP12"
-			(at 118.745 142.2399 90)
+		(property "Reference" "3V3"
+			(at 118.11 142.2399 90)
 			(effects
 				(font
@@
 		)
 		(property "Value" "TestPoint"
-			(at 118.745 144.7799 90)
+			(at 118.11 144.7799 90)
 			(effects
 				(font
@@
 			(project "Joulemeter"
 				(path "/ef45e13b-2349-4ec0-be73-c9420dd02b88"
-					(reference "TP12")
+					(reference "3V3")
 					(unit 1)
 				)
@@
 		(on_board yes)
 		(dnp no)
-		(property "Reference" "TP26"
+		(property "Reference" "MOSI1"
 			(at 207.01 78.74 90)
 			(effects
@@
 			(project "Joulemeter"
 				(path "/ef45e13b-2349-4ec0-be73-c9420dd02b88"
-					(reference "TP26")
+					(reference "MOSI1")
 					(unit 1)
 				)
@@
 		(on_board yes)
 		(dnp no)
-		(property "Reference" "TP7"
+		(property "Reference" "CAN_L1"
 			(at 137.16 101.6 90)
 			(effects
@@
 			(project "Joulemeter"
 				(path "/ef45e13b-2349-4ec0-be73-c9420dd02b88"
-					(reference "TP7")
+					(reference "CAN_L1")
 					(unit 1)
 				)
@@
 		(on_board yes)
 		(dnp no)
-		(property "Reference" "TP22"
+		(property "Reference" "MISO1"
 			(at 207.01 81.28 90)
 			(effects
@@
 			(project "Joulemeter"
 				(path "/ef45e13b-2349-4ec0-be73-c9420dd02b88"
-					(reference "TP22")
+					(reference "MISO1")
 					(unit 1)
 				)

Commit message: third update 1/25/25
Parts:
- added J5, J6, J7, J8: Screw_Terminal_01x01, TerminalBlock_MetzConnect:TerminalBlock_MetzConnect_360271_1x01_Horizontal_ScrewM3.0_Boxed, symbol Connector:Screw_Terminal_01x01

Commit message: small error lol
Connections:
- net GND: now also J4.N (NEG); no longer J4.P (POS)
- net SHUNT_OUT: now also J4.P (POS); no longer J4.N (NEG)
Other:
- moved on the sheet: C10
Changed lines of the file:
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@@
 	)
 	(junction
-		(at 262.89 25.4)
-		(diameter 0)
-		(color 0 0 0 0)
-	)
-	(junction
 		(at 30.48 162.56)
 		(diameter 0)
@@
 	)
 	(junction
+		(at 259.08 25.4)
+		(diameter 0)
+		(color 0 0 0 0)
+	)
+	(junction
 		(at 220.345 67.31)
 		(diameter 0)
@@
 	)
 	(junction
-		(at 252.73 25.4)
+		(at 35.56 162.56)
 		(diameter 0)
 		(color 0 0 0 0)
 	)
 	(junction
-		(at 35.56 162.56)
+		(at 113.03 156.21)
 		(diameter 0)
 		(color 0 0 0 0)
 	)
 	(junction
-		(at 113.03 156.21)
+		(at 252.73 25.4)
 		(diameter 0)
 		(color 0 0 0 0)
@@
 	(wire
 		(pts
-			(xy 262.89 22.86) (xy 257.81 22.86)
+			(xy 24.13 66.04) (xy 24.13 66.675)
 		)
 		(stroke
@@
 	(wire
 		(pts
-			(xy 24.13 66.04) (xy 24.13 66.675)
+			(xy 100.33 116.84) (xy 100.33 123.19)
 		)
 		(stroke
@@
 	(wire
 		(pts
-			(xy 100.33 116.84) (xy 100.33 123.19)
+			(xy 259.08 25.4) (xy 260.35 25.4)
 		)
 		(stroke
@@
 	(wire
 		(pts
+			(xy 252.73 25.4) (xy 259.08 25.4)
+		)
+		(stroke
+			(width 0)
+			(type default)
+		)
+	)
+	(wire
+		(pts
 			(xy 142.24 106.68) (xy 142.24 107.95)
 		)
@@
 	(wire
 		(pts
+			(xy 260.35 22.86) (xy 260.35 25.4)
+		)
+		(stroke
+			(width 0)
+			(type default)
+		)
+	)
+	(wire
+		(pts
 			(xy 275.59 139.7) (xy 275.59 144.78)
 		)
@@
 	(wire
 		(pts
-			(xy 262.89 35.56) (xy 262.89 38.1)
+			(xy 259.08 33.02) (xy 259.08 35.56)
 		)
 		(stroke
@@
 	(wire
 		(pts
-			(xy 252.73 25.4) (xy 262.89 25.4)
-		)
-		(stroke
-			(width 0)
-			(type default)
-		)
-	)
-	(wire
-		(pts
 			(xy 40.64 66.04) (xy 45.085 66.04)
 		)
@@
 	(wire
 		(pts
+			(xy 260.35 22.86) (xy 262.89 22.86)
+		)
+		(stroke
+			(width 0)
+			(type default)
+		)
+	)
+	(wire
+		(pts
 			(xy 77.47 127) (xy 77.47 128.27)
 		)
@@
 	(wire
 		(pts
-			(xy 257.81 22.86) (xy 257.81 20.32)
+			(xy 262.89 25.4) (xy 262.89 27.94)
 		)
 		(stroke
@@
 	(wire
 		(pts
-			(xy 262.89 25.4) (xy 262.89 27.94)
-		)
-		(stroke
-			(width 0)
-			(type default)
-		)
-	)
-	(wire
-		(pts
 			(xy 200.66 25.4) (xy 200.66 36.83)
 		)
@@
 	(symbol
 		(lib_id "power:GND")
-		(at 262.89 38.1 0)
+		(at 259.08 35.56 0)
 		(unit 1)
 		(exclude_from_sim no)
@@
 		(dnp no)
 		(property "Reference" "#PWR036"
-			(at 262.89 44.45 0)
+			(at 259.08 41.91 0)
 			(effects
 				(font
@@
 		)
 		(property "Value" "GND"
-			(at 262.89 42.545 0)
+			(at 259.08 40.005 0)
 			(effects
 				(font
@@
 		)
 		(property "Footprint" ""
-			(at 262.89 38.1 0)
+			(at 259.08 35.56 0)
 			(effects
 				(font
@@
 		)
 		(property "Datasheet" ""
-			(at 262.89 38.1 0)
+			(at 259.08 35.56 0)
 			(effects
 				(font
@@
 		)
 		(property "Description" "Power symbol creates a global label with name \"GND\" , ground"
-			(at 262.89 38.1 0)
+			(at 259.08 35.56 0)
 			(effects
 				(font
@@
 	(symbol
 		(lib_id "power:GND")
-		(at 257.81 20.32 180)
+		(at 262.89 27.94 0)
 		(unit 1)
 		(exclude_from_sim no)
@@
 		(fields_autoplaced yes)
 		(property "Reference" "#PWR032"
-			(at 257.81 13.97 0)
+			(at 262.89 34.29 0)
 			(effects
 				(font
@@
 		)
 		(property "Value" "GND"
-			(at 257.81 15.24 0)
+			(at 262.89 33.02 0)
 			(effects
 				(font
@@
 		)
 		(property "Footprint" ""
-			(at 257.81 20.32 0)
+			(at 262.89 27.94 0)
 			(effects
 				(font
@@
 		)
 		(property "Datasheet" ""
-			(at 257.81 20.32 0)
+			(at 262.89 27.94 0)
 			(effects
 				(font
@@
 		)
 		(property "Description" "Power symbol creates a global label with name \"GND\" , ground"
-			(at 257.81 20.32 0)
+			(at 262.89 27.94 0)
 			(effects
 				(font
@@
 	(symbol
 		(lib_id "SMV_Custom:C2220C475M1R2C7186")
-		(at 262.89 27.94 270)
+		(at 259.08 25.4 270)
 		(unit 1)
 		(exclude_from_sim no)
@@
 		(dnp no)
 		(property "Reference" "C10"
-			(at 266.7 30.4799 90)
+			(at 262.89 27.9399 90)
 			(effects
 				(font
@@
 		)
 		(property "Value" "4.7uF, 100V"
-			(at 266.7 33.0199 90)
+			(at 262.89 30.4799 90)
 			(effects
 				(font
@@
 		)
 		(property "Footprint" "CAP_C2220C_2S_KEM"
-			(at 262.89 27.94 0)
+			(at 259.08 25.4 0)
 			(effects
 				(font
@@
 		)
 		(property "Datasheet" "C2220C475M1R2C7186"
-			(at 262.89 27.94 0)
+			(at 259.08 25.4 0)
 			(effects
 				(font
@@
 		)
 		(property "Description" ""
-			(at 262.89 27.94 0)
+			(at 259.08 25.4 0)
 			(effects
 				(font

Commit message: i toast
Parts:
- C10, C13: footprint CAP_C2220C_2S_KEM -> SMV_Passives:CAPC340180_180N_KEM
- C12(notkemet)1: footprint SMV_Passives:0805RESC2012X60N -> SMV_Passives:Cap0805
- C2: footprint SMV_Passives:CAPC10555_55N_KEM -> SMV_Passives:Cap0805
- C3, C6: value 4.7uF,16V -> 4.7nF,16V; footprint SMV_Passives:Cap0805 -> SMV_Passives:CAPC17595_87N_KEM
- C8: footprint CAPC340180_180N_KEM -> SMV_Passives:CAPC340180_180N_KEM
- R1: value 604 kOHM, 0.26 W -> 500 kOHM, 0.26 W
- R11, R3, R4, R6, R7: footprint SMV_Passives:RESC1608X55N -> SMV_Passives:0805RESC2012X60N
- R2: value 26.1kohms, 0.13W -> 20kohms, 0.13W; footprint RES_TNPW0402_VIS -> SMV_Passives:0603_resistors
- U1: value INA240A1PWR -> INA240A3PWR

Commit message: imtired
Parts:
- removed J5, J6, J7, J8: Screw_Terminal_01x01, TerminalBlock_MetzConnect:TerminalBlock_MetzConnect_360271_1x01_Horizontal_ScrewM3.0_Boxed, symbol Connector:Screw_Terminal_01x01
- added TP1: TestPoint, SMV_Logo:SEM_logo, symbol Connector:TestPoint
- R1: footprint RES_TNPW0805_VIS -> SMV_Passives:RES_TNPW0805_VIS
- U1: footprint PW0008A_N_TEX -> SMV_ICs:PW0008A_N_TEX
- renumbered C12(notkemet)1 to C12, C12 to C21

Commit message: jaj
Parts:
- removed 3V3: TestPoint, TestPoint:TestPoint_Pad_1.5x1.5mm, symbol Connector:TestPoint
- added 3V1: TestPoint, TestPoint:TestPoint_Pad_1.5x1.5mm, symbol Connector:TestPoint
Connections:
- net +3V3: now also U3.5 (VDD), 3V1.1; no longer U3.2 (VSS)
- net GND: now also U3.2 (VSS); no longer U3.5 (VDD)
