File: edwin_joulemeter/Joulemeter.kicad_pcb (KiCad board)
At the start: 2 copper layers, 182.6 x 114 mm, 54 parts, among them J1 XT60-M, J2 22035035, J3 22035035, J4 XT60-M, U1 INA240A1PWR, U3 MCP6286T-E/OT, U4 PADS131M04QPWRQ1, U5 LTC1258CMS8-5-PBF

Commit message: updated 1/12/25
Parts:
- removed D1: WL-SMCW_0603, SMV_Passives:WL-SMCW_0603(diode)
- removed R6: 10kohms, 0.125W, SMV_Passives:0805RESC2012X60N
- removed R7: 150ohm, 0.1W, SMV_Passives:RESC1608X55N
- removed RP1: ~, SMV_Connectors:RP2040
- removed TP11, TP14, TP15, TP16, TP17, TP18, TP8: TestPoint, TestPoint:TestPoint_Pad_3.0x3.0mm
- added D2: WL-SMCW_0603, SMV_Passives:WL-SMCW_0603(diode), F.Cu at (150.3, 120.8)
- added R10: 10kohms, 0.125W, SMV_Passives:0805RESC2012X60N, F.Cu at (165.3, 84.3)
- added R11: 150ohm, 0.1W, SMV_Passives:RESC1608X55N, F.Cu at (156.5, 120.8)
- added RP2: ~, SMV_Connectors:RP2040, F.Cu at (144.6, 98.4)
- added TP21: TestPoint, TestPoint:TestPoint_Pad_3.0x3.0mm, F.Cu at (162.5, 90.5)
- added TP22: TestPoint, TestPoint:TestPoint_Pad_3.0x3.0mm, F.Cu at (162.5, 101.0)
- added TP23: TestPoint, TestPoint:TestPoint_Pad_3.0x3.0mm, F.Cu at (170.0, 82.0)
- added TP24: TestPoint, TestPoint:TestPoint_Pad_3.0x3.0mm, F.Cu at (161.5, 80.0)
- added TP25: TestPoint, TestPoint:TestPoint_Pad_3.0x3.0mm, F.Cu at (129.0, 75.0)
- added TP26: TestPoint, TestPoint:TestPoint_Pad_3.0x3.0mm, F.Cu at (129.0, 82.0)
- moved TP9 167.1 mm to (150.5, 70.5)
- moved TP7 163.1 mm to (140.0, 70.5)
- moved J1 158.4 mm to (34.0, 40.0)
- moved TP5 137.5 mm to (116.3, 103.3)
- moved TP2 123.4 mm to (96.5, 112.0)
- moved TP13 114.0 mm to (92.5, 40.5)
- moved R9 110.1 mm to (49.5, 58.0), turned to 90 degrees
- moved TP20 107.1 mm to (89.5, 55.0)
- moved TP6 104.3 mm to (69.0, 41.0)
- moved TP4 98.7 mm to (72.0, 90.0)
- moved J4 97.3 mm to (131.4, 39.5)
- moved TP10 97.0 mm to (80.5, 108.5)
- moved TP12 91.6 mm to (72.0, 77.5)
- moved TP19 89.7 mm to (72.5, 55.0)
- moved J3 89.2 mm to (163.0, 46.3), turned to 90 degrees
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Other:
- board size 182.6 x 114 mm -> 159.8 x 99.8 mm

Commit message: updated 1/14/25
Parts:
- moved TP22 34.2 mm to (128.5, 97.5)
- moved TP23 19.3 mm to (160.0, 98.5)
- moved TP24 14.6 mm to (160.0, 94.5)
- moved TP21 14.2 mm to (160.0, 104.5)
- moved R10 14.2 mm to (164.5, 98.5), turned to 0 degrees
- moved R11 13.8 mm to (142.7, 120.8)
- moved TP25 13.5 mm to (128.5, 88.5)
- moved TP26 11.0 mm to (128.5, 93.0)
- moved D2 10.8 mm to (139.5, 120.8)
- moved C12(notkemet)1 1.99 mm to (115.5, 88.5)
- moved C9 1.14 mm to (115.6, 85.5)
Connections:
- RP2 pad 11: /MOSI -> unconnected-(RP2-SCL-Pad11)
- RP2 pad 12: /GPIO_CLKIN -> unconnected-(RP2-SDA-Pad12)
- RP2 pad 14: /GPIO_RESET -> unconnected-(RP2-TX-Pad14)
- RP2 pad 15: /CS -> unconnected-(RP2-RX-Pad15)
- RP2 pad 18: /SCK -> unconnected-(RP2-SCK-Pad18)
- RP2 pad 20: unconnected-(RP2-D24-Pad20) -> /GPIO_RESET
- RP2 pad 21: unconnected-(RP2-A3-Pad21) -> /CS
- RP2 pad 22: /MISO -> unconnected-(RP2-A2-Pad22)
- RP2 pad 24: unconnected-(RP2-A0-Pad24) -> /SCK
- RP2 pad 5: unconnected-(RP2-D12-Pad5) -> /MISO
- RP2 pad 6: unconnected-(RP2-D11-Pad6) -> /MOSI
- RP2 pad 7: unconnected-(RP2-D10-Pad7) -> /GPIO_CLKIN
Routing:
- net /GPIO_RESET: track 0.00 -> 129.4 mm
- net /CS: track 0.00 -> 128.9 mm
- net /SCK: track 0.00 -> 114.4 mm
- net +3V3: track 0.00 -> 93.7 mm
- net /MISO: track 0.00 -> 28.0 mm
- net /GPIO_CLKIN: track 0.00 -> 26.7 mm
- net /MOSI: track 0.00 -> 25.8 mm
- net Net-(D2-Pad2): track 0.00 -> 1.64 mm

Commit message: updated 1/15/25
Parts:
- moved C7 51.9 mm to (141.0, 117.5)
- moved U4 46.8 mm to (147.1, 115.0), turned to 90 degrees
- moved U1 44.4 mm to (110.0, 96.0), turned to 180 degrees
- moved R3 40.1 mm to (113.8, 98.8)
- moved TP10 38.4 mm to (117.2, 97.2)
- moved R1 37.1 mm to (82.0, 107.1)
- moved C3 36.9 mm to (121.2, 97.3), turned to 90 degrees
- moved C5 35.6 mm to (115.5, 69.0)
- moved C8 35.6 mm to (107.0, 67.0)
- moved LDO1 35.6 mm to (111.4, 67.2)
- moved TP5 35.6 mm to (120.5, 68.0)
- moved C12(notkemet)1 35.0 mm to (144.5, 108.1), turned to 90 degrees
- moved TP3 34.3 mm to (85.5, 108.5)
- moved C9 34.1 mm to (141.5, 107.7), turned to 90 degrees
- moved R2 31.9 mm to (82.5, 110.5)
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Connections:
- U4 pad 10: unconnected-(U4-AIN3P-Pad10) -> /V_ADC
- U4 pad 5: GND -> unconnected-(U4-AIN1N-Pad5)
- U4 pad 6: /V_ADC -> unconnected-(U4-AIN1P-Pad6)
- U4 pad 9: unconnected-(U4-AIN3N-Pad9) -> GND
Routing:
- net +3V3: track 93.7 -> 6.25 mm
- net /CS: track 128.9 -> 54.7 mm
- net /SCK: track 114.4 -> 48.0 mm
- net +1V65: track 0.00 -> 66.2 mm
- net /V_ADC: track 0.00 -> 62.9 mm
- net /GPIO_RESET: track 129.4 -> 71.5 mm
- net /I_ADC: track 0.00 -> 48.6 mm
- net /GPIO_CLKIN: track 26.7 -> 69.8 mm
- net /MOSI: track 25.8 -> 63.2 mm
- net /MISO: track 28.0 -> 58.9 mm
- net Net-(U1-OUT): track 0.00 -> 6.84 mm
- net Net-(D2-Pad2): track 1.64 -> 0.00 mm

Commit message: updated second time 1/15/25
Parts:
- moved TP5 14.5 mm to (106.0, 69.0)
- moved C5 12.5 mm to (103.0, 70.0)
- moved LDO1 11.0 mm to (100.4, 68.2)
- moved C8 9.55 mm to (97.5, 68.0)
- moved C2 1.28 mm to (101.0, 100.5)
- moved TP2 1.18 mm to (101.0, 95.9)
Routing:
- net +3V3: track 6.25 -> 173.9 mm
Changed lines of the file:
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@@
 	(footprint "TestPoint:TestPoint_Pad_3.0x3.0mm"
 		(layer "F.Cu")
-		(at 99.8188 95.890002 180)
+		(at 101 95.890002 180)
 		(descr "SMD rectangular pad as test Point, square 3.0mm side length")
 		(tags "test point SMD pad rectangle square")
@@
 	(footprint "TestPoint:TestPoint_Pad_3.0x3.0mm"
 		(layer "F.Cu")
-		(at 120.5 68)
+		(at 106 69)
 		(descr "SMD rectangular pad as test Point, square 3.0mm side length")
 		(tags "test point SMD pad rectangle square")
@@
 	(footprint "SMV_Passives:CAP_8PACTU"
 		(layer "F.Cu")
-		(at 115.5 69 90)
+		(at 103 70 90)
 		(tags "C0805C106K8PACTU ")
 		(property "Reference" "C5"
@@
 			(polygon
 				(pts
-					(xy 114.8269 69.2921) (xy 114.8269 68.7079) (xy 116.1731 68.7079) (xy 116.1731 69.2921)
+					(xy 102.3269 70.2921) (xy 102.3269 69.7079) (xy 103.6731 69.7079) (xy 103.6731 70.2921)
 				)
 			)
@@
 	(footprint "SMV_ICs:U-DFN2020-6 (Type C)"
 		(layer "F.Cu")
-		(at 111.4055 67.150002 180)
+		(at 100.4055 68.150002 180)
 		(property "Reference" "LDO1"
 			(at 0.032 -1.9064 0)
@@
 	(footprint "SMV_Passives:CAPC340180_180N_KEM"
 		(layer "F.Cu")
-		(at 107 67 90)
+		(at 97.5 68 90)
 		(tags "C1206C105K1RACTU ")
 		(property "Reference" "C8"
@@
 			(polygon
 				(pts
-					(xy 106.150802 67.699199) (xy 106.150802 66.300801) (xy 107.849198 66.300801) (xy 107.849198 67.699199)
+					(xy 96.650802 68.699199) (xy 96.650802 67.300801) (xy 98.349198 67.300801) (xy 98.349198 68.699199)
 				)
 			)
@@
 	(footprint "SMV_Passives:Cap0805"
 		(layer "F.Cu")
-		(at 99.7188 100.490002 -90)
+		(at 101 100.490002 -90)
 		(descr "C0805")
 		(tags "Capacitor")
@@
 	)
 	(segment
+		(start 138 66)
+		(end 129.934314 66)
+		(width 0.2)
+		(layer "F.Cu")
+		(net 5)
+	)
+	(segment
+		(start 129.934314 66)
+		(end 124.5 71.434314)
+		(width 0.2)
+		(layer "F.Cu")
+		(net 5)
+	)
+	(segment
+		(start 124.5 71.5)
+		(end 124.5 80)
+		(width 0.2)
+		(layer "F.Cu")
+		(net 5)
+	)
+	(segment
+		(start 118 83.5)
+		(end 119.5 85)
+		(width 0.2)
+		(layer "F.Cu")
+		(net 5)
+	)
+	(segment
+		(start 138 80.5)
+		(end 138 66)
+		(width 0.2)
+		(layer "F.Cu")
+		(net 5)
+	)
+	(segment
+		(start 86 98.5)
+		(end 86 96.8)
+		(width 0.2)
+		(layer "F.Cu")
+		(net 5)
+	)
+	(segment
+		(start 124.5 97.565686)
+		(end 135.528814 108.5945)
+		(width 0.2)
+		(layer "F.Cu")
+		(net 5)
+	)
+	(segment
+		(start 86 96.8)
+		(end 99.3 83.5)
+		(width 0.2)
+		(layer "F.Cu")
+		(net 5)
+	)
+	(segment
+		(start 124.5 71.434314)
+		(end 124.5 71.5)
+		(width 0.2)
+		(layer "F.Cu")
+		(net 5)
+	)
+	(segment
+		(start 157 92.58)
+		(end 150.08 92.58)
+		(width 0.2)
+		(layer "F.Cu")
+		(net 5)
+	)
+	(segment
+		(start 150.08 92.58)
+		(end 138 80.5)
+		(width 0.2)
+		(layer "F.Cu")
+		(net 5)
+	)
+	(segment
+		(start 99.3 83.5)
+		(end 118 83.5)
+		(width 0.2)
+		(layer "F.Cu")
+		(net 5)
+	)
+	(segment
 		(start 161 82.97)
 		(end 160.4 83.57)
@@
 		(width 0.2)
 		(layer "F.Cu")
+		(net 5)
+	)
+	(segment
+		(start 107.100001 95.025001)
+		(end 109.474999 95.025001)
+		(width 0.2)
+		(layer "F.Cu")
+		(net 5)
+	)
+	(segment
+		(start 86 98.5)
+		(end 86.525 97.975)
+		(width 0.2)
+		(layer "F.Cu")
+		(net 5)
+	)
+	(segment
+		(start 124.5 80)
+		(end 124.5 97.565686)
+		(width 0.2)
+		(layer "F.Cu")
+		(net 5)
+	)
+	(segment
+		(start 119.5 85)
+		(end 124.5 80)
+		(width 0.2)
+		(layer "F.Cu")
+		(net 5)
+	)
+	(segment
+		(start 135.528814 108.5945)
+		(end 141.500002 108.5945)
+		(width 0.2)
+		(layer "F.Cu")
+		(net 5)
+	)
+	(segment
+		(start 109.474999 95.025001)
+		(end 119.5 85)
+		(width 0.2)
+		(layer "F.Cu")

Commit message: updated 1/16/2025
Parts:
- removed C2: 0.1uF,50V, SMV_Passives:Cap0805
- removed TP2, TP24: TestPoint, TestPoint:TestPoint_Pad_3.0x3.0mm
- removed U5: LTC1258CMS8-5-PBF, SMV_ICs:MSOP-8_MS_LIT
- added C14: 0.1uF,50V, SMV_Passives:Cap0805, F.Cu at (70.2, 87.4)
- added C15: 0.1uF,50V, SMV_Passives:Cap0805, F.Cu at (80.6, 90.5)
- added TP11: TestPoint, TestPoint:TestPoint_Pad_3.0x3.0mm, F.Cu at (80.7, 86.5)
- added TP8: TestPoint, TestPoint:TestPoint_Pad_3.0x3.0mm, F.Cu at (135.9, 79.2)
- added U2: REF2033QDDCRQ1, SMV_ICs:SOT-23-THIN-5_DDC_TEX, F.Cu at (74.6, 89.5)
- moved J1 106.4 mm to (140.4, 37.5)
- moved J4 102.0 mm to (32.4, 38.5)
- moved J3 81.4 mm to (148.0, 116.0), turned to 180 degrees
- moved R9 76.0 mm to (125.0, 49.4)
- moved J2 70.9 mm to (148.0, 107.5), turned to 180 degrees
- moved R8 56.2 mm to (47.5, 49.4)
- moved C10 54.0 mm to (61.0, 41.5)
- moved C13 53.9 mm to (113.5, 41.5)
- moved R11 50.3 mm to (134.5, 53.0)
- moved TP7 48.7 mm to (153.9, 99.2)
- moved C7 48.5 mm to (115.0, 76.5), turned to -90 degrees
- moved TP9 47.6 mm to (146.9, 99.2)
- moved D2 46.7 mm to (133.7, 56.0)
- moved U4 42.8 mm to (119.5, 82.3), turned to 0 degrees
- moved C6 39.2 mm to (106.4, 69.7)
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Connections:
- C1 pad 1: +5V -> GND
- C1 pad 2: GND -> +3V3
- RP2 pad 18: unconnected-(RP2-SCK-Pad18) -> /SCK
- RP2 pad 20: /GPIO_RESET -> unconnected-(RP2-D24-Pad20)
- RP2 pad 21: /CS -> unconnected-(RP2-A3-Pad21)
- RP2 pad 22: unconnected-(RP2-A2-Pad22) -> /MISO
- RP2 pad 23: unconnected-(RP2-A1-Pad23) -> /MOSI
- RP2 pad 24: /SCK -> /GPIO_CLKIN
- RP2 pad 4: unconnected-(RP2-D13-Pad4) -> /CS
- RP2 pad 5: /MISO -> /GPIO_RESET
- RP2 pad 6: /MOSI -> unconnected-(RP2-D11-Pad6)
- RP2 pad 7: /GPIO_CLKIN -> unconnected-(RP2-D10-Pad7)
- TP21 pad 1: /SCK -> /GPIO_CLKIN
- TP25 pad 1: /GPIO_CLKIN -> /GPIO_RESET
- U4 pad 10: /V_ADC -> /I_ADC
- U4 pad 3: /I_ADC -> /V_ADC
Routing:
- net +5V: track 0.00 -> 294.1 mm
- net +48V: track 0.00 -> 115.5 mm
- net +3V3: track 173.9 -> 94.6 mm
- net /GPIO_RESET: track 71.5 -> 0.00 mm
- net /CS: track 54.7 -> 0.00 mm
- net +1V65: track 66.2 -> 18.8 mm
- net /SHUNT_OUT: track 0.00 -> 45.0 mm
- net /V_ADC: track 62.9 -> 18.4 mm
- net /GPIO_CLKIN: track 69.8 -> 26.7 mm
- net /MOSI: track 63.2 -> 24.1 mm
- net /MISO: track 58.9 -> 20.2 mm
- net /I_ADC: track 48.6 -> 13.0 mm
- net /SCK: track 48.0 -> 15.1 mm
- net Net-(U1-OUT): track 6.84 -> 0.49 mm

Commit message: pcb 1/20/25
Parts:
- removed C1, C14: 0.1uF,50V, SMV_Passives:Cap0805
- removed TP19, TP20: TestPoint, TestPoint:TestPoint_Pad_3.0x3.0mm
- removed U2: REF2033QDDCRQ1, SMV_ICs:SOT-23-THIN-5_DDC_TEX
- added C2: 0.47uF, 6.3V, SMV_Passives:CAPC10555_55N_KEM, F.Cu at (115.1, 74.1)
- added R6: 1Mohm, 0.25W, SMV_Passives:RESC3015X65N, F.Cu at (113.6, 72.0)
- added R7: 370kohm, 0.125W, SMV_Passives:RESC2012X50N, F.Cu at (113.5, 74.9)
- added U5: TLV709A01DBVR, SMV_ICs:SOT-23-5_DBV_TEX, F.Cu at (109.1, 72.9)
- moved J4 119.8 mm to (126.8, 112.2)
- moved R8 93.7 mm to (127.4, 98.4), turned to 180 degrees
- moved C11 92.9 mm to (118.2, 101.0), turned to -90 degrees
- moved TP13 84.5 mm to (129.9, 104.4)
- moved J1 80.6 mm to (110.3, 112.3)
- moved TP1 77.8 mm to (50.5, 52.8)
- moved C10 75.4 mm to (118.2, 90.6)
- moved C12 64.5 mm to (105.2, 101.0), turned to -90 degrees
- moved J2 64.0 mm to (137.3, 44.4)
- moved C8 57.6 mm to (159.2, 64.2), turned to -90 degrees
- moved TP9 56.0 mm to (131.2, 45.5)
- moved TP7 53.9 mm to (148.3, 45.6)
- moved LDO1 51.8 mm to (156.3, 63.5), turned to 0 degrees
- moved R5 51.3 mm to (114.1, 83.5), turned to 0 degrees
- moved TP6 50.9 mm to (104.6, 87.6)
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Connections:
- C15 pad 2: +1V65 -> +3V3
- RP2 pad 20: unconnected-(RP2-D24-Pad20) -> /GPIO_RESET
- RP2 pad 21: unconnected-(RP2-A3-Pad21) -> /CS
- RP2 pad 4: /CS -> unconnected-(RP2-D13-Pad4)
- RP2 pad 5: /GPIO_RESET -> unconnected-(RP2-D12-Pad5)
Routing:
- net +5V: track 294.1 -> 5.58 mm
- net +48V: track 115.5 -> 21.1 mm
- net +3V3: track 94.6 -> 24.1 mm
- net /CAN_L: track 0.00 -> 54.5 mm
- net /CAN_H: track 0.00 -> 54.5 mm
- net /SHUNT_OUT: track 45.0 -> 14.3 mm
- net /GPIO_CLKIN: track 26.7 -> 7.54 mm
- net /MOSI: track 24.1 -> 6.75 mm
- net /MISO: track 20.2 -> 7.46 mm
- net /V_ADC: track 18.4 -> 5.70 mm
- net /GPIO_RESET: track 0.00 -> 10.1 mm
- net /I_ADC: track 13.0 -> 4.43 mm
- net /CS: track 0.00 -> 7.71 mm
- net /OP_AMP: track 0.00 -> 5.45 mm
- net Net-(U3-VIN+): track 0.00 -> 3.07 mm
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
Commit message: pcb updated 1/22/25
Parts:
- removed C2: 0.47uF, 6.3V, SMV_Passives:CAPC10555_55N_KEM
- removed U5: TLV709A01DBVR, SMV_ICs:SOT-23-5_DBV_TEX
- added C1: 1uF,50V, SMV_Passives:Cap0805, F.Cu at (115.9, 73.2)
- added D1: WL-SMCW_0603, SMV_Passives:WL-SMCW_0603(diode), F.Cu at (159.8, 70.3)
- added D3: WL-SMCW_0603, SMV_Passives:WL-SMCW_0603(diode), F.Cu at (159.8, 67.7)
- added REF35160QDBVR1: ~, SMV_ICs:SOT95P280X145-6N, F.Cu at (112.0, 73.2)
- R6: value 1Mohm, 0.25W -> 150ohm, 0.1W; footprint SMV_Passives:RESC3015X65N -> SMV_Passives:RESC1608X55N
- R7: value 370kohm, 0.125W -> 150ohm, 0.1W; footprint SMV_Passives:RESC2012X50N -> SMV_Passives:RESC1608X55N
- TP1, TP10, TP11, TP12, TP13, TP21, TP22, TP23, TP25, TP26, TP3, TP4, TP5, TP6, TP7, TP8, TP9: footprint TestPoint:TestPoint_Pad_3.0x3.0mm -> TestPoint:TestPoint_Pad_1.5x1.5mm
- moved R7 43.9 mm to (156.9, 67.7), turned to 0 degrees
- moved R6 43.3 mm to (156.9, 70.3), turned to 180 degrees
- moved TP21 34.1 mm to (128.4, 59.7)
- moved TP26 27.5 mm to (128.4, 62.3)
- moved TP6 21.9 mm to (118.3, 104.7)
- moved TP22 20.9 mm to (128.4, 64.8)
- moved R9 17.1 mm to (112.1, 107.2), turned to 90 degrees
- moved J4 16.4 mm to (141.8, 105.7), turned to 180 degrees
- moved J1 15.1 mm to (125.4, 111.1)
- moved TP8 14.4 mm to (128.4, 67.4)
- moved C12 7.62 mm to (112.1, 97.7)
- moved TP11 7.56 mm to (111.2, 70.0)
- moved C11 7.52 mm to (124.9, 97.7)
- moved R8 6.90 mm to (126.8, 105.3)
- moved TP23 6.60 mm to (124.7, 70.6)
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Connections:
- C11 pad 3: (no net) -> Net-(C11-Pad2)
- C11 pad 4: (no net) -> /SHUNT_OUT
- C12 pad 3: (no net) -> Net-(C12-Pad2)
- C12 pad 4: (no net) -> +48V
- R6 pad 2: +1V65 -> Net-(RP2-D12)
- R7 pad 1: +1V65 -> Net-(RP2-D13)
- R7 pad 2: GND -> Net-(D3-Pad2)
- RP2 pad 4: unconnected-(RP2-D13-Pad4) -> Net-(RP2-D13)
- RP2 pad 5: unconnected-(RP2-D12-Pad5) -> Net-(RP2-D12)
- TP11 pad 1: +1V65 -> +1V6
- U1 pad 6: +1V65 -> +1V6
- U1 pad 7: +1V65 -> +1V6
- U4 pad 5: unconnected-(U4-AIN1N-Pad5) -> GND
- U4 pad 6: unconnected-(U4-AIN1P-Pad6) -> GND
- U4 pad 7: +1V65 -> +1V6
Routing:
- net GND: track 0.00 -> 160.6 mm, vias 0 -> 13
- net +48V: track 21.1 -> 152.3 mm
- net +3V3: track 24.1 -> 52.5 mm
- net +1V65: track 20.9 -> 0.00 mm
- net +1V6: track 0.00 -> 19.8 mm
- net /SHUNT_OUT: track 14.3 -> 27.0 mm
- net /CS: track 7.71 -> 16.5 mm
- net /CAN_H: track 54.5 -> 61.7 mm
- net /CAN_L: track 54.5 -> 60.7 mm
- net Net-(C11-Pad2): track 0.00 -> 5.11 mm
- net Net-(C12-Pad2): track 0.00 -> 5.08 mm
- net Net-(RP2-D13): track 0.00 -> 3.35 mm
- net Net-(RP2-D12): track 0.00 -> 3.35 mm
- net /I_ADC: track 4.43 -> 7.60 mm
- net /GPIO_CLKIN: track 7.54 -> 10.7 mm
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
Commit message: updated 1/22/25 again
Parts:
- moved TP1 114.5 mm to (152.1, 105.6)
- moved TP7 4.43 mm to (146.3, 45.7)
- moved TP9 4.39 mm to (139.3, 45.8)
- moved J2 3.09 mm to (140.3, 41.1)
Routing:
- net /SHUNT_OUT: track 27.0 -> 44.9 mm
- net +48V: track 152.3 -> 170.0 mm
- net +3V3: track 52.5 -> 68.3 mm
- net /CAN_H: track 61.7 -> 57.6 mm
- net GND: track 160.6 -> 157.4 mm, vias 13 -> 15
- net /CAN_L: track 60.7 -> 57.6 mm
