File: edwin_joulemeter/Joulemeter.kicad_pcb (KiCad board)
At the start: 2 copper layers, 159.8 x 99.8 mm, 55 parts, among them J1 XT60-M, J2 22035035, J3 22035035, J4 XT60-M, U1 INA240A1PWR, U3 MCP6286T-E/OT, U4 PADS131M04QPWRQ1

Commit message: third update 1/22/25
Parts:
- added C2: 0.1uF, 16V, SMV_Passives:CAPC10555_55N_KEM, F.Cu at (121.9, 69.9)
- moved GND1 9.94 mm to (142.7, 102.5)
- moved J4 7.16 mm to (146.5, 111.2)
- moved CS1 2.83 mm to (125.5, 73.3)
- moved R5 1.38 mm to (117.7, 80.5)
- moved R10 1.16 mm to (123.5, 69.7)
- moved CLKIN1 0.50 mm to (128.2, 59.2)
- moved C12(notkemet)1 0.42 mm to (121.5, 58.5)
- moved C10 0.41 mm to (124.1, 87.7)
- moved RESET1 0.38 mm to (128.2, 70.8)
- moved C15 0.35 mm to (107.8, 73.3)
- moved C13 0.32 mm to (110.9, 87.7)
- moved SCK1 0.29 mm to (128.2, 67.7)
- moved MOSI1 0.25 mm to (128.2, 62.1)
- moved MISO1 0.24 mm to (128.2, 65.0)
- moved R4 0.21 mm to (111.8, 62.5)
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- renumbered TP11 to 1V6, TP12 to 3V3, TP6 to 48V1, TP5 to 5V1, TP9 to CAN_H1, TP7 to CAN_L1, TP21 to CLKIN1, TP23 to CS1, TP1 to GND1, TP10 to I_ADC1, TP22 to MISO1, TP26 to MOSI1, TP25 to RESET1, TP8 to SCK1, TP13 to SHUNT_OUT1, TP4 to V_ADC1, TP3 to V_DIVIDER1
Connections:
- C11 pad 3: Net-(C11-Pad2) -> (no net)
- C11 pad 4: /SHUNT_OUT -> (no net)
- C12 pad 3: Net-(C12-Pad2) -> (no net)
- C12 pad 4: +48V -> (no net)
Routing:
- net GND: track 157.4 -> 101.1 mm, vias 15 -> 21
- net /SHUNT_OUT: track 44.9 -> 51.0 mm
- net +3V3: track 68.3 -> 64.2 mm
- net +1V6: track 19.8 -> 16.5 mm
- net /CS: track 16.5 -> 19.2 mm
- net /MISO: track 8.22 -> 9.14 mm
- net +48V: track 170.0 -> 169.5 mm
- added copper zone on B.Cu, net GND
Other:
- board size 159.8 x 99.8 mm -> 67.3 x 82.5 mm
- board text added: "CANBUS"
- board text added: "IN CONNECTOR"
- board text added: "OUT CONNECTOR"

Commit message: updated 1/24/25
Parts:
- moved TPGND 8.63 mm to (151.0, 104.8)
- moved D1 5.55 mm to (162.1, 75.3)
- moved D3 3.98 mm to (162.2, 71.0)
- moved J3 2.71 mm to (140.3, 100.5)
- moved TPCS 2.62 mm to (127.8, 74.5)
- moved TP48V 1.64 mm to (119.9, 104.8)
- moved TPSHUNTOUT 0.51 mm to (132.8, 99.3)
- moved C12 0.18 mm to (111.9, 97.7)
- renumbered C12(notkemet)1 to C12, 3V3 to TP3.3, 48V1 to TP48V, 5V1 to TP5V, CAN_H1 to TPCANH, CAN_L1 to TPCANL, CLKIN1 to TPCLKIN, CS1 to TPCS, GND1 to TPGND, I_ADC1 to TPI, MISO1 to TPMISO, MOSI1 to TPMOSI, RESET1 to TPRESET, SCK1 to TPSCK, SHUNT_OUT1 to TPSHUNTOUT, V_ADC1 to TPV, V_DIVIDER1 to TPVDIV
Routing:
- net GND: track 101.1 -> 114.4 mm, vias 21 -> 24
- net /CAN_L: track 57.6 -> 62.9 mm
- net /CAN_H: track 57.6 -> 62.8 mm
- net Net-(D1-Pad2): track 1.40 -> 6.57 mm
- net Net-(D3-Pad2): track 1.40 -> 5.05 mm
- net /CS: track 19.2 -> 21.6 mm
- net /SHUNT_OUT: track 51.0 -> 53.3 mm
- net +48V: track 169.5 -> 170.7 mm
- net /MISO: track 9.14 -> 9.87 mm
- net +3V3: track 64.2 -> 64.8 mm
Other:
- board text removed: "CANBUS"

Commit message: updated 1/25/25
Parts:
- moved TPCANL 0.96 mm to (145.3, 45.8)
- moved TPCANH 0.89 mm to (140.2, 45.8)
- moved TPV 0.07 mm to (106.6, 58.4)
- moved TP3.3 0.07 mm to (104.0, 58.4)
- turned C2 to 90 degrees
- renumbered RP2 to RP2040
Connections:
- C11 pad 3: (no net) -> Net-(C11-Pad2)
- C11 pad 4: (no net) -> /SHUNT_OUT
- C12 pad 3: (no net) -> Net-(C12-Pad2)
- C12 pad 4: (no net) -> +48V
Routing:
- net GND: track 114.4 -> 59.7 mm, vias 24 -> 52
- net +48V: track 170.7 -> 164.4 mm
- net /SCK: track 15.7 -> 21.0 mm, vias 1 -> 0
- net +3V3: track 64.8 -> 69.6 mm, vias 0 -> 2
- net /CAN_H: track 62.8 -> 64.0 mm
- net /SHUNT_OUT: track 53.3 -> 54.5 mm
- net /CAN_L: track 62.9 -> 63.8 mm
- added copper zone on B.Cu, net +3V3
- added copper zone on F.Cu, net GND

Commit message: updated again 1/25/2025
Parts:
- moved TPSHUNTOUT 2.11 mm to (133.0, 101.4)
Routing:
- net /SHUNT_OUT: track 54.5 -> 50.7 mm
- net /MISO: track 9.87 -> 9.14 mm
- net /CS: track 21.6 -> 21.0 mm
Other:
- board text added: "EDWIN TANG 1/25/2025 JOULEMETER SMV"
Changed lines of the file:
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@@
 		(tags "test point SMD pad rectangle square")
 		(property "Reference" "TPVDIV"
-			(at -3.07 1.2 90)
+			(at -2.01 1.1 90)
 			(layer "F.SilkS")
 			(effects
@@
 	(footprint "TestPoint:TestPoint_Pad_1.5x1.5mm"
 		(layer "F.Cu")
-		(at 132.825 99.3)
+		(at 133 101.4)
 		(descr "SMD rectangular pad as test Point, square 1.5mm side length")
 		(tags "test point SMD pad rectangle square")
 		(property "Reference" "TPSHUNTOUT"
-			(at 2.105 -0.7 270)
+			(at 2.105 -0.7 -90)
 			(layer "F.SilkS")
 			(effects
@@
 		(layer "Edge.Cuts")
 	)
+	(gr_text "EDWIN TANG\n1/25/2025\nJOULEMETER\nSMV"
+		(at 101.8 46.8 0)
+		(layer "F.SilkS")
+		(effects
+			(font
+				(size 1.5 1.5)
+				(thickness 0.2)
+			)
+			(justify left bottom)
+		)
+	)
 	(gr_text "OUT CONNECTOR"
 		(at 139.8 116.79 0)
@@
 	)
 	(segment
-		(start 124.94 95.16175)
-		(end 129.24175 95.16175)
-		(width 0.8)
-		(layer "F.Cu")
-		(net 7)
-	)
-	(segment
 		(start 121.68 91.90175)
 		(end 124.94 95.16175)
@@
 	)
 	(segment
-		(start 142.825 111.15)
-		(end 142.925 111.15)
+		(start 121.68 88.11)
+		(end 121.68 91.90175)
 		(width 0.8)
 		(layer "F.Cu")
@@
 	)
 	(segment
-		(start 121.68 88.11)
-		(end 121.68 91.90175)
+		(start 126.93675 95.16175)
+		(end 142.925 111.15)
 		(width 0.8)
 		(layer "F.Cu")
@@
 	)
 	(segment
-		(start 138.85 107.175)
-		(end 142.825 111.15)
-		(width 0.8)
-		(layer "F.Cu")
-		(net 7)
-	)
-	(segment
-		(start 129.24175 95.16175)
-		(end 133.33 99.25)
-		(width 0.8)
-		(layer "F.Cu")
-		(net 7)
-	)
-	(segment
-		(start 134.9 107.175)
-		(end 138.85 107.175)
+		(start 124.94 95.16175)
+		(end 126.93675 95.16175)
 		(width 0.8)
 		(layer "F.Cu")
@@
 	)
 	(segment
-		(start 133.33 105.605)
-		(end 134.9 107.175)
-		(width 0.8)
-		(layer "F.Cu")
-		(net 7)
-	)
-	(segment
-		(start 133.33 99.25)
-		(end 133.33 105.605)
-		(width 0.8)
-		(layer "F.Cu")
-		(net 7)
-	)
-	(segment
 		(start 121.475 59.465)
 		(end 121.475 60.580352)
@@
 	)
 	(segment
-		(start 125.232152 66.500002)
-		(end 125.40435 66.6722)
+		(start 124.3995 66.500002)
+		(end 123.49465 66.500002)
 		(width 0.2)
 		(layer "F.Cu")
@@
 	(segment
 		(start 124.3995 66.500002)
-		(end 123.49465 66.500002)
+		(end 125.232152 66.500002)
 		(width 0.2)
 		(layer "F.Cu")
@@
 	)
 	(segment
-		(start 125.40435 66.6722)
-		(end 125.40435 67.90435)
+		(start 130.8365 69.25)
+		(end 132.3465 67.74)
 		(width 0.2)
 		(layer "F.Cu")
@@
 	)
 	(segment
-		(start 124.3995 66.500002)
-		(end 125.232152 66.500002)
+		(start 127.65 69.25)
+		(end 130.8365 69.25)
 		(width 0.2)
 		(layer "F.Cu")
@@
 	)
 	(segment
-		(start 123.05 66.944652)
-		(end 123.05 68.25)
+		(start 125.40435 67.00435)
+		(end 127.65 69.25)
 		(width 0.2)
 		(layer "F.Cu")
@@
 	)
 	(segment
-		(start 125.40435 67.90435)
-		(end 126.75 69.25)
+		(start 123.05 66.944652)
+		(end 123.05 68.25)
 		(width 0.2)
 		(layer "F.Cu")
@@
 	)
 	(segment
-		(start 130.8365 69.25)
-		(end 132.3465 67.74)
+		(start 125.40435 66.6722)
+		(end 125.40435 67.00435)
 		(width 0.2)
 		(layer "F.Cu")
@@
 	)
 	(segment
-		(start 126.75 69.25)
-		(end 130.8365 69.25)
+		(start 125.232152 66.500002)
+		(end 125.40435 66.6722)
 		(width 0.2)
 		(layer "F.Cu")
@@
 	)
 	(segment
-		(start 125.275685 64.550001)
-		(end 126.165686 63.66)
-		(width 0.2)
-		(layer "F.Cu")
-		(net 20)
-	)
-	(segment
-		(start 124.3995 64.550001)
-		(end 125.275685 64.550001)
-		(width 0.2)
-		(layer "F.Cu")
-		(net 20)
-	)
-	(segment
 		(start 131.9865 64.84)
 		(end 132.3465 65.2)
@@
 	)
 	(segment
-		(start 126.935 63.66)
-		(end 128.25 64.975)
+		(start 132.1215 64.975)
+		(end 132.3465 65.2)
 		(width 0.2)
 		(layer "F.Cu")
@@
 	)
 	(segment
-		(start 126.165686 63.66)
-		(end 126.935 63.66)
+		(start 124.3995 64.550001)
+		(end 127.825001 64.550001)
 		(width 0.2)
 		(layer "F.Cu")
@@
 	)
 	(segment
-		(start 132.1215 64.975)
-		(end 132.3465 65.2)
+		(start 127.825001 64.550001)
+		(end 128.25 64.975)
 		(width 0.2)
 		(layer "F.Cu")

Commit message: third update 1/25/25
Parts:
- added J5: Screw_Terminal_01x01, TerminalBlock_MetzConnect:TerminalBlock_MetzConnect_360271_1x01_Horizontal_ScrewM3.0_Boxed, F.Cu at (161.2, 40.6)
- added J6: Screw_Terminal_01x01, TerminalBlock_MetzConnect:TerminalBlock_MetzConnect_360271_1x01_Horizontal_ScrewM3.0_Boxed, F.Cu at (105.6, 40.6)
- added J7: Screw_Terminal_01x01, TerminalBlock_MetzConnect:TerminalBlock_MetzConnect_360271_1x01_Horizontal_ScrewM3.0_Boxed, F.Cu at (105.6, 113.4)
- added J8: Screw_Terminal_01x01, TerminalBlock_MetzConnect:TerminalBlock_MetzConnect_360271_1x01_Horizontal_ScrewM3.0_Boxed, F.Cu at (161.4, 113.4)
- renumbered RP2040 to RP2, 1V6 to TP1.6, TP48V to TP48, TP5V to TP5
Routing:
- net +48V: track 164.4 -> 162.0 mm
- net GND: vias 52 -> 47

Commit message: finished!
Parts:
- removed J5, J6, J7, J8: Screw_Terminal_01x01, TerminalBlock_MetzConnect:TerminalBlock_MetzConnect_360271_1x01_Horizontal_ScrewM3.0_Boxed
- added REF**: MountingHole_3.2mm_M3, MountingHole:MountingHole_3.2mm_M3, F.Cu at (101.0, 114.0)
- added REF**: MountingHole_3.2mm_M3, MountingHole:MountingHole_3.2mm_M3, F.Cu at (163.0, 114.0)
- added REF**: SEM_logo, SMV_Logo:SEM_logo, F.Cu at (119.9, 40.8)
- added REF**: MountingHole_3.2mm_M3, MountingHole:MountingHole_3.2mm_M3, F.Cu at (163.0, 40.0)
- added REF**: MountingHole_3.2mm_M3, MountingHole:MountingHole_3.2mm_M3, F.Cu at (101.0, 40.0)
- moved D2 0.93 mm to (126.3, 51.8)
- moved R11 0.93 mm to (128.7, 52.6)
- moved MISO 0.66 mm to (128.8, 65.3)
- moved MOSI 0.63 mm to (128.9, 62.3)
- moved SCK 0.61 mm to (128.8, 67.8)
- moved RESET 0.60 mm to (128.8, 70.9)
- moved CLKIN 0.59 mm to (128.8, 59.3)
- renumbered TP48 to 48V, J3 to CAN, J2 to CAN, TPCANH to CANH, TPCANL to CANL, TPCLKIN to CLKIN, TPCS to CS, TPGND to GND, TPMISO to MISO, TPMOSI to MOSI, TPRESET to RESET, TPSCK to SCK
Routing:
- net +3V3: track 69.6 -> 68.6 mm
Other:
- board size 67.3 x 82.5 mm -> 70.4 x 82.5 mm
- board text added: "48V IN"
- board text added: "EDWIN TANG 1/25/2025 HIGH POWER JOULEMETER"
- board text added: "Load"
- board text removed: "EDWIN TANG 1/25/2025 JOULEMETER SMV"
- board text removed: "IN CONNECTOR"
- board text removed: "OUT CONNECTOR"

Commit message: small error lol
Parts:
- added J5: Screw_Terminal_01x01, TerminalBlock_MetzConnect:TerminalBlock_MetzConnect_360271_1x01_Horizontal_ScrewM3.0_Boxed, F.Cu at (5.03, 4.17)
- added J6: Screw_Terminal_01x01, TerminalBlock_MetzConnect:TerminalBlock_MetzConnect_360271_1x01_Horizontal_ScrewM3.0_Boxed, F.Cu at (5.03, 13.5)
- added J7: Screw_Terminal_01x01, TerminalBlock_MetzConnect:TerminalBlock_MetzConnect_360271_1x01_Horizontal_ScrewM3.0_Boxed, F.Cu at (5.03, 22.9)
- added J8: Screw_Terminal_01x01, TerminalBlock_MetzConnect:TerminalBlock_MetzConnect_360271_1x01_Horizontal_ScrewM3.0_Boxed, F.Cu at (5.03, 32.2)
- moved J4 0.08 mm to (146.4, 111.2), turned to 0 degrees
- renumbered TP1.6 to 1V6, TP3.3 to 3V3, 48V to 48V1, TP5 to 5V1, CANH to CAN_H1, CANL to CAN_L1, CLKIN to CLKIN1, CS to CS1, GND to GND1, TPI to I_ADC1, CAN to J2, CAN to J3, MISO to MISO1, MOSI to MOSI1, RESET to RESET1, SCK to SCK1, TPSHUNTOUT to SHUNT_OUT1, TPV to V_ADC1, TPVDIV to V_DIVIDER1
Connections:
- J4 pad N: /SHUNT_OUT -> GND
- J4 pad P: GND -> /SHUNT_OUT
