File: edwin_joulemeter/Joulemeter.kicad_pcb (KiCad board)
At the start: 2 copper layers, 70.4 x 82.5 mm, 65 parts, among them J1 XT60-M, J2 22035035, J3 22035035, J4 XT60-M, J5 Screw_Terminal_01x01, J6 Screw_Terminal_01x01, J7 Screw_Terminal_01x01, J8 Screw_Terminal_01x01, U1 INA240A1PWR, U3 MCP6286T-E/OT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

Commit message: i toast
Parts:
- C10, C13: footprint SMV_Passives:CAP_C2220C_2S_KEM -> SMV_Passives:CAPC340180_180N_KEM
- C12(notkemet)1: renamed from C12; footprint SMV_Passives:0805RESC2012X60N -> SMV_Passives:Cap0805
- C2: footprint SMV_Passives:CAPC10555_55N_KEM -> SMV_Passives:Cap0805
- C3, C6: value 4.7uF,16V -> 4.7nF,16V; footprint SMV_Passives:Cap0805 -> SMV_Passives:CAPC17595_87N_KEM
- R1: value 604 kOHM, 0.26 W -> 500 kOHM, 0.26 W
- R11, R3, R4, R6, R7: footprint SMV_Passives:RESC1608X55N -> SMV_Passives:0805RESC2012X60N
- R2: value 26.1kohms, 0.13W -> 20kohms, 0.13W; footprint SMV_Passives:RES_TNPW0402_VIS -> SMV_Passives:0603_resistors
- U1: value INA240A1PWR -> INA240A3PWR
- moved R10 3.13 mm to (125.8, 71.8)
- moved CS1 1.81 mm to (129.6, 75.1)
- moved C2 1.40 mm to (123.0, 70.9)
- moved C9 1.12 mm to (125.5, 58.2)
- moved C6 0.90 mm to (116.0, 61.9)
- moved C13 0.88 mm to (111.8, 87.7)
- moved C10 0.85 mm to (123.3, 87.7)
- moved D2 0.67 mm to (125.8, 52.2)
- moved C12(notkemet)1 0.63 mm to (122.1, 58.3)
- moved C3 0.62 mm to (113.8, 68.0)
- moved I_ADC1 0.54 mm to (110.8, 66.9)
- moved 1V6 0.50 mm to (110.7, 69.7)
- moved R11 0.43 mm to (128.6, 53.0)
- moved R1 0.39 mm to (104.5, 64.3)
- moved R3 0.22 mm to (116.4, 68.2)
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Connections:
- C11 pad 3: Net-(C11-Pad2) -> (no net)
- C11 pad 4: /SHUNT_OUT -> (no net)
- C12 pad 3: Net-(C12-Pad2) -> (no net)
- C12 pad 4: +48V -> (no net)
Routing:
- net +3V3: track 68.6 -> 71.8 mm
- net /CS: track 21.0 -> 22.2 mm
- net GND: track 59.7 -> 58.8 mm, vias 47 -> 48
- net Net-(D2-Pad2): track 1.50 -> 2.05 mm

Commit message: flub
Parts:
- removed J5, J6, J7, J8: Screw_Terminal_01x01, TerminalBlock_MetzConnect:TerminalBlock_MetzConnect_360271_1x01_Horizontal_ScrewM3.0_Boxed
- renumbered C12(notkemet)1 to C12, CLKIN1 to CLKIN
Connections:
- C11 pad 3: (no net) -> Net-(C11-Pad2)
- C11 pad 4: (no net) -> /SHUNT_OUT
- C12 pad 3: (no net) -> Net-(C12-Pad2)
- C12 pad 4: (no net) -> +48V

Commit message: imtired
Parts:
- removed the REF** at (119.9, 40.8)
- added TP1: TestPoint, SMV_Logo:SEM_logo, F.Cu at (120.5, 40.6)
- renumbered C12 to C21, CLKIN to CLKIN1
Connections:
- C11 pad 3: Net-(C11-Pad2) -> (no net)
- C11 pad 4: /SHUNT_OUT -> (no net)
- C21 pad 3: Net-(C12-Pad2) -> (no net)
- C21 pad 4: +48V -> (no net)
- R9 pad 2: Net-(C12-Pad2) -> Net-(C21-Pad2)
Routing:
- net Net-(C21-Pad2): track 0.00 -> 5.18 mm
- net Net-(C12-Pad2): track 5.18 -> 0.00 mm

Commit message: jaj
Parts:
- moved 3V3 10.3 mm to (114.2, 56.8)
- moved C4 9.53 mm to (112.5, 59.8), turned to 0 degrees
- moved TP1 0.75 mm to (119.9, 41.1)
Connections:
- U3 pad 2: +3V3 -> GND
- U3 pad 5: GND -> +3V3
Routing:
- net +3V3: track 71.8 -> 65.2 mm
- net GND: track 58.8 -> 61.6 mm, vias 48 -> 47
- net Net-(U3-VIN+): track 5.73 -> 6.45 mm
