File: SMV Front and Center Board/SMV H and S Board.kicad_pcb (KiCad board)
At the start: 2 copper layers, 65 parts, among them J1 430450200, J2 22035035, J3 22035035, J4 22035035, J5 22035035, J6 Molex Micro-Fit 4 Pin, J7 430450200, J8 430450200, Q1 PSMN1R8-40YLC_115, Q2 PSMN1R8-40YLC_115, U1 PADS131M04QPWRQ1, U2 UA78M05QDCYRG4Q1, U3 MCP6286T-E/OT, U4 MCP6286T-E/OT

Commit message: Finalized layout
Parts:
- removed the D1 at (164.3, 60.5)
- removed the R1 at (135.0, 32.8)
- removed the R11 at (164.0, 57.5)
- added D4: WL-SMCW_0603, SMV_Passives:WL-SMCW_0603(diode), F.Cu at (164.7, 60.4)
- added R14: 150Ω, SMV_Passives:0805RESC2012X60N, F.Cu at (163.9, 57.5)
- added R9: RCS0603150RJNEA, 150Ω, SMV_Passives:0805RESC2012X60N, F.Cu at (132.8, 30.1)
- moved D2 50.6 mm to (132.0, 27.5), turned to 0 degrees
- moved D3 47.0 mm to (164.7, 65.8), turned to 180 degrees
- moved TP5 3.51 mm to (164.7, 42.0)
- moved C7 3.43 mm to (165.6, 38.5)
- moved TP17 1.94 mm to (174.4, 63.4)
- moved R12 0.44 mm to (163.9, 63.1)
Connections:
- R12 pad 1: Net-(D2-Pad2) -> Net-(D3-Pad2)
Routing:
- net GND: track 62.6 -> 37.2 mm, vias 29 -> 42
- net /Drain1: track 0.00 -> 5.44 mm
- net Net-(D1-Pad2): track 4.18 -> 1.78 mm
- net Net-(D4-Pad2): track 0.00 -> 1.88 mm
- net /SCLK: track 20.5 -> 18.7 mm

Commit message: Finished!
Parts:
- added G1: 3V3A, TestPoint:TestPoint_Pad_D1.0mm, F.Cu at (170.5, 53.8)
- added G2: 3V3A, TestPoint:TestPoint_Pad_D1.0mm, F.Cu at (167.6, 54.8)
- added REF**: MountingHole_3.2mm_M3, MountingHole:MountingHole_3.2mm_M3, F.Cu at (96.3, 81.4)
- added REF**: MountingHole_3.2mm_M3, MountingHole:MountingHole_3.2mm_M3, F.Cu at (96.3, 25.9)
- added REF**: SEM_logo, SMV_Logo:SEM_logo, F.Cu at (114.9, 26.9)
- added REF**: MountingHole_3.2mm_M3, MountingHole:MountingHole_3.2mm_M3, F.Cu at (191.1, 25.9)
- added REF**: MountingHole_3.2mm_M3, MountingHole:MountingHole_3.2mm_M3, F.Cu at (191.1, 81.4)
- Brake Pedal: renamed from J5
- Gas Pedal: renamed from J4
- moved CAN_N1 25.4 mm to (134.3, 75.3)
- moved CAN_P1 25.4 mm to (134.3, 77.9)
- moved CAN 25.4 mm to (123.6, 79.1)
- moved GND 16.6 mm to (133.8, 67.0)
- moved Power 5.24 mm to (183.5, 33.0)
- moved Power 4.17 mm to (183.5, 74.2)
- moved D3 2.70 mm to (164.7, 68.5)
- moved D4 2.70 mm to (164.7, 63.1)
- moved Horn 2.70 mm to (182.6, 63.0)
- moved R14 2.70 mm to (163.9, 60.2)
- moved Q2 2.70 mm to (169.0, 61.6)
- moved R12 2.70 mm to (163.9, 65.8)
- moved R16 2.70 mm to (164.9, 56.8)
- moved R18 2.70 mm to (168.5, 56.8)
- moved 3.3V 1.71 mm to (128.5, 33.8)
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- renumbered TP13 to 3.3V, J3 to CAN, J2 to CAN, TP9 to CLKIN, TP10 to CS, TP15 to D1, TP17 to D2, TP3 to GND, TP11 to H1, TP12 to H2, J7 to Horn, TP7 to MISO, TP6 to MOSI, J1 to Power, J8 to Power, TP8 to SCLK, TP4 to Test, J6 to Wipers
Routing:
- net /CAN_N: track 86.9 -> 61.3 mm
- net /CAN_P: track 86.8 -> 61.3 mm
- net Net-(Q2-Pad4): track 4.30 -> 6.33 mm
- net Net-(Q1-Pad4): track 4.82 -> 6.67 mm
- net /D11: track 3.77 -> 4.98 mm
- net Net-(RP1-D10): track 3.74 -> 4.86 mm
- net Net-(RP1-D6): track 3.95 -> 5.07 mm
- net GND: vias 42 -> 60
Other:
- board outline added: 102.3 x 63 mm
- board text added: "1/27/25"
- board text added: "Aritra Dhar"
- board text added: "Front Center Board"
