File: SMV Front and Center Board/SMV H and S Board.kicad_pcb (KiCad board)
At the start: 2 copper layers, 102.3 x 63 mm, 72 parts, among them Q1 PSMN1R8-40YLC_115, Q2 PSMN1R8-40YLC_115, U1 PADS131M04QPWRQ1, U2 UA78M05QDCYRG4Q1, U3 MCP6286T-E/OT, U4 MCP6286T-E/OT

Commit message: h
Parts:
- C11, C6: value 0603W475K250XD -> 4.7uF, 16V; footprint SMV_Passives:CAP_0603-X_NGC -> SMV_Passives:Cap0805
- C8: value C0805C224K3RACTU -> C0805C224K5RACAUTO; footprint SMV_Passives:Cap0805 -> SMV_Passives:CAP_8PACTU
- R1, R19, R2, R5: value 50Ω -> 49.9Ω, 0.125W
- R15, R16: value CRCW06031K00FKEA, 1KΩ -> 1kΩ
- R3, R4: value 40K -> 10K
- R6, R9: value RCS0603150RJNEA, 150Ω -> 150Ω
- moved R10 1.83 mm to (110.2, 50.6)
- moved R8 1.83 mm to (110.2, 54.6)
- moved REF** 1.25 mm to (116.1, 27.2)
- moved SCK 1.20 mm to (135.9, 53.2)
- moved C11 0.87 mm to (113.2, 51.2)
- moved C1 0.86 mm to (115.3, 42.2)
- moved R13 0.86 mm to (107.0, 42.0)
- moved U3 0.86 mm to (110.5, 43.3)
- moved CS 0.72 mm to (135.9, 56.1)
- renumbered TP1 to 12V, TP5 to 5V, SCLK to SCK
Connections:
- Power pad 1: GND -> +12V
- Power pad 2: +12V -> GND
Routing:
- net /HS2: track 5.68 -> 7.76 mm
- net /HS1: track 3.65 -> 5.01 mm
- net /ADC_IN2: track 4.31 -> 5.24 mm
- net Net-(J4-Pad3): track 17.7 -> 16.8 mm
- net GND: track 37.2 -> 37.9 mm

Commit message: gang
Parts:
- C8: value C0805C224K5RACAUTO -> 220nF,50V
- renumbered SCK to SCLK
Changed lines of the file:
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@@
 			)
 		)
-		(property "Description" ""
+		(property "Description" "C623478"
 			(at 0 0 0)
 			(layer "F.Fab")
@@
 			)
 		)
-		(property "Description" ""
+		(property "Description" "C623478"
 			(at 0 0 90)
 			(layer "F.Fab")
@@
 			)
 		)
-		(property "Value" "C0805C224K5RACAUTO"
+		(property "Value" "220nF,50V"
 			(at 0 0 90)
 			(unlocked yes)
@@
 			)
 		)
-		(property "Datasheet" ""
+		(property "Datasheet" "C0805C224K5RACAUTO"
 			(at 0 0 90)
 			(layer "F.Fab")
@@
 		(fp_arc
 			(start -8.304556 8.25436)
-			(mid -8.304689 8.247612)
+			(mid -8.304689 8.247611)
 			(end -8.300511 8.24231)
 			(stroke
@@
 		(fp_arc
 			(start -7.774364 12.655021)
-			(mid -7.771131 12.665266)
+			(mid -7.771131 12.665267)
 			(end -7.776942 12.674303)
 			(stroke
@@
 		(fp_arc
 			(start -4.883602 11.697921)
-			(mid -4.883173 11.693201)
+			(mid -4.883173 11.693202)
 			(end -4.878724 11.69157)
 			(stroke
@@
 		(fp_arc
 			(start -3.156379 11.616037)
-			(mid -3.161129 11.513181)
+			(mid -3.16113 11.513181)
 			(end -3.16328 11.410238)
 			(stroke
@@
 		(fp_arc
 			(start -0.45284 6.767971)
-			(mid -0.453954 6.770748)
+			(mid -0.453954 6.770747)
 			(end -0.456677 6.771986)
 			(stroke
@@
 		(tags "PADS131M04QPWRQ1 ")
 		(property "Reference" "U1"
-			(at 0 0 0)
+			(at 0.63 4.47 0)
 			(unlocked yes)
 			(layer "F.SilkS")
@@
 			)
 		)
-		(fp_text user "${REFERENCE}"
-			(at 0 0 0)
-			(unlocked yes)
+		(fp_text user "*"
+			(at -1.8669 -3.2258 0)
 			(layer "F.Fab")
 			(effects
@@
 			)
 		)
-		(fp_text user "*"
-			(at -1.8669 -3.2258 0)
+		(fp_text user "${REFERENCE}"
+			(at 0 0 0)
 			(unlocked yes)
 			(layer "F.Fab")
@@
 		(fp_text user "*"
 			(at -1.8669 -3.2258 0)
+			(unlocked yes)
 			(layer "F.Fab")
 			(effects
@@
 			)
 		)
-		(property "Description" ""
+		(property "Description" "C485570"
 			(at 0 0 0)
 			(layer "F.Fab")
@@
 		(descr "SMD pad as test Point, diameter 1.5mm")
 		(tags "test point SMD pad")
-		(property "Reference" "SCK"
+		(property "Reference" "SCLK"
 			(at -2.65 -0.16 0)
 			(layer "F.SilkS")

Commit message: im fried
Parts:
- removed C11, C6: 4.7uF, 16V, SMV_Passives:Cap0805
- removed R19, R5: 49.9Ω, 0.125W, SMV_Passives:0805RESC2012X60N
- C2: value 1uF,16V -> 4.7nF,16V; footprint SMV_Passives:Cap0805 -> SMV_Passives:CAPC17595_87N_KEM
- C3: value 1uF,16V -> 4.7F,16V; footprint SMV_Passives:Cap0805 -> SMV_Passives:CAPC17595_87N_KEM
- J4: renamed from Gas Pedal
- J5: renamed from Brake Pedal
- renumbered Power to J1, CAN to J2, CAN to J3, Wipers to J6, Horn to J7, Power to J8, 12V to TP1, CS to TP10, H1 to TP11, H2 to TP12, 3.3V to TP13, G2 to TP14, D1 to TP15, D2 to TP17, G1 to TP2, GND to TP3, Test to TP4, 5V to TP5, MOSI to TP6, MISO to TP7, SCLK to TP8, CLKIN to TP9
Connections:
- U3 pad 1: /FB -> /ADC_IN1
- U3 pad 4: /FB -> /ADC_IN1
- U4 pad 1: Net-(U4-VIN-) -> /ADC_IN2
- U4 pad 4: Net-(U4-VIN-) -> /ADC_IN2
Routing:
- net /FB: track 5.94 -> 0.00 mm
- net Net-(U4-VIN-): track 5.80 -> 0.00 mm
- net /ADC_IN1: track 5.11 -> 8.51 mm
- net /ADC_IN2: track 5.24 -> 8.37 mm
- net GND: track 37.9 -> 35.3 mm, vias 60 -> 58

Commit message: fuck
Parts:
- removed the REF** at (116.1, 27.2)
- added Hall1: HS1, TestPoint:TestPoint_Pad_D1.5mm, F.Cu at (114.1, 45.6)
- added Hall2: HS1, TestPoint:TestPoint_Pad_D1.5mm, F.Cu at (117.2, 51.4)
- added TP1: TestPoint, SMV_Logo:SEM_logo, F.Cu at (116.6, 27.1)
- Brake Pedal1: renamed from J4
- Gas Pedal1: renamed from J5
- moved 3.3V1 1.29 mm to (129.7, 34.2)
- moved C3 0.77 mm to (120.8, 49.8)
- moved R2 0.67 mm to (117.6, 49.1)
- moved C2 0.41 mm to (120.5, 46.0)
- moved R1 0.39 mm to (117.4, 46.7)
- renumbered TP1 to 12V1, TP13 to 3.3V1, TP5 to 5V1, J2 to CAN1, J3 to CAN2, TP9 to CLKIN1, TP10 to CS1, TP15 to Drain1, TP17 to Drain2, TP2 to G1, TP14 to G2, TP3 to GND1, TP12 to H1, TP11 to H2, J7 to Horn1, TP7 to MISO1, TP6 to MOSI1, J8 to Power1, TP8 to SCK1, TP4 to Test1, J6 to Wiper1
Routing:
- net Net-(U1-AIN1P): track 6.21 -> 5.07 mm
- net Net-(Brake Pedal1-Pad3): track 16.8 -> 15.9 mm
