File: SMV Front and Center Board/SMV H and S Board.kicad_sch (KiCad schematic)
At the start: 65 parts, among them J1 430450200, J2 22035035, J3 22035035, J4 22035035, J5 22035035, J6 Molex Micro-Fit 4 Pin, J7 430450200, J8 430450200, Q1 PSMN1R8-40YLC_115, Q2 PSMN1R8-40YLC_115, U1 PADS131M04QPWRQ1, U2 UA78M05QDCYRG4Q1, U3 MCP6286T-E/OT, U4 MCP6286T-E/OT

Commit message: Finished!
Parts:
- added TP14, TP2: 3V3A, TestPoint:TestPoint_Pad_D1.0mm, symbol Connector:TestPoint
Connections:
- net at Q1.4, R15.2, R17.1: now also TP2.1
- net at Q2.4, R16.2, R18.2: now also TP14.1
Changed lines of the file:
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@@
 	)
 	(symbol
+		(lib_id "Connector:TestPoint")
+		(at 228.6 60.96 90)
+		(unit 1)
+		(exclude_from_sim no)
+		(in_bom yes)
+		(on_board yes)
+		(dnp no)
+		(property "Reference" "TP2"
+			(at 226.06 59.69 90)
+			(effects
+				(font
+					(size 1.27 1.27)
+				)
+				(justify right)
+			)
+		)
+		(property "Value" "3V3A"
+			(at 220.472 57.404 0)
+			(effects
+				(font
+					(size 1.27 1.27)
+				)
+				(justify right)
+				(hide yes)
+			)
+		)
+		(property "Footprint" "TestPoint:TestPoint_Pad_D1.0mm"
+			(at 228.6 55.88 0)
+			(effects
+				(font
+					(size 1.27 1.27)
+				)
+				(hide yes)
+			)
+		)
+		(property "Datasheet" "~"
+			(at 228.6 55.88 0)
+			(effects
+				(font
+					(size 1.27 1.27)
+				)
+				(hide yes)
+			)
+		)
+		(property "Description" "test point"
+			(at 228.6 60.96 0)
+			(effects
+				(font
+					(size 1.27 1.27)
+				)
+				(hide yes)
+			)
+		)
+		(pin "1"
+		)
+		(instances
+			(project "SMV H and S Board"
+				(path "/65429182-9298-499e-afe0-28215a09a0c3"
+					(reference "TP2")
+					(unit 1)
+				)
+			)
+		)
+	)
+	(symbol
 		(lib_id "power:GND")
 		(at 267.97 73.66 0)
@@
 					(unit 1)
 				)
+			)
+		)
+	)
+	(symbol
+		(lib_id "Connector:TestPoint")
+		(at 234.95 104.14 90)
+		(unit 1)
+		(exclude_from_sim no)
+		(in_bom yes)
+		(on_board yes)
+		(dnp no)
+		(property "Reference" "TP14"
+			(at 232.41 102.87 90)
+			(effects
+				(font
+					(size 1.27 1.27)
+				)
+				(justify right)
+			)
+		)
+		(property "Value" "3V3A"
+			(at 226.822 100.584 0)
+			(effects
+				(font
+					(size 1.27 1.27)
+				)
+				(justify right)
+				(hide yes)
+			)
+		)
+		(property "Footprint" "TestPoint:TestPoint_Pad_D1.0mm"
+			(at 234.95 99.06 0)
+			(effects
+				(font
+					(size 1.27 1.27)
+				)
+				(hide yes)
+			)
+		)
+		(property "Datasheet" "~"
+			(at 234.95 99.06 0)
+			(effects
+				(font
+					(size 1.27 1.27)
+				)
+				(hide yes)
+			)
+		)
+		(property "Description" "test point"
+			(at 234.95 104.14 0)
+			(effects
+				(font
+					(size 1.27 1.27)
+				)
+				(hide yes)
+			)
+		)
+		(pin "1"
+		)
+		(instances
+			(project "SMV H and S Board"
+				(path "/65429182-9298-499e-afe0-28215a09a0c3"
+					(reference "TP14")
+					(unit 1)
+				)

Commit message: h
Parts:
- C11, C6: value 0603W475K250XD -> 4.7uF, 16V; footprint SMV_Passives:CAP_0603-X_NGC -> SMV_Passives:Cap0805
- C8: value C0805C224K3RACTU -> 220nF,50V; footprint SMV_Passives:Cap0805 -> SMV_Passives:CAP_8PACTU; Arrow Part Number C0805C224K3RACTU -> (none); Arrow Price/Stock https://www.arrow.com/en/products/c0805c224k3ractu/kemet-co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 -> (none); Height 1.1 -> (none); Manufacturer_Name KEMET -> (none); Manufacturer_Part_Number C0805C224K3RACTU -> (none); Mouser Part Number 80-C0805C224K3R -> (none); Mouser Price/Stock https://www.mouser.co.uk/ProductDetail/KEMET/C0805C224K3RAC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 -> (none)
- R1, R19, R2, R5: value 50Ω -> 49.9Ω, 0.125W
- R15, R16: value CRCW06031K00FKEA, 1KΩ -> 1kΩ
- R3, R4: value 40K -> 10K
- R6, R9: value RCS0603150RJNEA, 150Ω -> 150Ω
Connections:
- net +12V: now also J1.1; no longer J1.2
- net GND: now also J1.2; no longer J1.1

Commit message: im fried
Parts:
- removed C11, C6: 4.7uF, 16V, SMV_Passives:Cap0805, symbol SMV_Custom:0603W475K250XD
- removed R19, R5: 49.9Ω, 0.125W, SMV_Passives:0805RESC2012X60N, symbol SMV_Custom:CRCW020149R9FNED
- C2: value 1uF,16V -> 4.7nF,16V; footprint SMV_Passives:Cap0805 -> SMV_Passives:CAPC17595_87N_KEM
- C3: value 1uF,16V -> 4.7F,16V; footprint SMV_Passives:Cap0805 -> SMV_Passives:CAPC17595_87N_KEM
Connections:
- net FB is gone; now on net ADC_IN1: U3.1 (VOUT), U3.4 (VIN-)
- net ADC_IN2: now also U4.1 (VOUT), U4.4 (VIN-)

Commit message: fuck
Parts:
- added Hall1, Hall2: HS1, TestPoint:TestPoint_Pad_D1.5mm, symbol Connector:TestPoint
- added TP1: TestPoint, SMV_Logo:SEM_logo, symbol Connector:TestPoint
- Brake Pedal1: renamed from J4
- Gas Pedal1: renamed from J5
- Q1, Q2: footprint LFPAK56_SOT669_NEX -> SMV_Transistors:LFPAK56_SOT669_NEX
- U1: footprint TSSOP20_PW_TEX -> SMV_ICs:TSSOP20_PW_TEX
- renumbered TP1 to 12V1, TP13 to 3.3V1, TP5 to 5V1, J2 to CAN1, J3 to CAN2, TP9 to CLKIN1, TP10 to CS1, TP15 to Drain1, TP17 to Drain2, TP2 to G1, TP14 to G2, TP3 to GND1, TP12 to H1, TP11 to H2, J7 to Horn1, TP7 to MISO1, TP6 to MOSI1, J8 to Power1, TP8 to SCK1, TP4 to Test1, J6 to Wiper1
Connections:
- net ADC_IN1: now also Hall1.1
- net ADC_IN2: now also Hall2.1
