File: Nabeel's Joulemeter/Nabeel's Joulemeter.kicad_pcb (KiCad board)
At the start: 2 copper layers, 50 parts, among them J1 XT60-M, J2 XT60-M, J3 22035035, J4 22035035, U1 INA181A1QDBVRQ1, U2 PADS131M04QPWRQ1, U3 UA78M05QDCYRG4Q1, U4 MCP6286T-E/OT

Commit message: latest schematic and pcb draft
Parts:
- removed J2: XT60-M, SMV_Connectors:AMASS_XT60-M
- added C11: 470uF, 63V, SMV_Passives:Big_Chunky_Cap, F.Cu at (119.0, 88.5)
- added C9: 470uF, 63V, SMV_Passives:Big_Chunky_Cap, F.Cu at (101.5, 74.5)
- added J5: 430450200, SMV_Connectors:CONN_SD-43045-001_02_MOL, F.Cu at (125.5, 70.2)
- added R12: R_US, Resistor_THT:R_Axial_DIN0204_L3.6mm_D1.6mm_P1.90mm_Vertical, F.Cu at (126.6, 83.0)
- added R13: R_US, Resistor_THT:R_Axial_DIN0204_L3.6mm_D1.6mm_P1.90mm_Vertical, F.Cu at (101.1, 64.5)
- J1: value XT60-M -> 430450200; footprint SMV_Connectors:AMASS_XT60-M -> SMV_Connectors:CONN_SD-43045-001_02_MOL
- moved TP4 245.3 mm to (23.0, 33.5)
- moved TP15 195.3 mm to (31.0, 29.5)
- moved TP3 139.3 mm to (23.0, 29.5)
- moved C3 107.9 mm to (98.8, 96.3), turned to 180 degrees
- moved U1 99.3 mm to (102.6, 92.8), turned to 180 degrees
- moved R6 93.5 mm to (106.6, 93.3), turned to 180 degrees
- moved R1 92.7 mm to (102.6, 86.8), turned to 180 degrees
- moved J1 92.3 mm to (114.0, 70.7)
- moved R7 89.9 mm to (113.0, 108.1), turned to -90 degrees
- moved C2 88.6 mm to (109.9, 93.3), turned to 180 degrees
- moved C10 86.1 mm to (163.0, 79.5)
- moved U3 85.5 mm to (168.0, 84.0)
- moved R8 83.8 mm to (113.0, 104.5), turned to -90 degrees
- moved C1 82.9 mm to (173.0, 79.6)
- moved R4 75.9 mm to (97.0, 105.9), turned to 90 degrees
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Routing:
- net /SHUNT_TO_LOAD: track 6.37 -> 20.2 mm
- net +5V: track 0.00 -> 0.54 mm

Commit message: LFG BOARD DONE FR
Parts:
- added C12: 4.7uF, 100V, SMV_Passives:CAP_C2220C_2S_KEM, F.Cu at (136.0, 76.5)
- added C13: 4.7uF, 100V, SMV_Passives:CAP_C2220C_2S_KEM, F.Cu at (103.0, 77.5)
- TP1, TP10, TP11, TP12, TP13, TP14, TP15, TP16, TP17, TP18, TP2, TP3, TP4, TP5, TP6, TP7, TP8, TP9: footprint TestPoint:TestPoint_Pad_D2.0mm -> TestPoint:TestPoint_Pad_D1.0mm
- moved TP15 161.6 mm to (150.5, 138.2)
- moved TP16 155.1 mm to (145.5, 138.2)
- moved TP4 154.3 mm to (170.0, 80.5)
- moved TP7 132.7 mm to (133.5, 100.5)
- moved TP8 130.5 mm to (128.5, 107.5)
- moved TP9 130.4 mm to (133.5, 104.8)
- moved TP10 129.8 mm to (133.5, 107.8)
- moved TP5 124.8 mm to (133.5, 95.5)
- moved TP3 124.8 mm to (134.0, 86.5)
- moved TP6 124.1 mm to (133.5, 98.0)
- moved TP1 110.9 mm to (105.4, 95.5)
- moved TP13 109.7 mm to (92.8, 112.0)
- moved TP14 106.9 mm to (97.0, 109.5), turned to 90 degrees
- moved TP12 104.8 mm to (108.5, 107.5)
- moved TP17 104.5 mm to (111.1, 104.7), turned to 90 degrees
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Connections:
- net /CAN_H renamed /CAN_P
- net /CAN_L renamed /CAN_N
- C11 pad 3: (no net) -> Net-(C11-Pad2)
- C11 pad 4: (no net) -> +12V
- C9 pad 3: (no net) -> /SHUNT_TO_LOAD
- C9 pad 4: (no net) -> Net-(C9-Pad1)
Routing:
- net +3.3V: track 0.00 -> 84.1 mm, vias 0 -> 2
- net +12V: track 6.37 -> 90.5 mm
- net /CAN_P: track 0.00 -> 63.2 mm
- net /CAN_N: track 0.00 -> 63.2 mm
- net GND: track 0.00 -> 46.2 mm, vias 0 -> 46
- net /SHUNT_TO_LOAD: track 20.2 -> 64.3 mm
- net /SCK: track 0.00 -> 30.0 mm
- net +5V: track 0.54 -> 25.1 mm
- net /CS: track 0.00 -> 23.3 mm
- net /GPIO_CLKIN: track 0.00 -> 23.2 mm
- net /MOSI: track 0.00 -> 21.4 mm
- net /MISO: track 0.00 -> 19.6 mm
- net /GPIO_RESET: track 0.00 -> 18.8 mm
- net /DIVIDED_VOLTAGE: track 0.00 -> 13.1 mm
- net Net-(R6-Pad2): track 0.00 -> 10.9 mm
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- added copper zone on B.Cu, net +3.3V
- added copper zone on B.Cu, net GND
- added copper zone on F.Cu, net GND

Commit message: made some changes
Parts:
- moved TP4 2.59 mm to (170.0, 83.1)
- moved C1 1.78 mm to (169.7, 78.9)
Routing:
- net +5V: track 25.1 -> 28.6 mm
- net +12V: track 90.5 -> 93.1 mm
- net +3.3V: track 84.1 -> 86.0 mm
- net GND: track 46.2 -> 47.7 mm
Other:
- board outline added: 89.5 x 84.5 mm
Changed lines of the file:
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@@
 		(tags "Capacitor")
 		(property "Reference" "C3"
-			(at 3.5 0 90)
+			(at -0.5485 -2 180)
 			(layer "F.SilkS")
 			(effects
@@
 		)
 		(property "Footprint" "SMV_Connectors:CONN_SD-43045-001_02_MOL"
-			(at 0 0 0)
+			(at -0.508 5.588 0)
 			(layer "F.Fab")
 			(hide yes)
@@
 		(sheetfile "Nabeel's Joulemeter.kicad_sch")
 		(attr through_hole)
-		(fp_circle
-			(center 4.3434 0)
-			(end 4.7244 0)
-			(stroke
-				(width 0.508)
-				(type solid)
-			)
-			(fill none)
-			(layer "B.SilkS")
-		)
 		(fp_line
 			(start -3.7084 -1.117)
@@
 			(layer "F.SilkS")
 		)
-		(fp_circle
-			(center 4.3434 0)
-			(end 4.7244 0)
-			(stroke
-				(width 0.508)
-				(type solid)
-			)
-			(fill none)
-			(layer "F.SilkS")
-		)
 		(fp_line
 			(start -3.8354 -4.041399)
@@
 			(layer "F.Fab")
 		)
+		(pad "" np_thru_hole circle
+			(at 0 4.320002)
+			(size 3.048 3.048)
+			(drill 3.048)
+			(layers "F&B.Cu" "*.Mask")
+		)
 		(pad "1" thru_hole circle
 			(at 0 0)
@@
 			(pintype "unspecified")
 		)
-		(pad "3" thru_hole circle
-			(at 0 4.320002)
-			(size 3.048 3.048)
-			(drill 3.048)
-			(layers "*.Cu" "*.Mask")
-			(remove_unused_layers no)
-		)
 	)
 	(footprint "TestPoint:TestPoint_Pad_D1.0mm"
@@
 	(footprint "SMV_Passives:Cap0805"
 		(layer "F.Cu")
-		(at 170 77.1 90)
+		(at 169.72 78.86 90)
 		(descr "C0805")
 		(tags "Capacitor")
@@
 		)
 		(property "Footprint" "SMV_Passives:CAP_C2220C_2S_KEM"
-			(at 0 0 360)
+			(at 0 0 0)
 			(layer "F.Fab")
 			(hide yes)
@@
 		)
 		(property "Datasheet" "C2220C475M1R2C7186"
-			(at 0 0 360)
+			(at 0 0 0)
 			(layer "F.Fab")
 			(hide yes)
@@
 		)
 		(property "Description" ""
-			(at 0 0 360)
+			(at 0 0 0)
 			(layer "F.Fab")
 			(hide yes)
@@
 		(sheetfile "Nabeel's Joulemeter.kicad_sch")
 		(attr through_hole)
-		(fp_circle
-			(center 4.3434 0)
-			(end 4.7244 0)
-			(stroke
-				(width 0.508)
-				(type solid)
-			)
-			(fill none)
-			(layer "B.SilkS")
-		)
 		(fp_line
 			(start -3.7084 -1.117)
@@
 			(layer "F.SilkS")
 		)
-		(fp_circle
-			(center 4.3434 0)
-			(end 4.7244 0)
-			(stroke
-				(width 0.508)
-				(type solid)
-			)
-			(fill none)
-			(layer "F.SilkS")
-		)
 		(fp_line
 			(start -3.8354 -4.041399)
@@
 			(layer "F.Fab")
 		)
+		(pad "" np_thru_hole circle
+			(at 0 4.320002)
+			(size 3.048 3.048)
+			(drill 3.048)
+			(layers "F&B.Cu" "*.Mask")
+		)
 		(pad "1" thru_hole circle
 			(at 0 0)
@@
 			(pintype "unspecified")
 		)
-		(pad "3" thru_hole circle
-			(at 0 4.320002)
-			(size 3.048 3.048)
-			(drill 3.048)
-			(layers "*.Cu" "*.Mask")
-			(remove_unused_layers no)
-		)
 	)
 	(footprint "SMV_Passives:Big_Chunky_Cap"
@@
 	(footprint "TestPoint:TestPoint_Pad_D1.0mm"
 		(layer "F.Cu")
-		(at 170 80.5)
+		(at 170.01 83.09)
 		(descr "SMD pad as test Point, diameter 1.0mm")
 		(tags "test point SMD pad")
@@
 	(gr_poly
 		(pts
-			(xy 170 78) (xy 167.5 80) (xy 167.5 80.5) (xy 170 80.5)
+			(xy 116.75 107.75) (xy 115.5 108.25) (xy 115.5 107.5)
 		)
 		(stroke
@@
 		(fill solid)
 		(layer "F.Cu")
-		(net 2)
+		(net 1)
 	)
 	(gr_poly
 		(pts
-			(xy 116.75 107.75) (xy 115.5 108.25) (xy 115.5 107.5)
+			(xy 116.75 110.25) (xy 115.75 110.75) (xy 115.75 110.25)
 		)
 		(stroke
@@
 		(end 178 142)
 		(stroke
-			(width 0.2)
+			(width 0.05)
 			(type default)
 		)
 		(fill none)
-		(layer "F.Cu")
-	)
-	(gr_poly
-		(pts
-			(xy 116.75 110.25) (xy 115.75 110.75) (xy 115.75 110.25)
-		)
-		(stroke
-			(width 0.2)
-			(type solid)
-		)
-		(fill solid)
-		(layer "F.Cu")
-		(net 1)
+		(layer "Edge.Cuts")
 	)
 	(segment
@@
 	)
 	(segment
-		(start 135.75 81)
-		(end 138.4765 78.2735)
-		(width 1)
-		(layer "F.Cu")
-		(net 1)
-	)
-	(segment
 		(start 115.600001 110.25)
 		(end 115.5 110.149999)
@@
 	)
 	(segment
-		(start 112.75 115)
-		(end 112.682 114.932)
+		(start 102.25 97.75)
+		(end 102.143651 97.643651)
 		(width 0.2)
 		(layer "F.Cu")
@@
 	)
 	(segment
-		(start 102.25 97.75)
-		(end 102.143651 97.643651)
+		(start 112.826999 114)
+		(end 112.682 113.855001)
 		(width 0.2)
 		(layer "F.Cu")
@@
 	)
 	(segment
-		(start 112.682 114.932)
-		(end 112.682 113.855001)
-		(width 0.2)
-		(layer "F.Cu")
-		(net 1)
-	)
-	(segment
 		(start 97.5 101.195151)
 		(end 97.5515 101.143651)
@@
 	)
 	(segment
+		(start 138.4765 79.5235)
+		(end 138.4765 76.5)
+		(width 1)
+		(layer "F.Cu")
+		(net 1)
+	)
+	(segment
 		(start 165 82)
 		(end 165 86.5)
@@
 	)
 	(segment
+		(start 137 81)
+		(end 138.4765 79.5235)
+		(width 1)
+		(layer "F.Cu")
+		(net 1)
+	)
+	(segment
 		(start 120.25 101.75)
 		(end 121.380501 101.75)
@@
 	)
 	(segment
-		(start 138.4765 78.2735)
-		(end 138.4765 76.5)
-		(width 1)
+		(start 114.5 114)
+		(end 112.826999 114)
+		(width 0.2)
 		(layer "F.Cu")
 		(net 1)
@@
 		(net 1)
 	)
+	(segment
+		(start 135.75 81)
+		(end 137 81)
+		(width 1)
+		(layer "F.Cu")
+		(net 1)
+	)
 	(via
 		(at 157.5 64.25)
@@
 	)
 	(via
-		(at 112.75 115)
+		(at 114.5 114)
 		(size 0.6)
 		(drill 0.3)
@@
 	)
 	(segment
+		(start 169.72 79.76)
+		(end 169.95 79.99)
+		(width 1)
+		(layer "F.Cu")
+		(net 2)
+	)
+	(segment
 		(start 157.8835 100.6165)
 		(end 157.8835 100.62)
@@
 	)
 	(segment
-		(start 170 88.5035)
+		(start 169.4 80.08)
+		(end 169.72 79.76)
+		(width 1)
+		(layer "F.Cu")
+		(net 2)
+	)
+	(segment
+		(start 167.4957 80.08)
+		(end 169.4 80.08)
+		(width 1)
+		(layer "F.Cu")
+		(net 2)
+	)
+	(segment
+		(start 167.3114 80.2643)
+		(end 167.4957 80.08)
+		(width 0.8)
+		(layer "F.Cu")
+		(net 2)
+	)
+	(segment
+		(start 169.95 88.5535)
 		(end 157.8835 100.62)
 		(width 1)
@@
 	)
 	(segment
-		(start 170 80.5)
-		(end 170 88.5035)
+		(start 169.95 79.99)
+		(end 169.95 88.5535)
 		(width 1)
 		(layer "F.Cu")
@@
 	)
 	(segment
+		(start 121.4 105.39)
+		(end 121.4055 105.3845)
+		(width 0.5)
+		(layer "F.Cu")
+		(net 3)
+	)
+	(segment
 		(start 122 97.25)
 		(end 126.21 97.25)
@@
 		(start 115.5 104.425)
 		(end 115.5 105.5)
-		(width 0.6)
+		(width 0.55)
 		(layer "F.Cu")
 		(net 3)
@@
 	)
 	(segment
+		(start 121.4055 105.3845)
+		(end 121.4055 103.525001)
+		(width 0.5)
+		(layer "F.Cu")
+		(net 3)
+	)
+	(segment
 		(start 121.380499 103.5)
 		(end 121.4055 103.525001)
@@
 		(start 116.5 103.425)
 		(end 115.5 104.425)
-		(width 0.6)
+		(width 0.55)
 		(layer "F.Cu")
 		(net 3)
@@
 	)
 	(segment
-		(start 159.965052 80.25)
-		(end 160 80.284948)
-		(width 1)
+		(start 160 80.284948)
+		(end 162.667952 80.284948)
+		(width 0.9)
 		(layer "F.Cu")
 		(net 7)
@@
 	)
 	(segment
+		(start 162.667952 80.284948)
+		(end 162.6886 80.2643)
+		(width 0.2)
+		(layer "F.Cu")
+		(net 7)
+	)
+	(segment
 		(start 132.5 84.3)
 		(end 132.5 88.52)
@@
 	)
 	(segment
+		(start 105.4765 80.0235)
+		(end 105.4765 77.5)
+		(width 1)
+		(layer "F.Cu")
+		(net 11)
+	)
+	(segment
 		(start 95 99.5)
 		(end 95 106.327797)
@@
 	)
 	(segment
+		(start 99 86.5)
+		(end 105.4765 80.0235)
+		(width 1)
+		(layer "F.Cu")
+		(net 11)
+	)
+	(segment
 		(start 100.75 91.5)
 		(end 99.775001 90.525001)
@@
 	)
 	(segment
-		(start 98.5 86.5)
-		(end 105.4765 79.5235)
+		(start 95.75 86.5)
+		(end 99 86.5)
 		(width 1)
 		(layer "F.Cu")
@@
 	)
 	(segment
+		(start 95.75 88.504851)
+		(end 95.75 86.5)
+		(width 1)
+		(layer "F.Cu")
+		(net 11)
+	)
+	(segment
 		(start 99.775001 90.525001)
 		(end 97.77015 90.525001)
@@
 	)
 	(segment
-		(start 95.75 88.504851)
-		(end 95.75 86.5)
-		(width 1)
-		(layer "F.Cu")
-		(net 11)
-	)
-	(segment
-		(start 105.4765 79.5235)
-		(end 105.4765 77.5)
-		(width 1)
-		(layer "F.Cu")
-		(net 11)
-	)
-	(segment
 		(start 98.9055 95.5945)
 		(end 95 99.5)
@@
 		(width 1)
 		(layer "F.Cu")
-		(net 11)
-	)
-	(segment
-		(start 95.75 86.5)
-		(end 98.5 86.5)
-		(width 1)
-		(layer "F.Cu")

Commit message: almost final
Parts:
- added H1: MountingHole, MountingHole:MountingHole_3.2mm_M3, F.Cu at (167.5, 65.8)
- added H2: MountingHole, MountingHole:MountingHole_3.2mm_M3, F.Cu at (97.8, 65.8)
- added H3: MountingHole, MountingHole:MountingHole_3.2mm_M3, F.Cu at (167.5, 134.0)
- added H4: MountingHole, MountingHole:MountingHole_3.2mm_M3, F.Cu at (97.8, 134.0)
- moved TP1 22.2 mm to (125.0, 85.0)
- moved TP2 14.9 mm to (109.0, 84.5)
- moved C3 12.1 mm to (110.5, 100.5)
- moved R1 10.6 mm to (113.0, 90.0)
- moved TP18 10.3 mm to (116.6, 98.1)
- moved U1 10.3 mm to (112.6, 97.0)
- moved TP9 9.39 mm to (128.8, 112.9)
- moved TP8 7.48 mm to (134.4, 102.9)
- moved C9 5.34 mm to (107.7, 68.5)
- moved J1 5.14 mm to (118.7, 68.5)
- moved C13 5.10 mm to (107.8, 79.3)
- moved R3 5.05 mm to (100.0, 106.6)
- moved R4 5.04 mm to (100.0, 110.2)
- moved TP14 5.01 mm to (102.0, 109.2)
- moved C2 5.00 mm to (118.0, 105.8)
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Connections:
- C11 pad 3: Net-(C11-Pad2) -> (no net)
- C11 pad 4: +12V -> (no net)
- C9 pad 3: /SHUNT_TO_LOAD -> (no net)
- C9 pad 4: Net-(C9-Pad1) -> (no net)
Routing:
- net GND: track 47.7 -> 33.7 mm, vias 46 -> 45
- net +12V: track 93.1 -> 82.0 mm
- net /SHUNT_TO_LOAD: track 64.6 -> 54.4 mm
- net +3.3V: track 86.0 -> 77.7 mm, vias 2 -> 3
- net /GPIO_RESET: track 18.8 -> 13.8 mm
- net Net-(R6-Pad2): track 10.9 -> 7.06 mm
- net /SCK: track 30.0 -> 26.7 mm
- net /CS: track 23.3 -> 20.4 mm
- net /MISO: track 19.6 -> 17.3 mm
- net /MOSI: track 21.4 -> 19.4 mm
- net Net-(C11-Pad2): track 7.01 -> 5.21 mm
- net /GPIO_CLKIN: track 23.2 -> 21.6 mm
- net Net-(C9-Pad1): track 8.24 -> 7.26 mm
Other:
- board size 89.5 x 84.5 mm -> 80 x 79.1 mm

Commit message: Finalized!
Parts:
- added REF**: SEM_logo, SMV_Logo:SEM_logo, F.Cu at (116.0, 120.7)
- moved H3 2.80 mm to (169.3, 136.2)
- moved H4 2.18 mm to (97.4, 136.2)
- moved H1 1.82 mm to (169.2, 65.2)
- moved H2 0.64 mm to (97.4, 65.2)
- renumbered J5 to 12V_IN, J1 to 12V_OUT, TP4 to 5V, J3 to CAN, J4 to CAN, TP15 to CAN_N, TP16 to CAN_P, TP5 to CLKIN, TP9 to CS, TP11 to FEEDBACK, TP13 to GND, TP2 to LOAD, TP7 to MISO, TP6 to MOSI, TP17 to RC1, TP12 to RC2, TP10 to RESET, TP8 to SCK, TP18 to SENSE_OUT, TP14 to V_DIV
Other:
- board text added: "Nabeel Sonaseth 1/27/25 Low Power Joulemeter"

Commit message: fml
Parts:
- C10: value C1210C474K5RACTU, 0.47uF -> 0.47uF, 50V; footprint SMV_Passives:CAPC340270_105N_KEM -> SMV_Passives:Cap0805
- C12, C13: footprint SMV_Passives:CAP_C2220C_2S_KEM -> SMV_Passives:CAPC340180_180N_KEM
- C2: value C0603C472K4RACTU, 4700pF -> 4.7nF
- C4, C5: value 1uF,16V -> 1uF,50V
- C6: value GCM188R71H104KA57D, 220nF -> 220nF, 16V; footprint SMV_Passives:0805RESC2012X60N -> SMV_Passives:Cap0805
- C8: value C1808C472KGRACTU, 4700pF -> 4.7nF; footprint SMV_Passives:CAPC520220_215N_KEM -> SMV_Passives:CAPC17595_87N_KEM
- R10, R11, R9: value RCS0603150RJNEA, 150Ω -> 150Ω, 0.125W
- R2: value 10k -> 10kohms, 0.5W
- R3: value TNPW0805505KBEEA -> 51kohms
- R4: value TNPW0805101KBEEA -> 10kohms
- R5, R6: value CRCW020149R9FNED, 50Ω -> 49.9ohms, 0.125W
- moved C5 0.71 mm to (125.7, 102.6)
- moved C6 0.20 mm to (129.1, 105.6)
- renumbered 12V_OUT to J1, CAN to J3, CAN to J4, 12V_IN to J5, RESET to TP10, FEEDBACK to TP11, RC2 to TP12, GND to TP13, V_DIV to TP14, CAN_N to TP15, CAN_P to TP16, RC1 to TP17, SENSE_OUT to TP18, LOAD to TP2, 5V to TP4, CLKIN to TP5, MOSI to TP6, MISO to TP7, SCK to TP8, CS to TP9
Connections:
- C11 pad 3: (no net) -> Net-(C11-Pad2)
- C11 pad 4: (no net) -> +12V
- C9 pad 3: (no net) -> /SHUNT_TO_LOAD
Routing:
- net /DIVIDED_VOLTAGE: track 12.7 -> 15.4 mm
- net +12V: track 82.0 -> 82.5 mm

Commit message: hello
Parts:
- moved C13 1.06 mm to (108.8, 79.3)
- renumbered TP1 to 12V, J5 to 12V, TP3 to 3.3V, TP4 to 5V, J3 to CAN, J4 to CAN, TP15 to CAN_N, TP16 to CAN_P, TP5 to CLKIN, TP9 to CS, TP11 to FEEDBACK, TP13 to GND, J1 to Load, TP7 to MISO, TP6 to MOSI, TP10 to RST, TP8 to SCK, TP17 to SENSE, TP18 to SENSE_OUT, TP14 to V_DIV, TP12 to V_SENSE, TP2 to shunt_load
Connections:
- C9 pad 4: (no net) -> Net-(C9-Pad1)
Routing:
- net GND: track 33.9 -> 30.2 mm

Commit message: almost...
Parts:
- removed REF**: SEM_logo, SMV_Logo:SEM_logo
- added TP1: TestPoint, SMV_Logo:SEM_logo, F.Cu at (116.2, 120.6)
- renumbered 12V to 12V1, 12V to 12V2, 3.3V to 3.3V1, 5V to 5V1, CAN to CAN1, CAN to CAN2, CAN_N to CAN_N1, CAN_P to CAN_P1, CLKIN to CLKIN1, CS to CS1, FEEDBACK to FEEDBACK1, GND to GND1, Load to Load1, MISO to MISO1, MOSI to MOSI1, RST to RST1, SCK to SCK1, SENSE to SENSE1, SENSE_OUT to SENSE_OUT1, V_DIV to V_DIV1, V_SENSE to V_SENSE1, shunt_load to shunt_load1
Connections:
- C11 pad 3: Net-(C11-Pad2) -> (no net)
- C11 pad 4: +12V -> (no net)
- C9 pad 3: /SHUNT_TO_LOAD -> (no net)
- C9 pad 4: Net-(C9-Pad1) -> (no net)
