File: Nabeel's Joulemeter/Nabeel's Joulemeter.kicad_sch (KiCad schematic)
At the start: 60 parts, among them J1 430450200, J3 22035035, J4 22035035, J5 430450200, U1 INA181A1QDBVRQ1, U2 PADS131M04QPWRQ1, U3 UA78M05QDCYRG4Q1, U4 MCP6286T-E/OT

Commit message: almost...
Parts:
- added TP1: TestPoint, SMV_Logo:SEM_logo, symbol Connector:TestPoint
- R1: footprint WSR -> SMV_Passives:WSR
- renumbered J5 to 12V1, TP1 to 12V2, TP3 to 3.3V1, TP4 to 5V1, J3 to CAN1, J4 to CAN2, TP15 to CAN_N1, TP16 to CAN_P1, TP5 to CLKIN1, TP9 to CS1, TP11 to FEEDBACK1, TP13 to GND1, J1 to Load1, TP7 to MISO1, TP6 to MOSI1, TP10 to RST1, TP8 to SCK1, TP17 to SENSE1, TP18 to SENSE_OUT1, TP14 to V_DIV1, TP12 to V_SENSE1, TP2 to shunt_load1
Changed lines of the file:
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@@
 		(on_board yes)
 		(dnp no)
-		(property "Reference" "TP8"
+		(property "Reference" "SCK1"
 			(at 262.89 138.557 90)
 			(effects
@@
 			(project "Nabeel's Joulemeter"
 				(path "/5be733cb-4188-4a93-804c-a0c5e134cfd0"
-					(reference "TP8")
+					(reference "SCK1")
 					(unit 1)
 				)
@@
 		(on_board yes)
 		(dnp no)
-		(property "Reference" "J5"
+		(property "Reference" "12V1"
 			(at 48.895 80.0099 0)
 			(effects
@@
 			(project ""
 				(path "/5be733cb-4188-4a93-804c-a0c5e134cfd0"
-					(reference "J5")
+					(reference "12V1")
 					(unit 1)
 				)
@@
 		(dnp no)
 		(fields_autoplaced yes)
-		(property "Reference" "TP16"
+		(property "Reference" "CAN_P1"
 			(at 80.518 182.88 90)
 			(effects
@@
 			(project ""
 				(path "/5be733cb-4188-4a93-804c-a0c5e134cfd0"
-					(reference "TP16")
+					(reference "CAN_P1")
 					(unit 1)
 				)
@@
 		(on_board yes)
 		(dnp no)
-		(property "Reference" "TP9"
+		(property "Reference" "CS1"
 			(at 262.89 143.637 90)
 			(effects
@@
 			(project "Nabeel's Joulemeter"
 				(path "/5be733cb-4188-4a93-804c-a0c5e134cfd0"
-					(reference "TP9")
+					(reference "CS1")
 					(unit 1)
 				)
@@
 			)
 		)
-		(property "Footprint" "WSR"
+		(property "Footprint" "SMV_Passives:WSR"
 			(at 233.045 52.705 0)
 			(effects
@@
 			)
 		)
-		(property "Description" ""
+		(property "Description" "C499500"
 			(at 233.045 52.705 0)
 			(effects
@@
 		(dnp no)
 		(fields_autoplaced yes)
-		(property "Reference" "J4"
+		(property "Reference" "CAN2"
 			(at 159.385 186.6899 0)
 			(effects
@@
 			(project "Nabeel's Joulemeter"
 				(path "/5be733cb-4188-4a93-804c-a0c5e134cfd0"
-					(reference "J4")
+					(reference "CAN2")
 					(unit 1)
 				)
@@
 		(dnp no)
 		(fields_autoplaced yes)
-		(property "Reference" "TP15"
+		(property "Reference" "CAN_N1"
 			(at 100.965 185.4199 90)
 			(effects
@@
 			(project ""
 				(path "/5be733cb-4188-4a93-804c-a0c5e134cfd0"
-					(reference "TP15")
+					(reference "CAN_N1")
 					(unit 1)
 				)
@@
 		(on_board yes)
 		(dnp no)
-		(property "Reference" "TP1"
+		(property "Reference" "12V2"
 			(at 215.519 51.181 90)
 			(effects
@@
 			(project ""
 				(path "/5be733cb-4188-4a93-804c-a0c5e134cfd0"
-					(reference "TP1")
+					(reference "12V2")
 					(unit 1)
 				)
@@
 	)
 	(symbol
+		(lib_name "TestPoint_1")
+		(lib_id "Connector:TestPoint")
+		(at 118.11 105.41 0)
+		(unit 1)
+		(exclude_from_sim no)
+		(in_bom yes)
+		(on_board yes)
+		(dnp no)
+		(fields_autoplaced yes)
+		(property "Reference" "TP1"
+			(at 120.65 100.8379 0)
+			(effects
+				(font
+					(size 1.27 1.27)
+				)
+				(justify left)
+			)
+		)
+		(property "Value" "TestPoint"
+			(at 120.65 103.3779 0)
+			(effects
+				(font
+					(size 1.27 1.27)
+				)
+				(justify left)
+			)
+		)
+		(property "Footprint" "SMV_Logo:SEM_logo"
+			(at 123.19 105.41 0)
+			(effects
+				(font
+					(size 1.27 1.27)
+				)
+				(hide yes)
+			)
+		)
+		(property "Datasheet" "~"
+			(at 123.19 105.41 0)
+			(effects
+				(font
+					(size 1.27 1.27)
+				)
+				(hide yes)
+			)
+		)
+		(property "Description" "test point"
+			(at 118.11 105.41 0)
+			(effects
+				(font
+					(size 1.27 1.27)
+				)
+				(hide yes)
+			)
+		)
+		(pin "1"
+		)
+		(instances
+			(project ""
+				(path "/5be733cb-4188-4a93-804c-a0c5e134cfd0"
+					(reference "TP1")
+					(unit 1)
+				)
+			)
+		)
+	)
+	(symbol
 		(lib_id "power:GND")
 		(at 112.395 64.135 180)
@@
 		(dnp no)
 		(fields_autoplaced yes)
-		(property "Reference" "TP17"
+		(property "Reference" "SENSE1"
 			(at 264.795 67.9449 90)
 			(effects
@@
 			(project ""
 				(path "/5be733cb-4188-4a93-804c-a0c5e134cfd0"
-					(reference "TP17")
+					(reference "SENSE1")
 					(unit 1)
 				)
@@
 		(on_board yes)
 		(dnp no)
-		(property "Reference" "TP7"
+		(property "Reference" "MISO1"
 			(at 262.89 136.017 90)
 			(effects
@@
 			(project "Nabeel's Joulemeter"
 				(path "/5be733cb-4188-4a93-804c-a0c5e134cfd0"
-					(reference "TP7")
+					(reference "MISO1")
 					(unit 1)
 				)
@@
 		(on_board yes)
 		(dnp no)
-		(property "Reference" "TP5"
+		(property "Reference" "CLKIN1"
 			(at 262.89 130.8099 90)
 			(effects
@@
 			(project ""
 				(path "/5be733cb-4188-4a93-804c-a0c5e134cfd0"
-					(reference "TP5")
+					(reference "CLKIN1")
 					(unit 1)
 				)
@@
 		(on_board yes)
 		(dnp no)
-		(property "Reference" "TP2"
+		(property "Reference" "shunt_load1"
 			(at 268.351 48.387 90)
 			(effects
@@
 			(project "Nabeel's Joulemeter"
 				(path "/5be733cb-4188-4a93-804c-a0c5e134cfd0"
-					(reference "TP2")
+					(reference "shunt_load1")
 					(unit 1)
 				)
@@
 		(on_board yes)
 		(dnp no)
-		(property "Reference" "J1"
+		(property "Reference" "Load1"
 			(at 75.946 102.108 0)
 			(effects
@@
 			(project "Nabeel's Joulemeter"
 				(path "/5be733cb-4188-4a93-804c-a0c5e134cfd0"
-					(reference "J1")
+					(reference "Load1")
 					(unit 1)
 				)
@@
 		(on_board yes)
 		(dnp no)
-		(property "Reference" "TP3"
+		(property "Reference" "3.3V1"
 			(at 49.276 118.237 0)
 			(effects
@@
 			(project ""
 				(path "/5be733cb-4188-4a93-804c-a0c5e134cfd0"
-					(reference "TP3")
+					(reference "3.3V1")
 					(unit 1)
 				)
@@
 		(on_board yes)
 		(dnp no)
-		(property "Reference" "TP18"
+		(property "Reference" "SENSE_OUT1"
 			(at 212.598 28.194 0)
 			(effects
@@
 			(project "Nabeel's Joulemeter"
 				(path "/5be733cb-4188-4a93-804c-a0c5e134cfd0"
-					(reference "TP18")
+					(reference "SENSE_OUT1")
 					(unit 1)
 				)
@@
 		(dnp no)
 		(fields_autoplaced yes)
-		(property "Reference" "TP4"
+		(property "Reference" "5V1"
 			(at 104.648 74.93 90)
 			(effects
@@
 			(project ""
 				(path "/5be733cb-4188-4a93-804c-a0c5e134cfd0"
-					(reference "TP4")
+					(reference "5V1")
 					(unit 1)
 				)
@@
 		(dnp no)
 		(fields_autoplaced yes)
-		(property "Reference" "TP11"
+		(property "Reference" "FEEDBACK1"
 			(at 120.015 42.6719 0)
 			(effects
@@
 			(project ""
 				(path "/5be733cb-4188-4a93-804c-a0c5e134cfd0"
-					(reference "TP11")
+					(reference "FEEDBACK1")
 					(unit 1)
 				)
@@
 		(dnp no)
 		(fields_autoplaced yes)
-		(property "Reference" "J3"
+		(property "Reference" "CAN1"
 			(at 159.385 174.6249 0)
 			(effects
@@
 			(project ""
 				(path "/5be733cb-4188-4a93-804c-a0c5e134cfd0"
-					(reference "J3")
+					(reference "CAN1")
 					(unit 1)
 				)
@@
 		(dnp no)
 		(fields_autoplaced yes)
-		(property "Reference" "TP12"
+		(property "Reference" "V_SENSE1"
 			(at 150.495 28.4479 0)
 			(effects
@@
 			(project ""
 				(path "/5be733cb-4188-4a93-804c-a0c5e134cfd0"
-					(reference "TP12")
+					(reference "V_SENSE1")
 					(unit 1)
 				)
@@
 		(dnp no)
 		(fields_autoplaced yes)
-		(property "Reference" "TP14"
+		(property "Reference" "V_DIV1"
 			(at 29.845 45.2119 0)
 			(effects
@@
 			(project ""
 				(path "/5be733cb-4188-4a93-804c-a0c5e134cfd0"
-					(reference "TP14")
+					(reference "V_DIV1")
 					(unit 1)
 				)
@@
 		(on_board yes)
 		(dnp no)
-		(property "Reference" "TP10"
+		(property "Reference" "RST1"
 			(at 262.89 146.177 90)
 			(effects
@@
 			(project "Nabeel's Joulemeter"
 				(path "/5be733cb-4188-4a93-804c-a0c5e134cfd0"
-					(reference "TP10")
+					(reference "RST1")
 					(unit 1)
 				)
@@
 		(dnp no)
 		(fields_autoplaced yes)
-		(property "Reference" "TP13"
+		(property "Reference" "GND1"
 			(at 23.495 66.0399 90)
 			(effects
@@
 			(project ""
 				(path "/5be733cb-4188-4a93-804c-a0c5e134cfd0"
-					(reference "TP13")
+					(reference "GND1")
 					(unit 1)
 				)
@@
 		(on_board yes)
 		(dnp no)
-		(property "Reference" "TP6"
+		(property "Reference" "MOSI1"
 			(at 262.89 133.477 90)
 			(effects
@@
 			(project ""
 				(path "/5be733cb-4188-4a93-804c-a0c5e134cfd0"
-					(reference "TP6")
+					(reference "MOSI1")
 					(unit 1)
 				)
