File: safety_board/_autosave-safety_board.kicad_sch (KiCad schematic)
At the start: 74 parts, among them J1 430450200, J12 XT60-M, J13 XT60-M, J15 22035035, J18 XT60-M, J2 430450200, J3 22035035, J4 22035035, J5 22035035, J6 22035035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

Commit message: pcb
Changed lines of the file:
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@@
 	(wire
 		(pts
-			(xy 140.97 1.27) (xy 147.32 7.62)
+			(xy 140.97 -2.54) (xy 147.32 3.81)
 		)
 		(stroke
@@
 	(wire
 		(pts
-			(xy 147.32 7.62) (xy 147.32 25.4)
+			(xy 147.32 3.81) (xy 147.32 25.4)
 		)
 		(stroke
@@
 	(wire
 		(pts
-			(xy 129.54 1.27) (xy 140.97 1.27)
-		)
-		(stroke
-			(width 0)
-			(type default)
-		)
-	)
-	(wire
-		(pts
-			(xy 129.54 -26.67) (xy 129.54 1.27)
-		)
-		(stroke
+			(xy 129.54 -2.54) (xy 140.97 -2.54)
+		)
+		(stroke
+			(width 0)
+			(type default)
+		)
+	)
+	(wire
+		(pts
+			(xy 129.54 -26.67) (xy 129.54 -2.54)
+		)
+		(stroke
