File: safety_board/safety_board.kicad_pcb (KiCad board)
At the start: 2 copper layers, 74 parts, among them J1 430450200, J12 XT60-M, J13 XT60-M, J15 22035035, J18 XT60-M, J2 430450200, J3 22035035, J4 22035035, J5 22035035, J6 22035035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

Commit message: pcb almost done
Parts:
- removed R11: 10k ohms, SMV_Passives:RES_CRCW_0402
- removed U3: MCP6286T-E/OT, SMV_ICs:SOT-23-5_MC_MCH
- added R42: 5k ohms, SMV_Passives:RESC2012X50N, F.Cu at (75.7, 132.1)
- added R43: 5k ohms, SMV_Passives:RESC2012X50N, F.Cu at (76.1, 124.9)
- moved CR6 193.8 mm to (219.1, 100.6), turned to 180 degrees
- moved J13 189.5 mm to (174.8, 43.0), turned to 0 degrees
- moved U19 171.3 mm to (207.4, 93.3), turned to 0 degrees
- moved F3 162.8 mm to (167.1, 52.9), turned to 0 degrees
- moved F4 151.8 mm to (167.0, 60.2), turned to 0 degrees
- moved CR4 150.0 mm to (188.1, 100.7), turned to 180 degrees
- moved CR3 141.4 mm to (146.6, 58.9), turned to 180 degrees
- moved J12 136.9 mm to (233.8, 81.3), turned to -90 degrees
- moved U15 131.7 mm to (177.4, 93.3), turned to 0 degrees
- moved J6 76.8 mm to (64.7, 147.8), turned to 180 degrees
- moved U6 75.9 mm to (146.9, 93.2)
- moved CR8 73.4 mm to (157.5, 100.9)
- moved D1 68.6 mm to (103.9, 76.5), turned to 90 degrees
- moved R17 65.0 mm to (68.2, 142.6), turned to 0 degrees
- moved U14 63.3 mm to (94.1, 109.3)
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Connections:
- CR3 pad 1: Net-(J13-POS) -> Net-(U15-NO)
- J1 pad 1: /ESTOP1 -> +5V
- J1 pad 2: +3V3 -> Net-(J1-Pad2)
- J2 pad 1: /ESTOP2 -> +5V
- J2 pad 2: +3V3 -> Net-(J2-Pad2)
- J7 pad N: Net-(J7-NEG) -> GND
- J9 pad 1: Net-(U1-VIN) -> +12V
- J9 pad 2: +12V -> Net-(U1-VIN)
- U19 pad 4: Net-(J7-NEG) -> GND
- U6 pad 4: Net-(J7-NEG) -> GND
- U7 pad 5: /IGNITION_5V -> /IGNITION
Routing:
- net +12V: track 2.78 -> 217.1 mm
- net Net-(J12-POS): track 0.00 -> 114.1 mm
- net Net-(U15-COM): track 0.41 -> 95.9 mm
- net /CAN_H: track 0.00 -> 85.2 mm
- net Net-(J12-NEG): track 0.00 -> 75.8 mm
- net +5V: track 112.6 -> 183.9 mm, vias 1 -> 0
- net /CAN_L: track 0.00 -> 68.7 mm
- net /HSENSE_4: track 0.00 -> 60.9 mm
- net Net-(U15-NO): track 0.00 -> 60.5 mm
- net GND: track 0.74 -> 52.2 mm, vias 0 -> 14
- net /HSENSE_3: track 0.00 -> 48.3 mm
- net /DRAIN: track 129.0 -> 83.5 mm, vias 2 -> 1
- net /DRAIN2: track 124.4 -> 80.9 mm
- net /HSENSE_2: track 0.00 -> 37.7 mm
- net /IGNITION: track 6.42 -> 42.9 mm
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- added copper zone on B.Cu, net GND

Commit message: pcb
git commit -m pcb
Parts:
- F1, F2, F3, F4: value 3555-2 -> 3557-2; footprint SMV_Connectors:FUSE_3555-2 -> SMV_Connectors:FUSE_3557-2
- moved TP_48V1 3.65 mm to (63.9, 79.6)
- moved F2 0.68 mm to (82.3, 83.7)
- moved F1 0.36 mm to (82.0, 75.3)
Routing:
- net GND: track 52.2 -> 60.6 mm, vias 14 -> 18
- net Net-(J13-POS): track 18.1 -> 25.4 mm
- net Net-(J7-POS): track 21.1 -> 28.3 mm
- net +5V: track 183.9 -> 190.4 mm
- net Net-(U15-COM): track 95.9 -> 97.0 mm
- net Net-(U15-NO): track 60.5 -> 61.5 mm
- net /DRAIN: vias 1 -> 0
Other:
- board outline added: 201.2 x 121.8 mm

Commit message: maybe possibly final
Parts:
- removed CR3: 5KP48A, SMV_Passives:DIODE_P600_VIS
- added D3: SMA4S56AH, SMV_Passives:SODFL4725X110N, F.Cu at (153.2, 55.9)
- TP_48V1: footprint TestPoint:TestPoint_Pad_D1.0mm -> TestPoint:TestPoint_Pad_D2.0mm
- moved J9 24.7 mm to (200.4, 142.3), turned to 0 degrees
- moved TP_AND1 19.1 mm to (118.2, 114.4)
- moved J13 18.0 mm to (187.2, 56.2)
- moved TP_5V1 17.3 mm to (195.1, 142.7), turned to 90 degrees
- moved C3 15.1 mm to (193.6, 138.9), turned to 90 degrees
- moved C11 14.8 mm to (193.4, 142.1), turned to -90 degrees
- moved R18 14.7 mm to (120.5, 117.3)
- moved R4 14.7 mm to (120.5, 115.9)
- moved TS_CAN_L1 13.0 mm to (131.7, 137.1)
- moved TP_DRAIN1 11.4 mm to (121.1, 104.6)
- moved U2 10.8 mm to (121.0, 113.4)
- moved TS_CAN_H1 10.6 mm to (127.9, 138.8)
- moved F1 9.27 mm to (91.2, 74.3)
- moved F2 9.27 mm to (91.5, 82.8)
- moved TP_48V1 9.27 mm to (73.2, 78.7)
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Connections:
- net /CAN_H renamed /CAN_P
- net /CAN_L renamed /CAN_N
- C3 pad 1: Net-(U1-VIN) -> +12V
- J9 pad 2: Net-(U1-VIN) -> GND
- U1 pad 3: Net-(U1-VIN) -> +12V
Routing:
- net +12V: track 217.1 -> 236.4 mm
- net Net-(J13-NEG): track 57.5 -> 39.7 mm
- net Net-(U7-1Y): track 18.8 -> 5.33 mm
- net Net-(U15-NO): track 61.5 -> 51.9 mm
- net Net-(U1-VIN): track 8.90 -> 0.00 mm
- net Net-(U15-COM): track 97.0 -> 88.7 mm
- net /CAN_P: track 85.2 -> 77.0 mm
- net /CAN_N: track 68.7 -> 76.7 mm
- net Net-(J13-POS): track 25.4 -> 17.7 mm
- net Net-(J7-POS): track 28.3 -> 32.0 mm
- net Net-(U2-G): track 8.58 -> 4.86 mm
- net +5V: track 190.4 -> 186.9 mm
- net GND: track 60.6 -> 63.9 mm, vias 18 -> 41
- net /DRAIN: track 83.5 -> 81.3 mm
- net /DRAIN2: track 80.9 -> 79.9 mm
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Other:
- board size 201.2 x 121.8 mm -> 186.6 x 107.9 mm
