File: safety_board/safety_board.kicad_pcb (KiCad board)
At the start: 2 copper layers, 186.6 x 107.9 mm, 74 parts, among them J1 430450200, J12 XT60-M, J13 XT60-M, J15 22035035, J18 XT60-M, J2 430450200, J3 22035035, J4 22035035, J5 22035035, J6 22035035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

Commit message: yay
Parts:
- added H1: MountingHole, MountingHole:MountingHole_3.2mm_M3, F.Cu at (235.1, 53.6)
- added H2: MountingHole, MountingHole:MountingHole_3.2mm_M3, F.Cu at (59.5, 53.6)
- added H3: MountingHole, MountingHole:MountingHole_3.2mm_M3, F.Cu at (235.1, 148.9)
- added H4: MountingHole, MountingHole:MountingHole_3.2mm_M3, F.Cu at (58.9, 148.9)
- added TP1: TestPoint, SMV_Logo:SEM_logo, F.Cu at (222.4, 121.8)
- moved D3 33.5 mm to (186.6, 55.6)
- moved F3 33.5 mm to (200.6, 52.6)
- moved F4 33.5 mm to (200.4, 60.0)
- moved J13 33.5 mm to (220.6, 55.9)
- moved TP_12V1 18.3 mm to (201.0, 131.3)
- moved J4 4.03 mm to (95.4, 147.7)
- moved J5 4.03 mm to (82.2, 147.7)
- moved R10 4.03 mm to (74.8, 142.5)
- moved R14 4.03 mm to (109.8, 142.5)
- moved R15 4.03 mm to (96.7, 142.5)
- moved R16 4.03 mm to (85.0, 142.5)
- moved R17 4.03 mm to (72.3, 142.5)
- moved R8 4.03 mm to (99.4, 142.5)
- moved R9 4.03 mm to (87.6, 142.5)
- moved TP_HSENSE1 4.03 mm to (111.8, 140.0)
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Routing:
- net +12V: track 236.4 -> 25.6 mm
- net Net-(J12-POS): track 114.1 -> 0.00 mm
- net Net-(U15-NO): track 51.9 -> 0.00 mm
- net Net-(J13-NEG): track 39.7 -> 0.00 mm
- net Net-(J7-POS): track 32.0 -> 0.00 mm
- net Net-(U15-COM): track 88.7 -> 63.4 mm
- net Net-(J13-POS): track 17.7 -> 0.00 mm
- net +5V: track 186.9 -> 181.2 mm
- net GND: track 63.9 -> 58.5 mm, vias 41 -> 45
- net /HSENSE: track 26.6 -> 22.5 mm
- net /HSENSE_4: track 60.9 -> 56.9 mm
- net /HSENSE_3: track 48.3 -> 44.2 mm
- net /HSENSE_2: track 37.7 -> 33.6 mm
- net Net-(J12-NEG): track 75.8 -> 77.2 mm
- net +3V3: track 61.3 -> 62.0 mm
- added copper zone on F.Cu, net +12V
- added copper zone on F.Cu, net GND
Other:
- board text added: "12V"
- board text added: "CAN"
- board text added: "EStop"
- board text added: "H2_Sense"
- board text added: "H2_Shutdown_Valve"
- board text added: "HFC"
- board text added: "Motor Controller"
- board text added: "SuperCaps"

Commit message: yay
Parts:
- moved C6 40.4 mm to (127.4, 126.8), turned to 90 degrees
- moved TP1 13.0 mm to (225.6, 134.4)
Routing:
- net GND: track 58.5 -> 57.7 mm
Other:
- board text added: "Leo Chen 3/9/25 Safety Board"

Commit message: yay
Parts:
- removed R13: 10k ohms, SMV_Passives:RES_CRCW_0402
- added C4: 0.1uF,50V, SMV_Passives:Cap0805, F.Cu at (126.2, 133.5)
- added R3: 1.5k ohms, SMV_Passives:RES_CRCW_0402, F.Cu at (153.4, 116.0)
- added TP_48V2: V_DIVIDED, TestPoint:TestPoint_Pad_D2.0mm, F.Cu at (105.0, 82.8)
- added TP_48V3: V_DIVIDED, TestPoint:TestPoint_Pad_D2.0mm, F.Cu at (227.8, 80.6)
- added TP_48V4: V_DIVIDED, TestPoint:TestPoint_Pad_D2.0mm, F.Cu at (212.2, 61.8)
- added TP_48V5: V_DIVIDED, TestPoint:TestPoint_Pad_D2.0mm, F.Cu at (69.6, 99.4)
- added TP_48V6: V_DIVIDED, TestPoint:TestPoint_Pad_D2.0mm, F.Cu at (69.6, 106.8)
- added TP_AND2: TestPoint, TestPoint:TestPoint_Pad_D1.0mm, F.Cu at (118.4, 130.4)
- added TP_CAP_GATE_1: TestPoint, TestPoint:TestPoint_Pad_D1.0mm, F.Cu at (153.7, 113.4)
- added TP_INV1: TestPoint, TestPoint:TestPoint_Pad_D1.0mm, F.Cu at (123.4, 131.4)
- added TP_INV2: TestPoint, TestPoint:TestPoint_Pad_D1.0mm, F.Cu at (114.7, 139.3)
- added TP_INV3: TestPoint, TestPoint:TestPoint_Pad_D1.0mm, F.Cu at (112.9, 136.9)
- added TP_INV4: TestPoint, TestPoint:TestPoint_Pad_D1.0mm, F.Cu at (119.4, 132.4)
- added U3: SN74AHCT14QPWRQ1, SMV_ICs:PW14, F.Cu at (120.6, 136.4)
- moved TS_CAN_H1 54.1 mm to (182.0, 136.6)
- moved TS_CAN_L1 46.3 mm to (178.0, 136.5)
- moved TP_DRAIN2 10.7 mm to (164.8, 109.4)
- moved TP_HSENSE1 6.12 mm to (117.9, 140.8)
- moved CR1 3.55 mm to (107.0, 101.2)
- moved TP_HSENSE4 3.17 mm to (78.8, 139.3)
- moved U4 2.50 mm to (154.6, 110.4)
- moved U14 2.05 mm to (99.7, 109.3)
- moved TP1 1.71 mm to (224.0, 135.0)
- moved J15 0.54 mm to (127.5, 148.6)
Connections:
- U7 pad 10: /HSENSE_3 -> /INVERT3
- U7 pad 12: /HSENSE_2 -> /INVERT2
- U7 pad 13: /HSENSE -> /INVERT
- U7 pad 9: /HSENSE_4 -> /INVERT4
Routing:
- net /INVERT2: track 0.00 -> 15.5 mm
- net /CAN_P: track 77.0 -> 92.1 mm
- net /CAN_N: track 76.7 -> 91.7 mm
- net /INVERT3: track 0.00 -> 14.9 mm
- net GND: track 57.7 -> 68.0 mm, vias 45 -> 107
- net +3V3: track 62.0 -> 71.5 mm
- net /INVERT: track 0.00 -> 9.35 mm
- net /HSENSE_2: track 33.6 -> 24.4 mm
- net /INVERT4: track 0.00 -> 8.32 mm
- net /HSENSE_3: track 44.2 -> 36.6 mm
- net /HSENSE_4: track 56.9 -> 49.9 mm
- net Net-(U4-G): track 2.94 -> 5.63 mm
- net /DRAIN2: track 79.9 -> 77.2 mm
- net Net-(U7-1A): track 7.72 -> 10.3 mm
- net /DRAIN: track 81.3 -> 83.5 mm
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Other:
- board text added: "12V_INPUT"
- board text removed: "12V"

Commit message: holla
Parts:
- added R11: R, Resistor_SMD:R_0805_2012Metric, F.Cu at (81.4, 138.4)
- added R13: R, Resistor_SMD:R_0805_2012Metric, F.Cu at (93.4, 136.8)
- added R19: R, Resistor_SMD:R_0805_2012Metric, F.Cu at (102.6, 139.4)
- added R20: R, Resistor_SMD:R_0805_2012Metric, F.Cu at (114.8, 139.8)
- added R21: R, Resistor_SMD:R_0805_2012Metric, F.Cu at (124.8, 130.6)
- added R22: R, Resistor_SMD:R_0805_2012Metric, F.Cu at (118.4, 130.6)
- added R23: R, Resistor_SMD:R_0805_2012Metric, F.Cu at (120.6, 130.6)
- added R24: R, Resistor_SMD:R_0805_2012Metric, F.Cu at (122.7, 130.6)
- added R25: R, Resistor_SMD:R_0805_2012Metric, F.Cu at (119.7, 141.8)
- added R26: R, Resistor_SMD:R_0805_2012Metric, F.Cu at (122.7, 142.7)
- added R27: R, Resistor_SMD:R_0805_2012Metric, F.Cu at (84.8, 135.6)
- added R28: R, Resistor_SMD:R_0805_2012Metric, F.Cu at (84.8, 137.8)
- added R29: R, Resistor_SMD:R_0805_2012Metric, F.Cu at (97.7, 136.0)
- added R30: R, Resistor_SMD:R_0805_2012Metric, F.Cu at (100.5, 136.8)
- added R31: R, Resistor_SMD:R_0805_2012Metric, F.Cu at (105.6, 140.2)
- added R32: R, Resistor_SMD:R_0805_2012Metric, F.Cu at (108.6, 139.2)
- C11: value C0402C104K4RACTU -> ~; footprint SMV_Passives:CAPC1005X55N -> SMV_Passives:Cap0805
- moved TP_INV2 15.6 mm to (122.8, 126.0)
- moved TP_INV3 11.9 mm to (120.6, 127.8)
- moved C11 11.6 mm to (181.8, 141.8), turned to 180 degrees
- moved TP_AND2 6.81 mm to (118.0, 123.6)
- moved U7 5.30 mm to (122.2, 120.3)
- moved TP_INV4 5.26 mm to (118.6, 127.2)
- moved C6 4.90 mm to (127.2, 121.9)
- moved TP_INV1 4.84 mm to (124.9, 126.8)
- moved R18 3.00 mm to (120.5, 114.3)
- moved TP_AND1 3.00 mm to (118.2, 111.4)
- moved U2 3.00 mm to (121.0, 110.4)
- moved R4 3.00 mm to (120.5, 112.9)
- moved TP_5V1 1.60 mm to (193.8, 141.7)
- moved C4 1.14 mm to (126.9, 134.4), turned to 0 degrees
- moved TP_HSENSE1 1.10 mm to (116.8, 140.8)
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Connections:
- U3 pad 1: /HSENSE_4 -> Net-(U3-1A)
- U3 pad 12: /INVERT -> Net-(U3-6Y)
- U3 pad 13: /HSENSE -> Net-(U3-6A)
- U3 pad 2: /INVERT4 -> Net-(U3-1Y)
- U3 pad 3: /HSENSE_3 -> Net-(U3-2A)
- U3 pad 4: /INVERT3 -> Net-(U3-2Y)
- U3 pad 5: /HSENSE_2 -> Net-(U3-3A)
- U3 pad 6: /INVERT2 -> Net-(U3-3Y)
Routing:
- net /INVERT4: track 8.32 -> 49.5 mm
- net /HSENSE_4: track 49.9 -> 14.5 mm
- net Net-(U3-1A): track 0.00 -> 34.8 mm
- net /INVERT3: track 14.9 -> 38.9 mm, vias 0 -> 2
- net /HSENSE_3: track 36.6 -> 15.8 mm
- net Net-(U3-2A): track 0.00 -> 19.4 mm
- net /INVERT: track 9.35 -> 25.0 mm, vias 0 -> 2
- net /INVERT2: track 15.5 -> 30.9 mm, vias 0 -> 2
- net /HSENSE_2: track 24.4 -> 9.99 mm
- net /HSENSE: track 23.7 -> 10.9 mm
- net Net-(U3-3A): track 0.00 -> 12.6 mm
- net Net-(U3-6A): track 0.00 -> 11.8 mm
- net Net-(U3-3Y): track 0.00 -> 8.79 mm
- net GND: track 68.0 -> 75.7 mm, vias 107 -> 114
- net Net-(U3-2Y): track 0.00 -> 6.66 mm
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