File: safety_board/safety_board.kicad_sch (KiCad schematic)
At the start: 74 parts, among them J1 430450200, J12 XT60-M, J13 XT60-M, J15 22035035, J18 XT60-M, J2 430450200, J3 22035035, J4 22035035, J5 22035035, J6 22035035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

Commit message: pcb almost done
Parts:
- removed R11: 10k ohms, SMV_Passives:RES_CRCW_0402, symbol Device:R_US
- removed U3: MCP6286T-E/OT, SMV_ICs:SOT-23-5_MC_MCH, symbol SMV_Custom:MCP6286T-E_OT
- added R42, R43: 5k ohms, SMV_Passives:RESC2012X50N, symbol Device:R_US
Connections:
- net IGNITION_5V is gone; now on net IGNITION: U7.5 (1D)
- net +12V: now also J9.1; no longer J9.2
- net +3V3: no longer J1.2, J2.2
- net +5V: now also J1.1, J2.1
- net ESTOP1: now also R42.2; no longer J1.1
- net ESTOP2: now also R43.2; no longer J2.1
- net GND: now also J7.N (NEG), U19.4 (COM), U6.4 (COM)
- net at J13.N (NEG): now also U19.3 (NO); no longer U19.NO (3)
- net at F3.2_1, F4.2_1, J13.P (POS): no longer CR3.1
- net at C3.1, U1.3 (VIN): now also J9.2; no longer J9.1
- net at F3.1_1, F4.1_1, U15.3 (NO): now also CR3.1
- net at J18.N (NEG): now also U14.4 (COM); no longer U14.COM (4)
- net at J18.P (POS): now also U14.3 (NO); no longer U14.NO (3)
- new net: J1.2, R42.1
- new net: J2.2, R43.1
Other:
- moved on the sheet: CR3, J1, J2, J9, R1, R2, TP_12V1, TP_ESTOP1, TP_ESTOP2

Commit message: pcb
git commit -m pcb
Parts:
- F1, F2, F3, F4: value 3555-2 -> 3557-2; footprint SMV_Connectors:FUSE_3555-2 -> SMV_Connectors:FUSE_3557-2
Changed lines of the file:
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@@
 			)
 		)
-		(property "Value" "3555-2"
+		(property "Value" "3557-2"
 			(at 123.19 -8.8901 90)
 			(effects
@@
 			)
 		)
-		(property "Footprint" "SMV_Connectors:FUSE_3555-2"
+		(property "Footprint" "SMV_Connectors:FUSE_3557-2"
 			(at 119.38 -10.16 0)
 			(effects
@@
 			)
 		)
-		(property "Value" "3555-2"
+		(property "Value" "3557-2"
 			(at 105.41 38.1 0)
 			(effects
@@
 			)
 		)
-		(property "Footprint" "SMV_Connectors:FUSE_3555-2"
+		(property "Footprint" "SMV_Connectors:FUSE_3557-2"
 			(at 105.41 41.91 0)
 			(effects
@@
 			)
 		)
-		(property "Description" "48V Fuse, 50A limit"
+		(property "Description" ""
 			(at 105.41 41.91 0)
 			(effects
@@
 			)
 		)
-		(property "Value" "3555-2"
+		(property "Value" "3557-2"
 			(at 105.41 41.91 0)
 			(effects
@@
 			)
 		)
-		(property "Footprint" "SMV_Connectors:FUSE_3555-2"
+		(property "Footprint" "SMV_Connectors:FUSE_3557-2"
 			(at 105.41 45.72 0)
 			(effects
@@
 			)
 		)
-		(property "Description" "48V Fuse, 50A limit"
+		(property "Description" ""
 			(at 105.41 45.72 0)
 			(effects
@@
 			)
 		)
-		(property "Value" "3555-2"
+		(property "Value" "3557-2"
 			(at 106.934 -7.62 90)
 			(effects
@@
 			)
 		)
-		(property "Footprint" "SMV_Connectors:FUSE_3555-2"
+		(property "Footprint" "SMV_Connectors:FUSE_3557-2"
 			(at 116.84 -10.16 0)
 			(effects
@@
 			)
 		)
-		(property "Description" "48V Fuse, 50A limit"
+		(property "Description" ""
 			(at 116.84 -10.16 0)
 			(effects

Commit message: maybe possibly final
Parts:
- removed CR3: 5KP48A, DIODE_P600_VIS, symbol SMV_Custom:5KP48A
- added D3: SMA4S56AH, SMV_Passives:SODFL4725X110N, symbol SMV_Custom:SMA4S56AH
- TP_48V1: footprint TestPoint:TestPoint_Pad_D1.0mm -> TestPoint:TestPoint_Pad_D2.0mm
Connections:
- net +12V: now also C3.1, U1.3 (VIN)
- net GND: now also J9.2, D3.A
- net at F3.1_1, F4.1_1, U15.3 (NO): now also D3.C
- net CAN_H renamed CAN_P
- net CAN_L renamed CAN_N
Other:
- moved on the sheet: J9, TP_12V1

Commit message: yay
Parts:
- added H1, H2, H3, H4: MountingHole, MountingHole:MountingHole_3.2mm_M3, symbol Mechanical:MountingHole
- added TP1: TestPoint, SMV_Logo:SEM_logo, symbol Connector:TestPoint

Commit message: yay
Parts:
- removed R13: 10k ohms, SMV_Passives:RES_CRCW_0402, symbol Device:R_US
- added C4: 0.1uF,50V, SMV_Passives:Cap0805, symbol SMV_Custom:C0805C104K5RACTU
- added R3: 1.5k ohms, SMV_Passives:RES_CRCW_0402, symbol Device:R_US
- added TP_48V2, TP_48V3, TP_48V4, TP_48V5, TP_48V6: V_DIVIDED, TestPoint:TestPoint_Pad_D2.0mm, symbol Connector:TestPoint
- added TP_AND2, TP_CAP_GATE_1, TP_INV1, TP_INV2, TP_INV3, TP_INV4: TestPoint, TestPoint:TestPoint_Pad_D1.0mm, symbol Connector:TestPoint
- added U3: SN74AHCT14QPWRQ1, SMV_ICs:PW14, symbol SMV_Custom:SN74AHCT14QPWRQ1
Connections:
- net +3V3: now also C4.1, U3.14 (VCC)
- net GND: now also C4.2, U3.11 (5A), U3.7 (GND), U3.9 (4A)
- net HSENSE: now also U3.13 (6A); no longer U7.13 (2D)
- net HSENSE_2: now also U3.5 (3A); no longer U7.12 (2C)
- net HSENSE_3: now also U3.3 (2A); no longer U7.10 (2B)
- net HSENSE_4: now also U3.1 (1A); no longer U7.9 (2A)
- net at F3.2_1, F4.2_1, J13.P (POS): now also TP_48V4.1
- net at J12.P (POS), U5.3 (NO): now also TP_48V3.1
- net at RP2040.20 (D24): now also R3.1
- net at R12.2, U4.1 (G): now also R3.2, TP_CAP_GATE_1.1
- net at D1.C, F1.2_1, F2.2_1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: now also TP_48V2.1
- net at J18.N (NEG), U14.4 (COM): now also TP_48V6.1
- net at J18.P (POS), U14.3 (NO): now also TP_48V5.1
- net at U7.1 (1A), U7.8 (2Y): now also TP_AND2.1
- new net INVERT: TP_INV1.1, U3.12 (6Y), U7.13 (2D)
- new net INVERT2: TP_INV2.1, U3.6 (3Y), U7.12 (2C)
- new net INVERT3: TP_INV3.1, U3.4 (2Y), U7.10 (2B)
- new net INVERT4: TP_INV4.1, U3.2 (1Y), U7.9 (2A)
- no-connect marks 22 -> 24

Commit message: holla
Parts:
- added R11, R13, R19, R20, R21, R22, R23, R24, R25, R26, R27, R28, R29, R30, R31, R32: R, Resistor_SMD:R_0805_2012Metric, symbol Device:R
- C11: value C0402C104K4RACTU -> ~; footprint SMV_Passives:CAPC1005X55N -> SMV_Passives:Cap0805
Connections:
- net GND: now also R26.1, R27.1, R30.1, R32.1
- net HSENSE: now also R20.2, R25.2; no longer U3.13 (6A)
- net HSENSE_2: now also R19.2, R31.1; no longer U3.5 (3A)
- net HSENSE_3: now also R13.2, R29.1; no longer U3.3 (2A)
- net HSENSE_4: now also R11.2, R28.1; no longer U3.1 (1A)
- net INVERT: now also R20.1, R21.2; no longer U3.12 (6Y)
- net INVERT2: now also R19.1, R24.1; no longer U3.6 (3Y)
- net INVERT3: now also R13.1, R23.1; no longer U3.4 (2Y)
- net INVERT4: now also R11.1, R22.1; no longer U3.2 (1Y)
- new net: R21.1, U3.12 (6Y)
- new net: R25.1, R26.2, U3.13 (6A)
- new net: R29.2, R30.2, U3.3 (2A)
- new net: R22.2, U3.2 (1Y)
- new net: R23.2, U3.4 (2Y)
- new net: R27.2, R28.2, U3.1 (1A)
- new net: R31.2, R32.2, U3.5 (3A)
- new net: R24.2, U3.6 (3Y)
Other:
- moved on the sheet: TP_AND2, TP_INV2, TP_INV3, TP_INV4
