File: UI_Board_Edwin/UI Board.kicad_sch (KiCad schematic)
At the start: 44 parts, among them J1 XT60-M, J2 22035035, J3 22035035, SW1 A8L-11-12N1, U2 CD4511BPWR

Commit message: updated 3/6
Parts:
- removed J2: 22035035, SMV_Connectors:3pin_CON_22035035_MOL, symbol SMV_Custom:3-pin Mini Molex Spox
- removed R21, R22, R23: 220ohm, 1/16W, SMV_Passives:RESC1005X35N, symbol SMV_Custom:CRCW0402220RFKEDC
- removed U4: ~, SMV_ICs:Seven_Seg_display, symbol SMV_Custom:Seven_Seg_Display
- added U3: ~, SMV_ICs:Seven_Seg_display, symbol SMV_Custom:Seven_Seg_Display
Connections:
- net +12V: now also U1.1 (INPUT); no longer U1.3 (OUTPUT)
- net +3.3V: now also U2.4 (*BL); no longer U2.3 (*LT)
- net +5V: now also U1.3 (OUTPUT); no longer U1.1 (INPUT)
- net A: now also U3.11 (A)
- net B: now also U3.7 (B)
- net C: now also U3.4 (C)
- net D: now also U3.2 (D)
- net DIGIT_1: now also U3.12 (DIGIT_1); no longer R20.2
- net DIGIT_2: now also U3.9 (DIGIT_2)
- net DIGIT_3: now also U3.8 (DIGIT_3)
- net DIGIT_4: now also RP1.14 (TX), U3.6 (DIGIT_4); no longer RP1.12 (SDA)
- net DP: now also R20.1, RP1.12 (SDA); no longer RP1.14 (TX)
- net E: now also U3.1 (E)
- net F: now also U3.10 (F)
- net G: now also U3.5 (G)
- net GND: no longer U2.4 (*BL)
- net WIPERS: now also RP1.11 (SCL); no longer RP1.13 (D4)
- new net: R20.2, U3.3 (DP)
- new net LT: RP1.13 (D4), U2.3 (*LT)
- no-connect marks 9 -> 8
Other:
- moved on the sheet: C1, C2

Commit message: i think done
Parts:
- added TP1, TP2, TP3, TP4: TestPoint, TestPoint:TestPoint_Pad_2.5x2.5mm, symbol Connector:TestPoint
Connections:
- net +12V: now also TP2.1
- net +3.3V: now also TP3.1
- net +5V: now also TP1.1
- net DIGIT_1: now also RP1.15 (RX); no longer RP1.17 (MOSI)
- net DIGIT_3: now also RP1.17 (MOSI); no longer RP1.15 (RX)
- net GND: now also TP4.1

Commit message: added test points
Parts:
- added TP5, TP6, TP7: TestPoint, TestPoint:TestPoint_Pad_2.5x2.5mm, symbol Connector:TestPoint
Connections:
- net CAN_N: now also TP6.1
- net CAN_P: now also TP5.1
- net LT: now also TP7.1

Commit message: ay
Parts:
- added H1, H2, H3, H4: MountingHole, MountingHole:MountingHole_3.2mm_M3, symbol Mechanical:MountingHole
- added TP8: TestPoint, SMV_Logo:SEM_logo, symbol Connector:TestPoint
