File: UI_Board_Edwin/UI Board.kicad_pcb (KiCad board)
At the start: 2 copper layers, 170.4 x 95.8 mm, 45 parts, among them J1 XT60-M, J2 22035035, J3 22035035, SW1 A8L-11-12N1, U2 CD4511BPWR

Commit message: updated 3/6
Parts:
- removed J2: 22035035, SMV_Connectors:3pin_CON_22035035_MOL
- removed R21, R22, R23: 220ohm, 1/16W, SMV_Passives:RESC1005X35N
- removed U4: ~, SMV_ICs:Seven_Seg_display
- added U3: ~, SMV_ICs:Seven_Seg_display, F.Cu at (235.3, 112.3)
- moved R16 24.8 mm to (229.0, 101.6), turned to -90 degrees
- moved R20 22.7 mm to (234.0, 123.0)
- moved R14 21.4 mm to (239.1, 123.0), turned to 90 degrees
- moved J3 7.20 mm to (254.5, 76.2)
- moved R15 5.09 mm to (239.1, 101.6)
- moved C1 0.44 mm to (214.4, 54.7), turned to 0 degrees
- moved C2 0.16 mm to (214.3, 43.8), turned to 180 degrees
- moved U1 0.12 mm to (214.2, 49.4), turned to -90 degrees
Connections:
- R20 pad 1: Net-(U4-DIGIT_1) -> /DP
- R20 pad 2: /DIGIT_1 -> Net-(U3-DP)
- RP1 pad 11: unconnected-(RP1-SCL-Pad11) -> /WIPERS
- RP1 pad 12: /DIGIT_4 -> /DP
- RP1 pad 13: /WIPERS -> /LT
- RP1 pad 14: /DP -> /DIGIT_4
- U1 pad 1: +5V -> +12V
- U1 pad 3: +12V -> +5V
- U2 pad 3: +3.3V -> /LT
- U2 pad 4: GND -> +3.3V
Routing:
- net /DIGIT_4: track 71.6 -> 37.3 mm
- net /DP: track 39.7 -> 71.2 mm
- net Net-(R16-Pad1): track 35.3 -> 7.55 mm
- net /LT: track 0.00 -> 24.1 mm
- net +3.3V: track 5.59 -> 24.5 mm
- net Net-(R15-Pad1): track 10.7 -> 22.9 mm
- net Net-(U2-G): track 23.4 -> 33.6 mm
- net /CAN_P: track 19.4 -> 10.3 mm
- net /CAN_N: track 19.4 -> 10.3 mm
- net /DIGIT_2: track 40.7 -> 33.3 mm
- net /DIGIT_3: track 43.0 -> 35.8 mm
- net +12V: track 0.00 -> 4.45 mm
- net Net-(U4-DIGIT_4): track 2.59 -> 0.00 mm
- net Net-(U3-DP): track 0.00 -> 2.55 mm
- net Net-(U4-DIGIT_3): track 2.55 -> 0.00 mm
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Other:
- outline, holes or cut-outs redrawn

Commit message: i think done
Parts:
- added 12V: TestPoint, TestPoint:TestPoint_Pad_2.5x2.5mm, F.Cu at (236.4, 43.4)
- added 3.3V: TestPoint, TestPoint:TestPoint_Pad_2.5x2.5mm, F.Cu at (220.2, 91.8)
- added 5V: TestPoint, TestPoint:TestPoint_Pad_2.5x2.5mm, F.Cu at (206.3, 51.7)
- added GND: TestPoint, TestPoint:TestPoint_Pad_2.5x2.5mm, F.Cu at (161.0, 102.2)
- moved R16 12.7 mm to (241.7, 101.6)
- moved R15 7.53 mm to (231.6, 101.6)
- moved R13 2.46 mm to (234.1, 101.6)
Connections:
- RP1 pad 15: /DIGIT_3 -> /DIGIT_1
- RP1 pad 17: /DIGIT_1 -> /DIGIT_3
Routing:
- net /DIGIT_1: track 23.8 -> 46.2 mm
- net Net-(R16-Pad1): track 7.55 -> 26.3 mm
- net Net-(R15-Pad1): track 22.9 -> 8.32 mm
- net Net-(U2-G): track 33.6 -> 43.3 mm
- net /DIGIT_2: track 33.3 -> 40.5 mm
- net +5V: track 16.1 -> 20.9 mm
- net GND: track 41.0 -> 44.0 mm, vias 17 -> 18
- net +3.3V: track 24.5 -> 27.2 mm
- net /DIGIT_4: track 37.3 -> 39.7 mm
- net Net-(U2-F): track 11.2 -> 8.83 mm
- net /DIGIT_3: track 35.8 -> 34.0 mm
- net /DP: track 71.2 -> 72.0 mm
Other:
- outline, holes or cut-outs redrawn

Commit message: added test points
Parts:
- added CAN_N: TestPoint, TestPoint:TestPoint_Pad_2.5x2.5mm, F.Cu at (254.5, 64.5)
- added CAN_P: TestPoint, TestPoint:TestPoint_Pad_2.5x2.5mm, F.Cu at (254.5, 83.5)
- added LT: TestPoint, TestPoint:TestPoint_Pad_2.5x2.5mm, F.Cu at (249.4, 94.4)
- renumbered 5V to TP1, 12V to TP2, 3.3V to TP3, GND to TP4
Routing:
- net /LT: track 24.1 -> 36.6 mm
- net /CAN_P: track 10.3 -> 17.7 mm
- net /CAN_N: track 10.3 -> 17.1 mm
- net /DP: track 72.0 -> 76.8 mm
- net /WIPERS: track 99.4 -> 103.1 mm

Commit message: ay
Parts:
- added H1: MountingHole, MountingHole:MountingHole_3.2mm_M3, F.Cu at (262.2, 41.7)
- added H2: MountingHole, MountingHole:MountingHole_3.2mm_M3, F.Cu at (262.2, 126.8)
- added H3: MountingHole, MountingHole:MountingHole_3.2mm_M3, F.Cu at (104.1, 41.7)
- added H4: MountingHole, MountingHole:MountingHole_3.2mm_M3, F.Cu at (104.1, 126.2)
- added TP8: TestPoint, SMV_Logo:SEM_logo, F.Cu at (130.2, 116.7)
- moved TP5 6.60 mm to (254.5, 76.9)
- moved J3 6.50 mm to (261.0, 76.0)
- moved TP6 5.83 mm to (254.5, 70.3)
- moved C1 4.74 mm to (218.0, 57.8)
- moved C2 4.74 mm to (217.9, 46.9)
- moved TP1 4.74 mm to (209.9, 54.9)
- moved U1 4.74 mm to (217.8, 52.5)
- renumbered CAN_P to TP5, CAN_N to TP6, LT to TP7
Routing:
- net +5V: track 20.9 -> 16.3 mm
- net /CAN_N: track 17.1 -> 19.5 mm
- net /CAN_P: track 17.7 -> 19.2 mm
- net GND: vias 18 -> 26
- removed copper zone on F.Cu, net +12V
Other:
- board text added: "12V_IN"
- board text added: "Edwin Tang 3/9/25 UI Board"

Commit message: hu
Routing:
- net +3.3V: track 27.2 -> 37.7 mm, vias 0 -> 2
- net /Horn: track 100.9 -> 99.7 mm
Changed lines of the file:
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@@
 		(grid_origin -0.01 210.01)
 		(pcbplotparams
-			(layerselection 0x00010fc_ffffffff)
+			(layerselection 0x00010f0_ffffffff)
 			(plot_on_all_layers_selection 0x0000000_00000000)
 			(disableapertmacros no)
@@
 			(outputformat 1)
 			(mirror no)
-			(drillshape 1)
+			(drillshape 0)
 			(scaleselection 1)
-			(outputdirectory "")
+			(outputdirectory "../../UIorder/")
 		)
 	)
@@
 		(fp_arc
 			(start -14.415423 12.084309)
-			(mid -14.421008 12.080061)
+			(mid -14.421008 12.080062)
 			(end -14.41863 12.07346)
 			(stroke
@@
 		(fp_arc
 			(start -8.304556 8.25436)
-			(mid -8.304689 8.247612)
+			(mid -8.304689 8.247611)
 			(end -8.300511 8.24231)
 			(stroke
@@
 		(fp_arc
 			(start -7.774364 12.655021)
-			(mid -7.771131 12.665266)
+			(mid -7.771131 12.665267)
 			(end -7.776942 12.674303)
 			(stroke
@@
 		(fp_arc
 			(start -4.883602 11.697921)
-			(mid -4.883173 11.693201)
+			(mid -4.883173 11.693202)
 			(end -4.878724 11.69157)
 			(stroke
@@
 		(fp_arc
 			(start -3.156379 11.616037)
-			(mid -3.161129 11.513181)
+			(mid -3.16113 11.513181)
 			(end -3.16328 11.410238)
 			(stroke
@@
 		(fp_arc
 			(start -0.45284 6.767971)
-			(mid -0.453954 6.770748)
+			(mid -0.453954 6.770747)
 			(end -0.456677 6.771986)
 			(stroke
@@
 	)
 	(segment
+		(start 231.74 95.76)
+		(end 231.74 94.56)
+		(width 0.2)
+		(layer "F.Cu")
+		(net 1)
+	)
+	(segment
 		(start 227.42175 89.887201)
 		(end 227.42175 88.9212)
@@
 	)
 	(segment
+		(start 231.19 96.31)
+		(end 231.74 95.76)
+		(width 0.2)
+		(layer "F.Cu")
+		(net 1)
+	)
+	(segment
 		(start 210.88175 89.71)
 		(end 213.00675 91.835)
@@
 		(net 1)
 	)
+	(via
+		(at 231.19 96.31)
+		(size 0.6)
+		(drill 0.3)
+		(layers "F.Cu" "B.Cu")
+		(net 1)
+	)
+	(via
+		(at 222.89 96.91)
+		(size 0.6)
+		(drill 0.3)
+		(layers "F.Cu" "B.Cu")
+		(free yes)
+		(net 1)
+	)
+	(segment
+		(start 231.19 96.31)
+		(end 230.59 96.91)
+		(width 0.2)
+		(layer "B.Cu")
+		(net 1)
+	)
+	(segment
+		(start 230.59 96.91)
+		(end 222.89 96.91)
+		(width 0.2)
+		(layer "B.Cu")
+		(net 1)
+	)
 	(segment
 		(start 146.68175 63.253)
@@
 	)
 	(segment
-		(start 147.30175 64.92)
-		(end 146.48175 64.1)
-		(width 0.5)
-		(layer "F.Cu")
-		(net 2)
-	)
-	(segment
 		(start 150.04175 67.66)
 		(end 146.68175 64.3)
@@
 	)
 	(segment
-		(start 133.89 68.89)
-		(end 133.66241 68.89)
-		(width 0.5)
-		(layer "F.Cu")
-		(net 14)
-	)
-	(segment
